File: power.kicad_sch (KiCad schematic)
At the start: 24 parts, among them Q1 AO3401A, U1 TPS62933

Commit message: add sheet name, explain
Other:
- note added: "POWER"
Changed lines of the file:
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@@
     (effects (font (size 2.54 2.54)) (justify left bottom))
   )
-  (text "BUCK CONVERTER" (at 111.76 90.17 0)
+  (text "POWER" (at 190.5 177.8 0)
+    (effects (font (size 5.08 5.08)) (justify left bottom))
+  )
+  (text "BUCK CONVERTER" (at 111.76 91.44 0)
     (effects (font (size 1.27 1.27)) (justify left bottom))
   )
@@
     (effects (font (size 1.27 1.27)) (justify left bottom))
   )
-  (text "REVERSE POLARITY\nPROTECTION" (at 88.9 40.64 0)
+  (text "REVERSE POLARITY\nPROTECTION" (at 80.01 41.91 0)
     (effects (font (size 2.54 2.54)) (justify left bottom))
   )

Commit message: modify symbol number, constant
Parts:
- renumbered C5 to C1, C26 to C10, C6 to C2, C7 to C3, C12 to C4, C3 to C5, C11 to C6, C8 to C7, C9 to C8, C10 to C9, D4 to D1, D3 to D2, D2 to D3, R9 to R1, R10 to R2, R4 to R3, R14 to R4, R11 to R5, R12 to R6, R13 to R7

Commit message: decide constant
Parts:
- C1, C2: value C -> 10u
- C10, C3, C6: value C -> 0.1u
- C4: value C -> 33n
- C5: value C_Polarized -> 47u
- C7: value C -> 47p
- C8, C9: value C -> 22u
- L1: value L -> 6.8u
- R1: value R -> 430k
- R2: value R -> 51.1k
- R3: value R -> 10k
- R4: value R -> 0
- R5: renamed from R6; value R -> 52.3k
- R6: renamed from R5; value R -> 10k
- R7: value R -> 300
Connections:
- net GND: no longer C7.2
- net at R5.1, R6.1, U1.8 (FB): now also C7.2
Other:
- note added: ") + I_{h}"
- note added: "- V_{STOP}"
- note added: "I_{p} : 0.7 uA, I_{h} : 1.4 uA V_{EN_FALL} : 1.17 V, V_{EN_RISE} : 1.21 V V_{START} : THE INPUT VOLTAGE ENABLING THE DEVICE, 11 V V_{STOP} : THE INPUT VOLTAGE DISABLING THE DEVICE, 10 V"
- note added: "I_{p} x ( 1 -"
- note added: "R_{1} ="
- note added: "R_{1} x V_{EN_FALL}"
- note added: "R_{2} ="
- note added: "R_{5} ="
- note added: "V_{EN_FALL}"
- note added: "V_{EN_RISE}"
- note added: "V_{OUT} - V_{REF}"
- note added: "V_{REF}"
- note added: "V_{REF} : IC IS DESIGNED AT 0.8 V V_{OUT} : THE OUTPUT VOLTAGE, 5 V R_{7} : 10.2 kOHM"
- note added: "V_{START} x"
- note added: "V_{STOP} - V_{EN_FALL} + R_{1} x ( I_{p} + I_{h} )"
- note added: "x R_{6}"
- moved on the sheet: C10, C8, C9, R5, R6

Commit message: decide constant
Parts:
- D3: value LED -> LED_R
Changed lines of the file:
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@@
       (effects (font (size 1.27 1.27)) (justify right))
     )
-    (property "Value" "LED" (at 232.41 110.8075 90)
+    (property "Value" "LED_R" (at 232.41 110.8075 90)
       (effects (font (size 1.27 1.27)) (justify right))
     )

Commit message: modify constant
Parts:
- R3: value 10k -> 15k
Changed lines of the file:
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@@
       (effects (font (size 1.27 1.27)) (justify left))
     )
-    (property "Value" "10k" (at 104.14 71.12 0)
+    (property "Value" "15k" (at 104.14 71.12 0)
       (effects (font (size 1.27 1.27)) (justify left))
     )

Commit message: add and modify 発注先 and footprint
Parts:
- C1, C2, C4, C5, C7, C8, C9, R1, R2, R4, R5, U1: 発注先 (none) -> Digi-Key
- C10, C3, C6: footprint (none) -> Capacitor_SMD:C_0603_1608Metric; 発注先 (none) -> Digi-Key
- D1: value UDZV5.1B -> UDZVTE-175.1B; 発注先 (none) -> 秋月電子
- D3: footprint (none) -> LED_SMD:LED_0603_1608Metric; 発注先 (none) -> Digi-Key
- Q1: 発注先 (none) -> 秋月電子
- R3, R6, R7: footprint (none) -> Resistor_SMD:R_0603_1608Metric; 発注先 (none) -> Digi-Key
Changed lines of the file:
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@@
+      (effects (font (size 1.27 1.27)) hide)
+    )
+    (property "発注先" "Digi-Key" (at 63.5 107.95 0)
       (effects (font (size 1.27 1.27)) hide)
     )
@@
       (effects (font (size 1.27 1.27)))
     )
-    (property "Footprint" "" (at 149.86 100.6348 0)
+    (property "Footprint" "Capacitor_SMD:C_0603_1608Metric" (at 149.86 100.6348 0)
       (effects (font (size 1.27 1.27)) hide)
     )
@@
       (effects (font (size 1.27 1.27)) hide)
     )
+    (property "発注先" "Digi-Key" (at 146.05 101.6 0)
+      (effects (font (size 1.27 1.27)) hide)
+    )
     (pin "1")
     (pin "2")
@@
     )
     (property "在庫" "" (at 101.6 118.11 0)
+      (effects (font (size 1.27 1.27)) hide)
+    )
+    (property "発注先" "Digi-Key" (at 101.6 118.11 0)
       (effects (font (size 1.27 1.27)) hide)
     )
@@
       (effects (font (size 1.27 1.27)) (justify right))
     )
-    (property "Footprint" "" (at 228.6 107.95 0)
+    (property "Footprint" "LED_SMD:LED_0603_1608Metric" (at 228.6 107.95 0)
       (effects (font (size 1.27 1.27)) hide)
     )
@@
       (effects (font (size 1.27 1.27)) hide)
     )
+    (property "発注先" "Digi-Key" (at 228.6 107.95 0)
+      (effects (font (size 1.27 1.27)) hide)
+    )
     (pin "1")
     (pin "2")
@@
       (effects (font (size 1.27 1.27)) (justify left))
     )
-    (property "Footprint" "" (at 99.822 69.85 90)
+    (property "Footprint" "Resistor_SMD:R_0603_1608Metric" (at 99.822 69.85 90)
       (effects (font (size 1.27 1.27)) hide)
     )
@@
     )
     (property "在庫" "" (at 101.6 69.85 0)
+      (effects (font (size 1.27 1.27)) hide)
+    )
+    (property "発注先" "Digi-Key" (at 101.6 69.85 0)
       (effects (font (size 1.27 1.27)) hide)
     )
@@
       (effects (font (size 1.27 1.27)) hide)
     )
+    (property "発注先" "Digi-Key" (at 88.9 107.95 0)
+      (effects (font (size 1.27 1.27)) hide)
+    )
     (pin "1")
     (pin "2")
@@
       (effects (font (size 1.27 1.27)) (justify left))
     )
-    (property "Footprint" "" (at 77.1652 111.76 0)
+    (property "Footprint" "Capacitor_SMD:C_0603_1608Metric" (at 77.1652 111.76 0)
       (effects (font (size 1.27 1.27)) hide)
     )
@@
       (effects (font (size 1.27 1.27)) hide)
     )
+    (property "発注先" "Digi-Key" (at 76.2 107.95 0)
+      (effects (font (size 1.27 1.27)) hide)
+    )
     (pin "1")
     (pin "2")
@@
       (effects (font (size 1.27 1.27)) hide)
     )
+    (property "発注先" "Digi-Key" (at 190.5 107.95 0)
+      (effects (font (size 1.27 1.27)) hide)
+    )
     (pin "1")
     (pin "2")
@@
       (effects (font (size 1.27 1.27)) (justify left))
     )
-    (property "Value" "UDZV5.1B" (at 104.14 58.42 90)
+    (property "Value" "UDZVTE-175.1B" (at 104.14 58.42 90)
       (effects (font (size 1.27 1.27)) (justify left))
     )
@@
     )
     (property "在庫" "" (at 101.6 57.15 0)
+      (effects (font (size 1.27 1.27)) hide)
+    )
+    (property "発注先" "秋月電子" (at 101.6 57.15 0)
       (effects (font (size 1.27 1.27)) hide)
     )
@@
       (effects (font (size 1.27 1.27)) hide)
     )
+    (property "発注先" "Digi-Key" (at 177.8 107.95 0)
+      (effects (font (size 1.27 1.27)) hide)
+    )
     (pin "1")
     (pin "2")
@@
       (effects (font (size 1.27 1.27)) (justify left))
     )
-    (property "Footprint" "" (at 226.822 120.65 90)
+    (property "Footprint" "Resistor_SMD:R_0603_1608Metric" (at 226.822 120.65 90)
       (effects (font (size 1.27 1.27)) hide)
     )
@@
       (effects (font (size 1.27 1.27)) hide)
     )
+    (property "発注先" "Digi-Key" (at 228.6 120.65 0)
+      (effects (font (size 1.27 1.27)) hide)
+    )
     (pin "1")
     (pin "2")
@@
       (effects (font (size 1.27 1.27)) (justify left))
     )
-    (property "Footprint" "" (at 176.022 120.65 90)
+    (property "Footprint" "Resistor_SMD:R_0603_1608Metric" (at 176.022 120.65 90)
       (effects (font (size 1.27 1.27)) hide)
     )
@@
       (effects (font (size 1.27 1.27)) hide)
     )
+    (property "発注先" "Digi-Key" (at 177.8 120.65 0)
+      (effects (font (size 1.27 1.27)) hide)
+    )
     (pin "1")
     (pin "2")
@@
       (effects (font (size 1.27 1.27)) (justify left))
     )
-    (property "Footprint" "" (at 216.8652 111.76 0)
+    (property "Footprint" "Capacitor_SMD:C_0603_1608Metric" (at 216.8652 111.76 0)
       (effects (font (size 1.27 1.27)) hide)
     )
@@
       (effects (font (size 1.27 1.27)) hide)
     )
+    (property "発注先" "Digi-Key" (at 215.9 107.95 0)
+      (effects (font (size 1.27 1.27)) hide)
+    )
     (pin "1")
     (pin "2")
@@
     )
     (property "在庫" "" (at 88.9 120.65 0)
+      (effects (font (size 1.27 1.27)) hide)
+    )
+    (property "発注先" "Digi-Key" (at 88.9 120.65 0)
       (effects (font (size 1.27 1.27)) hide)
     )
@@
       (effects (font (size 1.27 1.27)) hide)
     )
+    (property "発注先" "秋月電子" (at 88.9 53.34 0)
+      (effects (font (size 1.27 1.27)) hide)
+    )
     (pin "1")
     (pin "2")
@@
       (effects (font (size 1.27 1.27)) hide)
     )
+    (property "発注先" "Digi-Key" (at 133.35 101.6 0)
+      (effects (font (size 1.27 1.27)) hide)
+    )
     (pin "1")
     (pin "2")
@@
       (effects (font (size 1.27 1.27)) hide)
     )
+    (property "発注先" "Digi-Key" (at 203.2 107.95 0)
+      (effects (font (size 1.27 1.27)) hide)
+    )
     (pin "1")
     (pin "2")
@@
       (effects (font (size 1.27 1.27)) hide)
     )
+    (property "発注先" "Digi-Key" (at 165.1 107.95 0)
+      (effects (font (size 1.27 1.27)) hide)
+    )
     (pin "1")
     (pin "2")
@@
       (effects (font (size 1.27 1.27)) hide)
     )
+    (property "発注先" "Digi-Key" (at 127 57.15 0)
+      (effects (font (size 1.27 1.27)) hide)
+    )
     (pin "1")
     (pin "2")
@@
     )
     (property "在庫" "" (at 120.65 109.22 0)
+      (effects (font (size 1.27 1.27)) hide)
+    )
+    (property "発注先" "Digi-Key" (at 120.65 109.22 0)
       (effects (font (size 1.27 1.27)) hide)
     )
@@
       (effects (font (size 1.27 1.27)) hide)
     )
+    (property "発注先" "Digi-Key" (at 50.8 107.95 0)
+      (effects (font (size 1.27 1.27)) hide)
+    )

Commit message: add footprint
Parts:
- R1, R2, R4, R5: footprint (none) -> Resistor_SMD:R_0603_1608Metric
Changed lines of the file:
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@@
       (effects (font (size 1.27 1.27)) (justify left))
     )
-    (property "Footprint" "" (at 87.122 107.95 90)
+    (property "Footprint" "Resistor_SMD:R_0603_1608Metric" (at 87.122 107.95 90)
       (effects (font (size 1.27 1.27)) hide)
     )
@@
       (effects (font (size 1.27 1.27)) (justify right))
     )
-    (property "Footprint" "" (at 179.578 107.95 90)
+    (property "Footprint" "Resistor_SMD:R_0603_1608Metric" (at 179.578 107.95 90)
       (effects (font (size 1.27 1.27)) hide)
     )
@@
       (effects (font (size 1.27 1.27)) (justify left))
     )
-    (property "Footprint" "" (at 87.122 120.65 90)
+    (property "Footprint" "Resistor_SMD:R_0603_1608Metric" (at 87.122 120.65 90)
       (effects (font (size 1.27 1.27)) hide)
     )
@@
       (effects (font (size 1.27 1.27)))
     )
-    (property "Footprint" "" (at 133.35 103.378 90)
-      (effects (font (size 1.27 1.27)) hide)
-    )
+    (property "Footprint" "Resistor_SMD:R_0603_1608Metric" (at 133.35 103.378 90)
+      (effects (font (size 1.27 1.27)) hide)
+    )
