File: power.kicad_sch (KiCad schematic)
At the start: 24 parts, among them Q1 AO3401A, U1 TPS62933

Commit message: add footprints to C
Parts:
- C1, C2, C8, C9: footprint (none) -> Capacitor_SMD:C_0805_2012Metric
- C4, C7: footprint (none) -> Capacitor_SMD:C_0402_1005Metric
- C5: footprint (none) -> Capacitor_SMD:CP_Elec_6.3x5.4_Nichicon
- L1: footprint (none) -> ProjectEV-kicad-library:NR10050T150M
Changed lines of the file:
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@@
       (effects (font (size 1.27 1.27)) (justify left))
     )
-    (property "Footprint" "" (at 64.4652 111.76 0)
+    (property "Footprint" "Capacitor_SMD:C_0805_2012Metric" (at 64.4652 111.76 0)
       (effects (font (size 1.27 1.27)) hide)
     )
@@
       (effects (font (size 1.27 1.27)) (justify left))
     )
-    (property "Footprint" "" (at 102.5652 121.92 0)
+    (property "Footprint" "Capacitor_SMD:C_0402_1005Metric" (at 102.5652 121.92 0)
       (effects (font (size 1.27 1.27)) hide)
     )
@@
       (effects (font (size 1.27 1.27)) (justify left))
     )
-    (property "Footprint" "" (at 191.4652 111.76 0)
+    (property "Footprint" "Capacitor_SMD:C_0805_2012Metric" (at 191.4652 111.76 0)
       (effects (font (size 1.27 1.27)) hide)
     )
@@
       (effects (font (size 1.27 1.27)))
     )
-    (property "Footprint" "" (at 158.75 101.6 0)
+    (property "Footprint" "ProjectEV-kicad-library:NR10050T150M" (at 158.75 101.6 0)
       (effects (font (size 1.27 1.27)) hide)
     )
@@
       (effects (font (size 1.27 1.27)) (justify left))
     )
-    (property "Footprint" "" (at 204.1652 111.76 0)
+    (property "Footprint" "Capacitor_SMD:C_0805_2012Metric" (at 204.1652 111.76 0)
       (effects (font (size 1.27 1.27)) hide)
     )
@@
       (effects (font (size 1.27 1.27)) (justify left))
     )
-    (property "Footprint" "" (at 166.0652 111.76 0)
+    (property "Footprint" "Capacitor_SMD:C_0402_1005Metric" (at 166.0652 111.76 0)
       (effects (font (size 1.27 1.27)) hide)
     )
@@
       (effects (font (size 1.27 1.27)) (justify left))
     )
-    (property "Footprint" "" (at 127.9652 60.96 0)
+    (property "Footprint" "Capacitor_SMD:CP_Elec_6.3x5.4_Nichicon" (at 127.9652 60.96 0)
       (effects (font (size 1.27 1.27)) hide)
     )
@@
       (effects (font (size 1.27 1.27)) (justify left))
     )
-    (property "Footprint" "" (at 51.7652 111.76 0)
-      (effects (font (size 1.27 1.27)) hide)
-    )
+    (property "Footprint" "Capacitor_SMD:C_0805_2012Metric" (at 51.7652 111.76 0)
+      (effects (font (size 1.27 1.27)) hide)
+    )

Commit message: add tolerance
Other:
- note added: "0.1%"
Changed lines of the file:
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@@
     (effects (font (size 5.08 5.08)) (justify left bottom))
+  )
+  (text "0.1%" (at 180.34 113.03 0)
+    (effects (font (size 1.27 1.27)) (justify left bottom))
   )
   (text "- V_{STOP}" (at 90.17 146.05 0)
@@
     (effects (font (size 1.27 1.27)) (justify left bottom))
   )
+  (text "0.1%" (at 180.34 125.73 0)
+    (effects (font (size 1.27 1.27)) (justify left bottom))
+  )

Commit message: modify footprint path and 3dmodel path
Parts:
- D2: footprint SamacSys_Parts:CUHS20S40H3F -> ProjectEV-kicad-library:CUHS20S40H3F
Changed lines of the file:
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@@
       (effects (font (size 1.27 1.27)) (justify right))
     )
-    (property "Footprint" "SamacSys_Parts:CUHS20S40H3F" (at 190.5 95.25 0)
+    (property "Footprint" "ProjectEV-kicad-library:CUHS20S40H3F" (at 190.5 95.25 0)
       (effects (font (size 1.27 1.27)) hide)
     )

Commit message: modify L1
value, footprint, 発注先
Parts:
- L1: value 6.8u -> 22u; footprint ProjectEV-kicad-library:NR10050T150M -> ProjectEV-kicad-library:L_MGAH0603; 発注先 (none) -> Digi-Key
Changed lines of the file:
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@@
       (effects (font (size 1.27 1.27)))
     )
-    (property "Value" "6.8u" (at 158.75 99.06 90)
+    (property "Value" "22u" (at 158.75 99.06 90)
       (effects (font (size 1.27 1.27)))
     )
-    (property "Footprint" "ProjectEV-kicad-library:NR10050T150M" (at 158.75 101.6 0)
+    (property "Footprint" "ProjectEV-kicad-library:L_MGAH0603" (at 158.75 101.6 0)
       (effects (font (size 1.27 1.27)) hide)
     )
@@
       (effects (font (size 1.27 1.27)) hide)
     )
+    (property "発注先" "Digi-Key" (at 158.75 101.6 0)
+      (effects (font (size 1.27 1.27)) hide)
+    )

Commit message: ヒューズ変更、コネクタ配置変更、CANまわり配置修正
Parts:
- removed F1: MF-USHT020KX-2, Fuse:Fuse_1210_3225Metric, symbol Device:Polyfuse
- added F1: ERB-RD1R50X, Fuse:Fuse_0402_1005Metric, symbol Device:Fuse
Connections:
- net +BATT: now also F1.1
- net at Q1.3 (D): now also F1.2
Changed lines of the file:
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@@
+    )
+  )
+  (symbol (lib_id "Device:Fuse") (at 63.5 50.8 90) (unit 1)
+    (in_bom yes) (on_board yes) (dnp no) (fields_autoplaced)
+    (property "Reference" "F1" (at 63.5 45.72 90)
+      (effects (font (size 1.27 1.27)))
+    )
+    (property "Value" "ERB-RD1R50X" (at 63.5 48.26 90)
+      (effects (font (size 1.27 1.27)))
+    )
+    (property "Footprint" "Fuse:Fuse_0402_1005Metric" (at 63.5 52.578 90)
+      (effects (font (size 1.27 1.27)) hide)
+    )
+    (property "Datasheet" "~" (at 63.5 50.8 0)
+      (effects (font (size 1.27 1.27)) hide)
+    )
+    (property "発注先" "Digi-Key" (at 63.5 50.8 0)
+      (effects (font (size 1.27 1.27)) hide)
+    )
+    (pin "2")
+    (pin "1")
+    (instances
+      (project "main-ECU-board"
+        (path "/10edd9b6-c7a8-40f4-bfe3-c9724324d30f/66822db1-000e-41a8-b261-6f81d2c690fe"
+          (reference "F1") (unit 1)
+        )
+      )
     )
   )
@@
         )
       )
-    )
-  )
-  (symbol (lib_id "Device:Polyfuse") (at 63.5 50.8 270) (unit 1)
-    (in_bom yes) (on_board yes) (dnp no) (fields_autoplaced)
-    (property "Reference" "F1" (at 63.5 44.45 90)
-      (effects (font (size 1.27 1.27)))
-    )
-    (property "Value" "MF-USHT020KX-2" (at 63.5 46.99 90)
-      (effects (font (size 1.27 1.27)))
-    )
-    (property "Footprint" "Fuse:Fuse_1210_3225Metric" (at 58.42 52.07 0)
-      (effects (font (size 1.27 1.27)) (justify left) hide)
-    )
-    (property "Datasheet" "~" (at 63.5 50.8 0)
-      (effects (font (size 1.27 1.27)) hide)
-    )
-    (property "発注先" "Digi-Key" (at 63.5 50.8 90)
-      (effects (font (size 1.27 1.27)) hide)
-    )
-    (pin "1")
-    (pin "2")
-    (instances
-      (project "main-ECU-board"
-        (path "/10edd9b6-c7a8-40f4-bfe3-c9724324d30f/66822db1-000e-41a8-b261-6f81d2c690fe"
-          (reference "F1") (unit 1)
-        )
-      )
