File: main-ECU-board.kicad_sch (KiCad schematic)
At the start: 4 parts, among them J1 Power, J2 Analog, J3 Digital/PWM, J4 Digital/PWM

Commit message: add MCU, type-C
Parts:
- added IC1: R7FA4M1AB3CFM#AA0, QFP50P1200X1200X170-64N, symbol SamacSys_Parts:R7FA4M1AB3CFM#AA0
- added J5: USB_C_Receptacle, SamacSys_Parts:5077CR-16-SMC2-BK-TR, symbol Connector:USB_C_Receptacle
Connections:
- new net: J5.A1 (GND), J5.A12 (GND), J5.B1 (GND), J5.B12 (GND)
- new net: J5.A4 (VBUS), J5.A9 (VBUS), J5.B4 (VBUS), J5.B9 (VBUS)
Changed lines of the file:
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@@
+    )
+  )
+  (symbol (lib_id "Connector:USB_C_Receptacle") (at 76.2 139.7 0) (unit 1)
+    (in_bom yes) (on_board yes) (dnp no) (fields_autoplaced)
+    (property "Reference" "J5" (at 76.2 106.68 0)
+      (effects (font (size 1.27 1.27)))
+    )
+    (property "Value" "USB_C_Receptacle" (at 76.2 109.22 0)
+      (effects (font (size 1.27 1.27)))
+    )
+    (property "Footprint" "SamacSys_Parts:5077CR-16-SMC2-BK-TR" (at 80.01 139.7 0)
+      (effects (font (size 1.27 1.27)) hide)
+    )
+    (property "Datasheet" "https://www.usb.org/sites/default/files/documents/usb_type-c.zip" (at 80.01 139.7 0)
+      (effects (font (size 1.27 1.27)) hide)
+    )
+    (pin "A1")
+    (pin "A10")
+    (pin "A11")
+    (pin "A12")
+    (pin "A2")
+    (pin "A3")
+    (pin "A4")
+    (pin "A5")
+    (pin "A6")
+    (pin "A7")
+    (pin "A8")
+    (pin "A9")
+    (pin "B1")
+    (pin "B10")
+    (pin "B11")
+    (pin "B12")
+    (pin "B2")
+    (pin "B3")
+    (pin "B4")
+    (pin "B5")
+    (pin "B6")
+    (pin "B7")
+    (pin "B8")
+    (pin "B9")
+    (pin "S1")
+    (instances
+      (project "main-ECU-board"
+        (path "/10edd9b6-c7a8-40f4-bfe3-c9724324d30f"
+          (reference "J5") (unit 1)
+        )
+      )
     )
   )
@@
         )
       )
+    )
+  )
+  (symbol (lib_id "SamacSys_Parts:R7FA4M1AB3CFM#AA0") (at 101.6 63.5 0) (unit 1)
+    (in_bom yes) (on_board yes) (dnp no) (fields_autoplaced)
+    (property "Reference" "IC1" (at 161.29 56.5719 0)
+      (effects (font (size 1.27 1.27)))
+    )
+    (property "Value" "R7FA4M1AB3CFM#AA0" (at 161.29 59.1119 0)
+      (effects (font (size 1.27 1.27)))
+    )
+    (property "Footprint" "QFP50P1200X1200X170-64N" (at 151.13 43.18 0)
+      (effects (font (size 1.27 1.27)) (justify left) hide)
+    )
+    (property "Datasheet" "https://www.renesas.com/document/dst/renesas-ra4m1-group-datasheet?language=en&r=1054146" (at 151.13 45.72 0)
+      (effects (font (size 1.27 1.27)) (justify left) hide)
+    )
+    (property "Description" "The Renesas RA4M1 group of microcontrollers (MCUs) uses the high-performance Arm Cortex-M4 core and offers a segment LCD controller and a capacitive touch sensing unit input for intensive HMI designs. The RA4M1 MCU is built on a highly efficient low power process and is supported by an open and flexible ecosystem conceptthe Flexible Software Package (FSP), built on FreeRTOSand is expandable to use other RTOSes and middleware. The RA4M1 is suitable for applications where a large amount of capacitive touc" (at 151.13 48.26 0)
+      (effects (font (size 1.27 1.27)) (justify left) hide)
+    )
+    (property "Height" "1.7" (at 151.13 50.8 0)
+      (effects (font (size 1.27 1.27)) (justify left) hide)
+    )
+    (property "Manufacturer_Name" "Renesas Electronics" (at 151.13 53.34 0)
+      (effects (font (size 1.27 1.27)) (justify left) hide)
+    )
+    (property "Manufacturer_Part_Number" "R7FA4M1AB3CFM#AA0" (at 151.13 55.88 0)
+      (effects (font (size 1.27 1.27)) (justify left) hide)
+    )
+    (property "Mouser Part Number" "968-7FA4M1AB3CFM#AA0" (at 151.13 58.42 0)
+      (effects (font (size 1.27 1.27)) (justify left) hide)
+    )
+    (property "Mouser Price/Stock" "https://www.mouser.co.uk/ProductDetail/Renesas-Electronics/R7FA4M1AB3CFMAA0?qs=d0WKAl%252BL4KbrKuAsyurXHw%3D%3D" (at 151.13 60.96 0)
+      (effects (font (size 1.27 1.27)) (justify left) hide)
+    )
+    (property "Arrow Part Number" "" (at 151.13 63.5 0)
+      (effects (font (size 1.27 1.27)) (justify left) hide)
+    )
+    (property "Arrow Price/Stock" "" (at 151.13 66.04 0)
+      (effects (font (size 1.27 1.27)) (justify left) hide)
+    )
+    (pin "1")
+    (pin "10")
+    (pin "11")
+    (pin "12")
+    (pin "13")
+    (pin "14")
+    (pin "15")
+    (pin "16")
+    (pin "17")
+    (pin "18")
+    (pin "19")
+    (pin "2")
+    (pin "20")
+    (pin "21")
+    (pin "22")
+    (pin "23")
+    (pin "24")
+    (pin "25")
+    (pin "26")
+    (pin "27")
+    (pin "28")
+    (pin "29")
+    (pin "3")
+    (pin "30")
+    (pin "31")
+    (pin "32")
+    (pin "33")
+    (pin "34")
+    (pin "35")
+    (pin "36")
+    (pin "37")
+    (pin "38")
+    (pin "39")
+    (pin "4")
+    (pin "40")
+    (pin "41")
+    (pin "42")
+    (pin "43")
+    (pin "44")
+    (pin "45")
+    (pin "46")
+    (pin "47")
+    (pin "48")
+    (pin "49")
+    (pin "5")
+    (pin "50")
+    (pin "51")
+    (pin "52")
+    (pin "53")
+    (pin "54")
+    (pin "55")
+    (pin "56")
+    (pin "57")
+    (pin "58")
+    (pin "59")
+    (pin "6")
+    (pin "60")
+    (pin "61")
+    (pin "62")
+    (pin "63")
+    (pin "64")
+    (pin "7")
+    (pin "8")
+    (pin "9")
+    (instances
+      (project "main-ECU-board"
+        (path "/10edd9b6-c7a8-40f4-bfe3-c9724324d30f"
+          (reference "IC1") (unit 1)
+        )
+      )

Commit message: add parts
Parts:
- added D1: PRTR5V0U2X_215, digikey-footprints:TO-253-4, symbol dk_TVS-Diodes:PRTR5V0U2X_215
Changed lines of the file:
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@@
+    )
+  )
+  (symbol (lib_id "dk_TVS-Diodes:PRTR5V0U2X_215") (at 39.37 181.61 0) (unit 1)
+    (in_bom yes) (on_board yes) (dnp no) (fields_autoplaced)
+    (property "Reference" "D1" (at 39.37 170.18 0)
+      (effects (font (size 1.524 1.524)))
+    )
+    (property "Value" "PRTR5V0U2X_215" (at 39.37 172.72 0)
+      (effects (font (size 1.524 1.524)))
+    )
+    (property "Footprint" "digikey-footprints:TO-253-4" (at 44.45 176.53 0)
+      (effects (font (size 1.524 1.524)) (justify left) hide)
+    )
+    (property "Datasheet" "https://assets.nexperia.com/documents/data-sheet/PRTR5V0U2X.pdf" (at 44.45 173.99 0)
+      (effects (font (size 1.524 1.524)) (justify left) hide)
+    )
+    (property "Digi-Key_PN" "1727-3884-1-ND" (at 44.45 171.45 0)
+      (effects (font (size 1.524 1.524)) (justify left) hide)
+    )
+    (property "MPN" "PRTR5V0U2X,215" (at 44.45 168.91 0)
+      (effects (font (size 1.524 1.524)) (justify left) hide)
+    )
+    (property "Category" "Circuit Protection" (at 44.45 166.37 0)
+      (effects (font (size 1.524 1.524)) (justify left) hide)
+    )
+    (property "Family" "TVS - Diodes" (at 44.45 163.83 0)
+      (effects (font (size 1.524 1.524)) (justify left) hide)
+    )
+    (property "DK_Datasheet_Link" "https://assets.nexperia.com/documents/data-sheet/PRTR5V0U2X.pdf" (at 44.45 161.29 0)
+      (effects (font (size 1.524 1.524)) (justify left) hide)
+    )
+    (property "DK_Detail_Page" "/product-detail/en/nexperia-usa-inc/PRTR5V0U2X,215/1727-3884-1-ND/1589981" (at 44.45 158.75 0)
+      (effects (font (size 1.524 1.524)) (justify left) hide)
+    )
+    (property "Description" "TVS DIODE 5.5V SOT143B" (at 44.45 156.21 0)
+      (effects (font (size 1.524 1.524)) (justify left) hide)
+    )
+    (property "Manufacturer" "Nexperia USA Inc." (at 44.45 153.67 0)
+      (effects (font (size 1.524 1.524)) (justify left) hide)
+    )
+    (property "Status" "Active" (at 44.45 151.13 0)
+      (effects (font (size 1.524 1.524)) (justify left) hide)
+    )
+    (pin "1")
+    (pin "2")
+    (pin "3")
+    (pin "4")
+    (instances
+      (project "main-ECU-board"
+        (path "/10edd9b6-c7a8-40f4-bfe3-c9724324d30f"
+          (reference "D1") (unit 1)
+        )
+      )
     )
   )

Commit message: add part
Parts:
- added D2: CUHS20S30, SamacSys_Parts:CUHS20S40H3F, symbol Device:D_Schottky
Changed lines of the file:
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@@
+    )
+  )
+  (symbol (lib_id "Device:D_Schottky") (at 64.77 83.82 0) (unit 1)
+    (in_bom yes) (on_board yes) (dnp no) (fields_autoplaced)
+    (property "Reference" "D2" (at 64.4525 77.47 0)
+      (effects (font (size 1.27 1.27)))
+    )
+    (property "Value" "CUHS20S30" (at 64.4525 80.01 0)
+      (effects (font (size 1.27 1.27)))
+    )
+    (property "Footprint" "SamacSys_Parts:CUHS20S40H3F" (at 64.77 83.82 0)
+      (effects (font (size 1.27 1.27)) hide)
+    )
+    (property "Datasheet" "~" (at 64.77 83.82 0)
+      (effects (font (size 1.27 1.27)) hide)
+    )
+    (pin "1")
+    (pin "2")
+    (instances
+      (project "main-ECU-board"
+        (path "/10edd9b6-c7a8-40f4-bfe3-c9724324d30f"
+          (reference "D2") (unit 1)
+        )
+      )
     )
   )

Commit message: 発注先ラベル追加
Parts:
- D1, IC1: 発注先 (none) -> Digi-Key
- D2, J5: 発注先 (none) -> 秋月電子
Changed lines of the file:
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@@
+      (effects (font (size 1.27 1.27)) hide)
+    )
+    (property "発注先" "秋月電子" (at 76.2 139.7 0)
       (effects (font (size 1.27 1.27)) hide)
     )
@@
       (effects (font (size 1.27 1.27)) hide)
     )
+    (property "発注先" "秋月電子" (at 64.77 83.82 0)
+      (effects (font (size 1.27 1.27)) hide)
+    )
     (pin "1")
     (pin "2")
@@
       (effects (font (size 1.524 1.524)) (justify left) hide)
     )
+    (property "発注先" "Digi-Key" (at 39.37 181.61 0)
+      (effects (font (size 1.27 1.27)) hide)
+    )
     (pin "1")
     (pin "2")
@@
       (effects (font (size 1.27 1.27)) (justify left) hide)
     )
-    (pin "1")
+    (property "発注先" "Digi-Key" (at 101.6 63.5 0)
+      (effects (font (size 1.27 1.27)) hide)
+    )
+    (pin "1")

Commit message: usb周り修正
Parts:
- added C1: C, symbol Device:C
- added IC2: TCAN1042DQ1, SOIC127P600X175-8N, symbol SamacSys_Parts:TCAN1042DQ1
- added J6: Conn_01x02_Pin, symbol Connector:Conn_01x02_Pin
- added R1, R2, R3: R, symbol Device:R
Connections:
- net GND: now also J5.A1 (GND), J5.A12 (GND), J5.B1 (GND), J5.B12 (GND), C1.2, R1.2, R2.2, R3.2
- net VUSB: now reaches J5.A4 (VBUS), J5.A9 (VBUS), J5.B4 (VBUS), J5.B9 (VBUS)
- net VUSB: now also D1.4 (VCC)
- net CC1: now reaches J5.A5 (CC1)
- net CC1: now also R2.1
- net USB_D_P: now reaches J5.A6 (D+)
- net USB_D_P: now also D1.3 (I/O2)
- net USB_D_M: now reaches J5.A7 (D-)
- net USB_D_M: now also D1.2 (I/O1)
- net CC2: now reaches J5.B5 (CC2)
- net CC2: now also R3.1
- net SHIELD: now reaches J5.S1 (SHIELD)
- net SHIELD: now also D1.1 (GND), C1.1, R1.1
- no-connect marks 1 -> 11
Other:
- added sheet Power (power.kicad_sch)
- note added: "12V IN"
- note added: "CC RESISTERS"
- note added: "ESD PROTECTION"
- note added: "USB CONNECTOR"
- moved on the sheet: D1, D2, IC1, J5

Commit message: add Power, CAN Transceiver and modify
Parts:
- removed IC2: TCAN1042DQ1, SOIC127P600X175-8N, symbol SamacSys_Parts:TCAN1042DQ1
Connections:
- net USB_D_M: now also J5.B7 (D-)
- net USB_D_P: now also J5.B6 (D+)
- net VCC renamed +BATT
- net VUSB renamed VBUS
Other:
- added sheet CAN-Transceiver (CAN-transceiver.kicad_sch)
- moved on the sheet: IC1

Commit message: almost completed power, can, mcu
Parts:
- removed C1: C, symbol Device:C
- removed D1: PRTR5V0U2X_215, digikey-footprints:TO-253-4, symbol dk_TVS-Diodes:PRTR5V0U2X_215
- removed D2: CUHS20S30, SamacSys_Parts:CUHS20S40H3F, symbol Device:D_Schottky
- removed IC1: R7FA4M1AB3CFM#AA0, QFP50P1200X1200X170-64N, symbol SamacSys_Parts:R7FA4M1AB3CFM#AA0
- removed J1: Power, Connector_PinSocket_2.54mm:PinSocket_1x08_P2.54mm_Vertical, symbol Connector_Generic:Conn_01x08
- removed J2: Analog, Connector_PinSocket_2.54mm:PinSocket_1x06_P2.54mm_Vertical, symbol Connector_Generic:Conn_01x06
- removed J3: Digital/PWM, Connector_PinSocket_2.54mm:PinSocket_1x10_P2.54mm_Vertical, symbol Connector_Generic:Conn_01x10
- removed J4: Digital/PWM, Connector_PinSocket_2.54mm:PinSocket_1x08_P2.54mm_Vertical, symbol Connector_Generic:Conn_01x08
- removed J5: USB_C_Receptacle, SamacSys_Parts:5077CR-16-SMC2-BK-TR, symbol Connector:USB_C_Receptacle
- removed J6: Conn_01x02_Pin, symbol Connector:Conn_01x02_Pin
- removed R1, R2, R3: R, symbol Device:R
Connections:
- no-connect marks 11 -> 0
Other:
- added sheet Connectors (connectors.kicad_sch)
- added sheet MCU (MCU.kicad_sch)
- sheet Power ports: added +5V, +BATT, VBUS; removed none
- note removed: "12V IN"
- note removed: "CC RESISTERS"
- note removed: "ESD PROTECTION"
- note removed: "USB CONNECTOR"

Commit message: add, modify
Other:
- sheet CAN-Transceiver ports: added VCC; removed none
- sheet Connectors ports: added +12V, ACCEL_SENSOR_OUT2, ACCEL_SENSOR_OUT_1, AIR_SIG_M, AIR_SIG_P, BRAKE_SENSOR_OUT, PRECHARGE_SIG, READY_TO_DRIVE_SIG, READY_TO_DRIVE_SWITCH, VCC; removed none
- sheet MCU ports: added AREF, VCC; removed none
- sheet Power ports: added VCC; removed +5V
Changed lines of the file:
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@@
+    )
+  )
+  (global_label "AREF" (shape bidirectional) (at 190.5 99.06 0) (fields_autoplaced)
+    (effects (font (size 1.27 1.27)) (justify left))
+    (property "Intersheetrefs" "${INTERSHEET_REFS}" (at 199.1927 99.06 0)
+      (effects (font (size 1.27 1.27)) (justify left) hide)
     )
   )
@@
     )
   )
-  (sheet (at 50.8 25.4) (size 38.1 76.2) (fields_autoplaced)
+  (sheet (at 50.8 25.4) (size 50.8 76.2) (fields_autoplaced)
     (stroke (width 0.1524) (type solid))
     (fill (color 0 0 0 0.0000))
@@
       (effects (font (size 1.27 1.27)) (justify left top))
     )
-    (pin "VBUS" output (at 88.9 27.94 0)
-      (effects (font (size 1.27 1.27)) (justify right))
-    )
-    (pin "+BATT" output (at 88.9 30.48 0)
-      (effects (font (size 1.27 1.27)) (justify right))
-    )
-    (pin "USB_D_M" bidirectional (at 88.9 35.56 0)
-      (effects (font (size 1.27 1.27)) (justify right))
-    )
-    (pin "USB_D_P" bidirectional (at 88.9 33.02 0)
-      (effects (font (size 1.27 1.27)) (justify right))
-    )
-    (pin "2" bidirectional (at 88.9 93.98 0)
-      (effects (font (size 1.27 1.27)) (justify right))
-    )
-    (pin "TX{slash}1" bidirectional (at 88.9 96.52 0)
-      (effects (font (size 1.27 1.27)) (justify right))
-    )
-    (pin "RX{slash}0" bidirectional (at 88.9 99.06 0)
-      (effects (font (size 1.27 1.27)) (justify right))
-    )
-    (pin "SCL" bidirectional (at 88.9 55.88 0)
-      (effects (font (size 1.27 1.27)) (justify right))
-    )
-    (pin "SDA" bidirectional (at 88.9 58.42 0)
-      (effects (font (size 1.27 1.27)) (justify right))
-    )
-    (pin "CS{slash}10" bidirectional (at 88.9 73.66 0)
-      (effects (font (size 1.27 1.27)) (justify right))
-    )
-    (pin "MOSI{slash}11" bidirectional (at 88.9 71.12 0)
-      (effects (font (size 1.27 1.27)) (justify right))
-    )
-    (pin "MISO{slash}12" bidirectional (at 88.9 68.58 0)
-      (effects (font (size 1.27 1.27)) (justify right))
-    )
-    (pin "SCK{slash}13" bidirectional (at 88.9 66.04 0)
-      (effects (font (size 1.27 1.27)) (justify right))
-    )
-    (pin "9" bidirectional (at 88.9 76.2 0)
-      (effects (font (size 1.27 1.27)) (justify right))
-    )
-    (pin "8" bidirectional (at 88.9 78.74 0)
-      (effects (font (size 1.27 1.27)) (justify right))
-    )
-    (pin "3" bidirectional (at 88.9 91.44 0)
-      (effects (font (size 1.27 1.27)) (justify right))
-    )
-    (pin "5" bidirectional (at 88.9 86.36 0)
-      (effects (font (size 1.27 1.27)) (justify right))
-    )
-    (pin "4" bidirectional (at 88.9 88.9 0)
-      (effects (font (size 1.27 1.27)) (justify right))
-    )
-    (pin "6" bidirectional (at 88.9 83.82 0)
-      (effects (font (size 1.27 1.27)) (justify right))
-    )
-    (pin "7" bidirectional (at 88.9 81.28 0)
-      (effects (font (size 1.27 1.27)) (justify right))
-    )
-    (pin "AREF" bidirectional (at 88.9 60.96 0)
+    (pin "VBUS" output (at 101.6 27.94 0)
+      (effects (font (size 1.27 1.27)) (justify right))
+    )
+    (pin "+BATT" output (at 101.6 30.48 0)
+      (effects (font (size 1.27 1.27)) (justify right))
+    )
+    (pin "USB_D_M" bidirectional (at 101.6 35.56 0)
+      (effects (font (size 1.27 1.27)) (justify right))
+    )
+    (pin "USB_D_P" bidirectional (at 101.6 33.02 0)
+      (effects (font (size 1.27 1.27)) (justify right))
+    )
+    (pin "2" bidirectional (at 101.6 93.98 0)
+      (effects (font (size 1.27 1.27)) (justify right))
+    )
+    (pin "TX{slash}1" bidirectional (at 101.6 96.52 0)
+      (effects (font (size 1.27 1.27)) (justify right))
+    )
+    (pin "RX{slash}0" bidirectional (at 101.6 99.06 0)
+      (effects (font (size 1.27 1.27)) (justify right))
+    )
+    (pin "SCL" bidirectional (at 101.6 55.88 0)
+      (effects (font (size 1.27 1.27)) (justify right))
+    )
+    (pin "SDA" bidirectional (at 101.6 58.42 0)
+      (effects (font (size 1.27 1.27)) (justify right))
+    )
+    (pin "CS{slash}10" bidirectional (at 101.6 73.66 0)
+      (effects (font (size 1.27 1.27)) (justify right))
+    )
+    (pin "MOSI{slash}11" bidirectional (at 101.6 71.12 0)
+      (effects (font (size 1.27 1.27)) (justify right))
+    )
+    (pin "MISO{slash}12" bidirectional (at 101.6 68.58 0)
+      (effects (font (size 1.27 1.27)) (justify right))
+    )
+    (pin "SCK{slash}13" bidirectional (at 101.6 66.04 0)
+      (effects (font (size 1.27 1.27)) (justify right))
+    )
+    (pin "9" bidirectional (at 101.6 76.2 0)
+      (effects (font (size 1.27 1.27)) (justify right))
+    )
+    (pin "8" bidirectional (at 101.6 78.74 0)
+      (effects (font (size 1.27 1.27)) (justify right))
+    )
+    (pin "3" bidirectional (at 101.6 91.44 0)
+      (effects (font (size 1.27 1.27)) (justify right))
+    )
+    (pin "5" bidirectional (at 101.6 86.36 0)
+      (effects (font (size 1.27 1.27)) (justify right))
+    )
+    (pin "4" bidirectional (at 101.6 88.9 0)
+      (effects (font (size 1.27 1.27)) (justify right))
+    )
+    (pin "6" bidirectional (at 101.6 83.82 0)
+      (effects (font (size 1.27 1.27)) (justify right))
+    )
+    (pin "7" bidirectional (at 101.6 81.28 0)
+      (effects (font (size 1.27 1.27)) (justify right))
+    )
+    (pin "AREF" bidirectional (at 101.6 60.96 0)
       (effects (font (size 1.27 1.27)) (justify right))
     )
@@
     )
     (pin "A2" bidirectional (at 50.8 91.44 180)
+      (effects (font (size 1.27 1.27)) (justify left))
+    )
+    (pin "VCC" input (at 50.8 27.94 180)
+      (effects (font (size 1.27 1.27)) (justify left))
+    )
+    (pin "BRAKE_SENSOR_OUT" output (at 101.6 43.18 0)
+      (effects (font (size 1.27 1.27)) (justify right))
+    )
+    (pin "ACCEL_SENSOR_OUT_1" output (at 101.6 38.1 0)
+      (effects (font (size 1.27 1.27)) (justify right))
+    )
+    (pin "ACCEL_SENSOR_OUT2" output (at 101.6 40.64 0)
+      (effects (font (size 1.27 1.27)) (justify right))
+    )
+    (pin "READY_TO_DRIVE_SIG" input (at 50.8 33.02 180)
+      (effects (font (size 1.27 1.27)) (justify left))
+    )
+    (pin "+12V" input (at 50.8 30.48 180)
+      (effects (font (size 1.27 1.27)) (justify left))
+    )
+    (pin "READY_TO_DRIVE_SWITCH" output (at 101.6 45.72 0)
+      (effects (font (size 1.27 1.27)) (justify right))
+    )
+    (pin "AIR_SIG_M" input (at 50.8 40.64 180)
+      (effects (font (size 1.27 1.27)) (justify left))
+    )
+    (pin "AIR_SIG_P" input (at 50.8 38.1 180)
+      (effects (font (size 1.27 1.27)) (justify left))
+    )
+    (pin "PRECHARGE_SIG" input (at 50.8 35.56 180)
       (effects (font (size 1.27 1.27)) (justify left))
     )
@@
       (effects (font (size 1.27 1.27)) (justify left))
     )
-    (pin "+5V" output (at 165.1 27.94 0)
+    (pin "VCC" output (at 165.1 27.94 0)
       (effects (font (size 1.27 1.27)) (justify right))
     )
@@
     )
   )
-  (sheet (at 228.6 114.3) (size 25.4 12.7) (fields_autoplaced)
+  (sheet (at 241.3 114.3) (size 25.4 12.7) (fields_autoplaced)
     (stroke (width 0.1524) (type solid))
     (fill (color 0 0 0 0.0000))
-    (property "Sheetname" "CAN-Transceiver" (at 228.6 113.5884 0)
+    (property "Sheetname" "CAN-Transceiver" (at 241.3 113.5884 0)
       (effects (font (size 1.27 1.27)) (justify left bottom))
     )
-    (property "Sheetfile" "CAN-transceiver.kicad_sch" (at 228.6 127.5846 0)
+    (property "Sheetfile" "CAN-transceiver.kicad_sch" (at 241.3 127.5846 0)
       (effects (font (size 1.27 1.27)) (justify left top))
     )
-    (pin "RXD" output (at 228.6 116.84 180)
-      (effects (font (size 1.27 1.27)) (justify left))
-    )
-    (pin "TXD" input (at 228.6 124.46 180)
-      (effects (font (size 1.27 1.27)) (justify left))
-    )
-    (pin "CANH" bidirectional (at 254 116.84 0)
-      (effects (font (size 1.27 1.27)) (justify right))
-    )
-    (pin "CANL" bidirectional (at 254 124.46 0)
-      (effects (font (size 1.27 1.27)) (justify right))
+    (pin "RXD" output (at 241.3 121.92 180)
+      (effects (font (size 1.27 1.27)) (justify left))
+    )
+    (pin "TXD" input (at 241.3 124.46 180)
+      (effects (font (size 1.27 1.27)) (justify left))
+    )
+    (pin "CANH" bidirectional (at 266.7 116.84 0)
+      (effects (font (size 1.27 1.27)) (justify right))
+    )
+    (pin "CANL" bidirectional (at 266.7 124.46 0)
+      (effects (font (size 1.27 1.27)) (justify right))
+    )
+    (pin "VCC" input (at 241.3 116.84 180)
+      (effects (font (size 1.27 1.27)) (justify left))
     )
     (instances
@@
       (effects (font (size 1.27 1.27)) (justify left))
     )
-    (instances
+    (pin "VCC" input (at 127 54.61 180)
+      (effects (font (size 1.27 1.27)) (justify left))
+    )
+    (pin "AREF" bidirectional (at 190.5 99.06 0)
+      (effects (font (size 1.27 1.27)) (justify right))
+    )
+    (instances
