File: main-ECU-board.kicad_sch (KiCad schematic)
At the start: 0 parts

Commit message: add circuit, modify
add load switch, add connector, connect blocks, etc...
Other:
- added sheet Load-Switch (load-switch.kicad_sch)
- sheet Connectors ports: added ACCEL_SENSOR_OUT_2, AIR_M_OUT, AIR_P_OUT, CANH, CANL, ECO_SPORTS_SELECT_SWITCH, PRECHARGE_OUT, READY_TO_DRIVE_OUT, SHUTDOWN_CIRCUIT; removed +12V, ACCEL_SENSOR_OUT2, AIR_SIG_M, AIR_SIG_P, PRECHARGE_SIG, READY_TO_DRIVE_SIG
- note added: "ARDUINO HEADER"
- note added: "ARDUINO PIN"

Commit message: modify, add module
信号の向きの修正、レベルシフター追加、ポート追加
Other:
- added sheet Level-Shift (level-shift.kicad_sch)
- sheet MCU ports: added P408_IRQ07_GPT5_B, P409_IRQ06_GPT5_A, P410_IRQ05_GPT6_B, P411_IRQ04_GPT6_A; removed none

Commit message: modify, add parts
Other:
- sheet Connectors ports: added OPT_I/O_1, OPT_I/O_2, OPT_I/O_3, OPT_I/O_4, SWCLK, SWDIO, UART_RX, UART_TX; removed none
- sheet Load-Switch ports: added AIR_M_OUT, AIR_M_SIG, AIR_P_OUT, AIR_P_SIG, PRECHARGE_OUT, PRECHARGE_SIG, READY_TO_DRIVE_OUT, READY_TO_DRIVE_SIG; removed AIR_M_OUT_12V, AIR_M_SIG_5V, AIR_P_OUT_12V, AIR_P_SIG_5V, PRECHARGE_OUT_12V, PRECHARGE_SIG_5V, READY_TO_DRIVE_OUT_12V, READY_TO_DRIVE_SIG_5V
- sheet MCU ports: added P002_AN02_AMP0O, P003_AN03_AMP1O, P004_AN04_AMP2O, P108_SWDIO, P113_GPT2_A, P204_GPT4_B, P205_GPT4_A, P300_SWCLK, P501_SCI1_TXD, P502_SCI1_RXD; removed P002_AN02_AMPO
