File: main-ECU-board.kicad_sch (KiCad schematic)
At the start: 0 parts

Commit message: Arduino header削除、ピンアサイン修正
ハイサイドスイッチ信号、UARTなど
Arduino互換ピンはXHで出す
回路図一部修正
パターン削除、部品配置
Other:
- sheet Connectors ports: added ANALOG_I/O_1, RX, TX; removed +3V3, +5V, 2, 3, 4, 5, 6, 7, 8, 9, A0, A1, A2, A3, A4, A5, AREF, IOREF, NC, RX/0, TX/1, VIN
- sheet MCU ports: added none; removed AREF, P201_MD
- note removed: "ARDUINO HEADER"

Commit message: シャットダウン検知をMOSFETから分圧回路に変更、リファレンス指定子"IC?"を"U?"に変更
Other:
- sheet Level-Shift ports: added none; removed VCC
