File: CAN-transceiver.kicad_sch (KiCad schematic)
At the start: 8 parts, among them IC2 TCAN1042DQ1

Commit message: modify symbol number, constant
Parts:
- C11: renamed from C2; value C -> 0.1u
- renumbered C4 to C12, D5 to D4, R5 to R10, R6 to R11, R7 to R8, R8 to R9
Changed lines of the file:
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@@
   (symbol (lib_id "Device:R") (at 152.4 82.55 0) (unit 1)
     (in_bom yes) (on_board yes) (dnp no) (fields_autoplaced)
-    (property "Reference" "R8" (at 154.94 81.28 0)
+    (property "Reference" "R9" (at 154.94 81.28 0)
       (effects (font (size 1.27 1.27)) (justify left))
     )
@@
       (project "main-ECU-board"
         (path "/10edd9b6-c7a8-40f4-bfe3-c9724324d30f/a6f2c8d0-7153-435f-8690-872c30ac6e56"
-          (reference "R8") (unit 1)
+          (reference "R9") (unit 1)
         )
       )
@@
   (symbol (lib_id "power:GND") (at 182.88 82.55 90) (unit 1)
     (in_bom yes) (on_board yes) (dnp no) (fields_autoplaced)
-    (property "Reference" "#PWR022" (at 189.23 82.55 0)
+    (property "Reference" "#PWR035" (at 189.23 82.55 0)
       (effects (font (size 1.27 1.27)) hide)
     )
@@
       (project "main-ECU-board"
         (path "/10edd9b6-c7a8-40f4-bfe3-c9724324d30f/a6f2c8d0-7153-435f-8690-872c30ac6e56"
-          (reference "#PWR022") (unit 1)
+          (reference "#PWR035") (unit 1)
         )
       )
@@
   (symbol (lib_id "Device:C") (at 101.6 57.15 0) (unit 1)
     (in_bom yes) (on_board yes) (dnp no) (fields_autoplaced)
-    (property "Reference" "C2" (at 105.41 55.88 0)
-      (effects (font (size 1.27 1.27)) (justify left))
-    )
-    (property "Value" "C" (at 105.41 58.42 0)
+    (property "Reference" "C11" (at 105.41 55.88 0)
+      (effects (font (size 1.27 1.27)) (justify left))
+    )
+    (property "Value" "0.1u" (at 105.41 58.42 0)
       (effects (font (size 1.27 1.27)) (justify left))
     )
@@
       (project "main-ECU-board"
         (path "/10edd9b6-c7a8-40f4-bfe3-c9724324d30f/a6f2c8d0-7153-435f-8690-872c30ac6e56"
-          (reference "C2") (unit 1)
+          (reference "C11") (unit 1)
         )
       )
@@
   (symbol (lib_id "power:GND") (at 134.62 101.6 0) (unit 1)
     (in_bom yes) (on_board yes) (dnp no) (fields_autoplaced)
-    (property "Reference" "#PWR021" (at 134.62 107.95 0)
+    (property "Reference" "#PWR034" (at 134.62 107.95 0)
       (effects (font (size 1.27 1.27)) hide)
     )
@@
       (project "main-ECU-board"
         (path "/10edd9b6-c7a8-40f4-bfe3-c9724324d30f/a6f2c8d0-7153-435f-8690-872c30ac6e56"
-          (reference "#PWR021") (unit 1)
+          (reference "#PWR034") (unit 1)
         )
       )
@@
   (symbol (lib_id "power:GND") (at 99.06 81.28 270) (unit 1)
     (in_bom yes) (on_board yes) (dnp no) (fields_autoplaced)
-    (property "Reference" "#PWR017" (at 92.71 81.28 0)
+    (property "Reference" "#PWR032" (at 92.71 81.28 0)
       (effects (font (size 1.27 1.27)) hide)
     )
@@
       (project "main-ECU-board"
         (path "/10edd9b6-c7a8-40f4-bfe3-c9724324d30f/a6f2c8d0-7153-435f-8690-872c30ac6e56"
-          (reference "#PWR017") (unit 1)
+          (reference "#PWR032") (unit 1)
         )
       )
@@
   (symbol (lib_id "Device:C") (at 176.53 82.55 90) (unit 1)
     (in_bom yes) (on_board yes) (dnp no) (fields_autoplaced)
-    (property "Reference" "C4" (at 176.53 74.93 90)
+    (property "Reference" "C12" (at 176.53 74.93 90)
       (effects (font (size 1.27 1.27)))
     )
@@
       (project "main-ECU-board"
         (path "/10edd9b6-c7a8-40f4-bfe3-c9724324d30f/a6f2c8d0-7153-435f-8690-872c30ac6e56"
-          (reference "C4") (unit 1)
+          (reference "C12") (unit 1)
         )
       )
@@
   (symbol (lib_id "Device:R") (at 165.1 88.9 0) (unit 1)
     (in_bom yes) (on_board yes) (dnp no) (fields_autoplaced)
-    (property "Reference" "R6" (at 167.64 87.63 0)
+    (property "Reference" "R11" (at 167.64 87.63 0)
       (effects (font (size 1.27 1.27)) (justify left))
     )
@@
       (project "main-ECU-board"
         (path "/10edd9b6-c7a8-40f4-bfe3-c9724324d30f/a6f2c8d0-7153-435f-8690-872c30ac6e56"
-          (reference "R6") (unit 1)
+          (reference "R11") (unit 1)
         )
       )
@@
   (symbol (lib_id "power:GND") (at 205.74 82.55 90) (unit 1)
     (in_bom yes) (on_board yes) (dnp no) (fields_autoplaced)
-    (property "Reference" "#PWR023" (at 212.09 82.55 0)
+    (property "Reference" "#PWR036" (at 212.09 82.55 0)
       (effects (font (size 1.27 1.27)) hide)
     )
@@
       (project "main-ECU-board"
         (path "/10edd9b6-c7a8-40f4-bfe3-c9724324d30f/a6f2c8d0-7153-435f-8690-872c30ac6e56"
-          (reference "#PWR023") (unit 1)
+          (reference "#PWR036") (unit 1)
         )
       )
@@
   (symbol (lib_id "Device:R") (at 134.62 95.25 0) (unit 1)
     (in_bom yes) (on_board yes) (dnp no) (fields_autoplaced)
-    (property "Reference" "R7" (at 137.16 93.98 0)
+    (property "Reference" "R8" (at 137.16 93.98 0)
       (effects (font (size 1.27 1.27)) (justify left))
     )
@@
       (project "main-ECU-board"
         (path "/10edd9b6-c7a8-40f4-bfe3-c9724324d30f/a6f2c8d0-7153-435f-8690-872c30ac6e56"
-          (reference "R7") (unit 1)
+          (reference "R8") (unit 1)
         )
       )
@@
         )
         (path "/10edd9b6-c7a8-40f4-bfe3-c9724324d30f/a6f2c8d0-7153-435f-8690-872c30ac6e56"
-          (reference "IC2") (unit 1)
+          (reference "IC1") (unit 1)
         )
       )
@@
   (symbol (lib_id "Power_Protection:NUP2105L") (at 198.12 82.55 90) (unit 1)
     (in_bom yes) (on_board yes) (dnp no) (fields_autoplaced)
-    (property "Reference" "D5" (at 198.12 73.66 90)
+    (property "Reference" "D4" (at 198.12 73.66 90)
       (effects (font (size 1.27 1.27)))
     )
@@
       (project "main-ECU-board"
         (path "/10edd9b6-c7a8-40f4-bfe3-c9724324d30f/a6f2c8d0-7153-435f-8690-872c30ac6e56"
-          (reference "D5") (unit 1)
+          (reference "D4") (unit 1)
         )
       )
@@
   (symbol (lib_id "power:GND") (at 101.6 63.5 0) (unit 1)
     (in_bom yes) (on_board yes) (dnp no) (fields_autoplaced)
-    (property "Reference" "#PWR019" (at 101.6 69.85 0)
+    (property "Reference" "#PWR033" (at 101.6 69.85 0)
       (effects (font (size 1.27 1.27)) hide)
     )
@@
       (project "main-ECU-board"
         (path "/10edd9b6-c7a8-40f4-bfe3-c9724324d30f/a6f2c8d0-7153-435f-8690-872c30ac6e56"
-          (reference "#PWR019") (unit 1)
+          (reference "#PWR033") (unit 1)
         )
       )
@@
   (symbol (lib_id "Device:R") (at 165.1 76.2 0) (unit 1)
     (in_bom yes) (on_board yes) (dnp no) (fields_autoplaced)
-    (property "Reference" "R5" (at 167.64 74.93 0)
+    (property "Reference" "R10" (at 167.64 74.93 0)
       (effects (font (size 1.27 1.27)) (justify left))
     )
@@
       (project "main-ECU-board"
         (path "/10edd9b6-c7a8-40f4-bfe3-c9724324d30f/a6f2c8d0-7153-435f-8690-872c30ac6e56"
-          (reference "R5") (unit 1)
-        )
-      )
+          (reference "R10") (unit 1)
+        )
+      )
