File: CAN-transceiver.kicad_sch (KiCad schematic)
At the start: 8 parts, among them IC2 TCAN1042DQ1

Commit message: decide constant
Parts:
- R10, R11: value R -> 60
- R9: value R -> 1k
Other:
- note added: "IF END-NODE AND NORMAL TERMINATION, NOT 1k OHM, BUT 120 OHM."
Changed lines of the file:
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@@
     (effects (font (size 2.54 2.54)) (justify left bottom))
+  )
+  (text "IF END-NODE AND\nNORMAL TERMINATION,\nNOT 1k OHM, BUT 120 OHM."
+    (at 143.51 102.87 0)
+    (effects (font (size 1.27 1.27)) (justify left bottom))
   )
   (text "TERMINATION" (at 146.05 68.58 0)
@@
       (effects (font (size 1.27 1.27)) (justify left))
     )
-    (property "Value" "R" (at 154.94 83.82 0)
+    (property "Value" "1k" (at 154.94 83.82 0)
       (effects (font (size 1.27 1.27)) (justify left))
     )
@@
       (effects (font (size 1.27 1.27)) (justify left))
     )
-    (property "Value" "R" (at 167.64 90.17 0)
+    (property "Value" "60" (at 167.64 90.17 0)
       (effects (font (size 1.27 1.27)) (justify left))
     )
@@
       (effects (font (size 1.27 1.27)) (justify left))
     )
-    (property "Value" "R" (at 167.64 77.47 0)
-      (effects (font (size 1.27 1.27)) (justify left))
-    )
+    (property "Value" "60" (at 167.64 77.47 0)
+      (effects (font (size 1.27 1.27)) (justify left))
+    )

Commit message: decide constant
Parts:
- C12: value C -> 0.1u
- R8: value R -> 3k
Changed lines of the file:
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@@
       (effects (font (size 1.27 1.27)))
     )
-    (property "Value" "C" (at 176.53 77.47 90)
+    (property "Value" "0.1u" (at 176.53 77.47 90)
       (effects (font (size 1.27 1.27)))
     )
@@
       (effects (font (size 1.27 1.27)) (justify left))
     )
-    (property "Value" "R" (at 137.16 96.52 0)
+    (property "Value" "3k" (at 137.16 96.52 0)
       (effects (font (size 1.27 1.27)) (justify left))
     )

Commit message: modify constant
Parts:
- R8: value 3k -> 15k
Changed lines of the file:
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@@
       (effects (font (size 1.27 1.27)) (justify left))
     )
-    (property "Value" "3k" (at 137.16 96.52 0)
+    (property "Value" "15k" (at 137.16 96.52 0)
       (effects (font (size 1.27 1.27)) (justify left))
     )

Commit message: add and modify 発注先 and footprint
Parts:
- C11, C12: footprint (none) -> Capacitor_SMD:C_0603_1608Metric; 発注先 (none) -> Digi-Key
- D4: 発注先 (none) -> MOUSER
- R10, R11: 発注先 (none) -> Digi-Key
- R8, R9: footprint (none) -> Resistor_SMD:R_0603_1608Metric; 発注先 (none) -> Digi-Key
Changed lines of the file:
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@@
       (effects (font (size 1.27 1.27)) (justify left))
     )
-    (property "Footprint" "" (at 150.622 82.55 90)
+    (property "Footprint" "Resistor_SMD:R_0603_1608Metric" (at 150.622 82.55 90)
       (effects (font (size 1.27 1.27)) hide)
     )
@@
     )
     (property "在庫" "" (at 152.4 82.55 0)
+      (effects (font (size 1.27 1.27)) hide)
+    )
+    (property "発注先" "Digi-Key" (at 152.4 82.55 0)
       (effects (font (size 1.27 1.27)) hide)
     )
@@
       (effects (font (size 1.27 1.27)) (justify left))
     )
-    (property "Footprint" "" (at 102.5652 60.96 0)
+    (property "Footprint" "Capacitor_SMD:C_0603_1608Metric" (at 102.5652 60.96 0)
       (effects (font (size 1.27 1.27)) hide)
     )
@@
     )
     (property "在庫" "" (at 101.6 57.15 0)
+      (effects (font (size 1.27 1.27)) hide)
+    )
+    (property "発注先" "Digi-Key" (at 101.6 57.15 0)
       (effects (font (size 1.27 1.27)) hide)
     )
@@
       (effects (font (size 1.27 1.27)))
     )
-    (property "Footprint" "" (at 180.34 81.5848 0)
+    (property "Footprint" "Capacitor_SMD:C_0603_1608Metric" (at 180.34 81.5848 0)
       (effects (font (size 1.27 1.27)) hide)
     )
@@
       (effects (font (size 1.27 1.27)) hide)
     )
+    (property "発注先" "Digi-Key" (at 176.53 82.55 0)
+      (effects (font (size 1.27 1.27)) hide)
+    )
     (pin "1")
     (pin "2")
@@
     )
     (property "在庫" "" (at 165.1 88.9 0)
+      (effects (font (size 1.27 1.27)) hide)
+    )
+    (property "発注先" "Digi-Key" (at 165.1 88.9 0)
       (effects (font (size 1.27 1.27)) hide)
     )
@@
       (effects (font (size 1.27 1.27)) (justify left))
     )
-    (property "Footprint" "" (at 132.842 95.25 90)
+    (property "Footprint" "Resistor_SMD:R_0603_1608Metric" (at 132.842 95.25 90)
       (effects (font (size 1.27 1.27)) hide)
     )
@@
     )
     (property "在庫" "" (at 134.62 95.25 0)
+      (effects (font (size 1.27 1.27)) hide)
+    )
+    (property "発注先" "Digi-Key" (at 134.62 95.25 0)
       (effects (font (size 1.27 1.27)) hide)
     )
@@
       (effects (font (size 1.27 1.27)) hide)
     )
+    (property "発注先" "MOUSER" (at 198.12 82.55 0)
+      (effects (font (size 1.27 1.27)) hide)
+    )
     (pin "3")
     (pin "1")
@@
       (effects (font (size 1.27 1.27)) hide)
     )
+    (property "発注先" "Digi-Key" (at 165.1 76.2 0)
+      (effects (font (size 1.27 1.27)) hide)
+    )

Commit message: modify constant, footprint
Parts:
- R10, R11: value 60 -> 60.4; footprint (none) -> Resistor_SMD:R_0603_1608Metric
Changed lines of the file:
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@@
       (effects (font (size 1.27 1.27)) (justify left))
     )
-    (property "Value" "60" (at 167.64 90.17 0)
-      (effects (font (size 1.27 1.27)) (justify left))
-    )
-    (property "Footprint" "" (at 163.322 88.9 90)
+    (property "Value" "60.4" (at 167.64 90.17 0)
+      (effects (font (size 1.27 1.27)) (justify left))
+    )
+    (property "Footprint" "Resistor_SMD:R_0603_1608Metric" (at 163.322 88.9 90)
       (effects (font (size 1.27 1.27)) hide)
     )
@@
       (effects (font (size 1.27 1.27)) (justify left))
     )
-    (property "Value" "60" (at 167.64 77.47 0)
-      (effects (font (size 1.27 1.27)) (justify left))
-    )
-    (property "Footprint" "" (at 163.322 76.2 90)
-      (effects (font (size 1.27 1.27)) hide)
-    )
+    (property "Value" "60.4" (at 167.64 77.47 0)
+      (effects (font (size 1.27 1.27)) (justify left))
+    )
+    (property "Footprint" "Resistor_SMD:R_0603_1608Metric" (at 163.322 76.2 90)
+      (effects (font (size 1.27 1.27)) hide)
+    )
