File: MCU.kicad_sch (KiCad schematic)
At the start: 31 parts, among them IC1 R7FA4M1AB3CFM#AA0, J7 Conn_01x02_Pin, SW1 SW_MEC_5E, Y1 ABM8W-12.0000MHZ-8-K1Z-T3

Commit message: modify, add I/O port
Connections:
- net +5V: no longer IC1.21 (VCC_USB_LDO)
- net VCC: now also IC1.21 (VCC_USB_LDO)
- net P411_IRQ04_GPT6_A: now reaches IC1.12 (P411)
- net P410_IRQ05_GPT6_B: now reaches IC1.13 (P410)
- net P409_IRQ06_GPT5_A: now reaches IC1.14 (P409)
- net P408_IRQ07_GPT5_B: now reaches IC1.15 (P408)
- no-connect marks 17 -> 13
Other:
- moved on the sheet: C16, C17, C18, C19, C20, FB1, FB2, IC1, R15, R17, R21, R22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

Commit message: modify, add port
add optional port, debug interface
Connections:
- net P205_GPT4_A: now reaches IC1.23 (P205)
- net P113_GPT2_A: now reaches IC1.38 (P113)
- net P004_AN04_AMP2O: now reaches IC1.60 (P004)
- net P003_AN03_AMP1O: now reaches IC1.61 (P003)
- net P002_AN02_AMPO renamed P002_AN02_AMP0O
- net P204 renamed P204_GPT4_B
- no-connect marks 13 -> 9
Other:
- moved on the sheet: C13, C14, C15, D6, D7, D8, J7, R16, R18, R24, R25, R26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

Commit message: add sheet name, explain
Other:
- note added: "MCU"
Changed lines of the file:
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@@
     (effects (font (size 1.27 1.27)) (justify left bottom))
+  )
+  (text "MCU" (at 190.5 177.8 0)
+    (effects (font (size 5.08 5.08)) (justify left bottom))
   )
   (text "RESET PUSHBUTTON" (at 191.77 30.48 0)

Commit message: modify symbol number, constant
Parts:
- C20: renamed from C13; value C -> 0.1u
- C21: renamed from C14; value C -> 0.1u
- C22: renamed from C15; value C -> 0.1u
- renumbered C22 to C13, C21 to C14, C18 to C15, C20 to C17, C17 to C18, D8 to D5, D7 to D6, D6 to D7, FB2 to FB1, FB1 to FB2, J7 to J1, R15 to R12, R21 to R13, R22 to R14, R23 to R15, R17 to R16, R19 to R17, R20 to R18, R26 to R19, R18 to R20, R25 to R21, R24 to R22, R16 to R23
