File: MCU.kicad_sch (KiCad schematic)
At the start: 31 parts, among them IC1 R7FA4M1AB3CFM#AA0, J1 Conn_01x02_Pin, SW1 SW_MEC_5E, Y1 ABM8W-12.0000MHZ-8-K1Z-T3

Commit message: decide constant
Parts:
- C15: value C -> 4.7u
- C16, C17: value C -> 0.1u
- C18: value C -> 1u
- D5, D6, D7: value LED -> LED_G
- R12, R13, R14, R15: value R -> 5.1k
- R16, R20, R23: value R -> 15k
- R19, R21, R22: value R -> 300
Changed lines of the file:
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@@
       (effects (font (size 1.27 1.27)) (justify right))
     )
-    (property "Value" "R" (at 91.44 147.32 0)
+    (property "Value" "5.1k" (at 91.44 147.32 0)
       (effects (font (size 1.27 1.27)) (justify right))
     )
@@
       (effects (font (size 1.27 1.27)) (justify left))
     )
-    (property "Value" "R" (at 218.44 96.52 0)
+    (property "Value" "300" (at 218.44 96.52 0)
       (effects (font (size 1.27 1.27)) (justify left))
     )
@@
       (effects (font (size 1.27 1.27)) (justify right))
     )
-    (property "Value" "R" (at 91.44 172.72 0)
+    (property "Value" "5.1k" (at 91.44 172.72 0)
       (effects (font (size 1.27 1.27)) (justify right))
     )
@@
       (effects (font (size 1.27 1.27)) (justify left))
     )
-    (property "Value" "R" (at 205.74 96.52 0)
+    (property "Value" "300" (at 205.74 96.52 0)
       (effects (font (size 1.27 1.27)) (justify left))
     )
@@
       (effects (font (size 1.27 1.27)) (justify right))
     )
-    (property "Value" "LED" (at 219.71 85.4075 90)
+    (property "Value" "LED_G" (at 219.71 85.4075 90)
       (effects (font (size 1.27 1.27)) (justify right))
     )
@@
       (effects (font (size 1.27 1.27)) (justify left))
     )
-    (property "Value" "R" (at 243.84 96.52 0)
+    (property "Value" "300" (at 243.84 96.52 0)
       (effects (font (size 1.27 1.27)) (justify left))
     )
@@
       (effects (font (size 1.27 1.27)))
     )
-    (property "Value" "R" (at 68.58 21.59 90)
+    (property "Value" "5.1k" (at 68.58 21.59 90)
       (effects (font (size 1.27 1.27)))
     )
@@
       (effects (font (size 1.27 1.27)) (justify right))
     )
-    (property "Value" "R" (at 91.44 160.02 0)
+    (property "Value" "5.1k" (at 91.44 160.02 0)
       (effects (font (size 1.27 1.27)) (justify right))
     )
@@
       (effects (font (size 1.27 1.27)) (justify left))
     )
-    (property "Value" "R" (at 218.44 39.37 0)
+    (property "Value" "15k" (at 218.44 39.37 0)
       (effects (font (size 1.27 1.27)) (justify left))
     )
@@
       (effects (font (size 1.27 1.27)) (justify left))
     )
-    (property "Value" "C" (at 85.09 45.72 0)
+    (property "Value" "0.1u" (at 85.09 45.72 0)
       (effects (font (size 1.27 1.27)) (justify left))
     )
@@
       (effects (font (size 1.27 1.27)) (justify left))
     )
-    (property "Value" "R" (at 134.62 185.42 0)
+    (property "Value" "15k" (at 134.62 185.42 0)
       (effects (font (size 1.27 1.27)) (justify left))
     )
@@
       (effects (font (size 1.27 1.27)) (justify left))
     )
-    (property "Value" "C" (at 97.79 45.72 0)
+    (property "Value" "1u" (at 97.79 45.72 0)
       (effects (font (size 1.27 1.27)) (justify left))
     )
@@
       (effects (font (size 1.27 1.27)) (justify right))
     )
-    (property "Value" "LED" (at 207.01 85.4075 90)
+    (property "Value" "LED_G" (at 207.01 85.4075 90)
       (effects (font (size 1.27 1.27)) (justify right))
     )
@@
       (effects (font (size 1.27 1.27)) (justify right))
     )
-    (property "Value" "LED" (at 245.11 85.4075 90)
+    (property "Value" "LED_G" (at 245.11 85.4075 90)
       (effects (font (size 1.27 1.27)) (justify right))
     )
@@
       (effects (font (size 1.27 1.27)) (justify left))
     )
-    (property "Value" "R" (at 262.89 39.37 0)
+    (property "Value" "15k" (at 262.89 39.37 0)
       (effects (font (size 1.27 1.27)) (justify left))
     )
@@
       (effects (font (size 1.27 1.27)))
     )
-    (property "Value" "C" (at 88.9 99.06 90)
+    (property "Value" "0.1u" (at 88.9 99.06 90)
       (effects (font (size 1.27 1.27)))
     )
@@
       (effects (font (size 1.27 1.27)))
     )
-    (property "Value" "C" (at 69.85 101.6 90)
-      (effects (font (size 1.27 1.27)))
-    )
+    (property "Value" "4.7u" (at 69.85 101.6 90)
+      (effects (font (size 1.27 1.27)))
+    )

Commit message: add and modify 発注先 and footprint
Parts:
- C13, C14, C15, C19, FB1, FB2, R12, R13, R14, R15, R17, R18, Y1: 発注先 (none) -> Digi-Key
- C16, C17, C18, C20, C21, C22: footprint (none) -> Capacitor_SMD:C_0603_1608Metric; 発注先 (none) -> Digi-Key
- D5, D6, D7: footprint (none) -> LED_SMD:LED_0603_1608Metric; 発注先 (none) -> Digi-Key
- R16, R19, R20, R21, R22, R23: footprint (none) -> Resistor_SMD:R_0603_1608Metric; 発注先 (none) -> Digi-Key
- SW1: 発注先 秋月電子 -> Digi-Key
Changed lines of the file:
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@@
+      (effects (font (size 1.27 1.27)) hide)
+    )
+    (property "発注先" "Digi-Key" (at 88.9 146.05 0)
       (effects (font (size 1.27 1.27)) hide)
     )
@@
       (effects (font (size 1.27 1.27)) hide)
     )
-    (property "発注先" "秋月電子" (at 205.74 46.99 0)
+    (property "発注先" "Digi-Key" (at 205.74 46.99 0)
       (effects (font (size 1.27 1.27)) hide)
     )
@@
       (effects (font (size 1.27 1.27)) (justify left))
     )
-    (property "Footprint" "" (at 153.3652 35.56 0)
+    (property "Footprint" "Capacitor_SMD:C_0603_1608Metric" (at 153.3652 35.56 0)
       (effects (font (size 1.27 1.27)) hide)
     )
@@
       (effects (font (size 1.27 1.27)) hide)
     )
+    (property "発注先" "Digi-Key" (at 152.4 31.75 0)
+      (effects (font (size 1.27 1.27)) hide)
+    )
     (pin "1")
     (pin "2")
@@
       (effects (font (size 1.27 1.27)) (justify left))
     )
-    (property "Footprint" "" (at 214.122 95.25 90)
+    (property "Footprint" "Resistor_SMD:R_0603_1608Metric" (at 214.122 95.25 90)
       (effects (font (size 1.27 1.27)) hide)
     )
@@
       (effects (font (size 1.27 1.27)) hide)
     )
+    (property "発注先" "Digi-Key" (at 215.9 95.25 0)
+      (effects (font (size 1.27 1.27)) hide)
+    )
     (pin "1")
     (pin "2")
@@
     )
     (property "Datasheet" "~" (at 88.9 171.45 0)
+      (effects (font (size 1.27 1.27)) hide)
+    )
+    (property "発注先" "Digi-Key" (at 88.9 171.45 0)
       (effects (font (size 1.27 1.27)) hide)
     )
@@
       (effects (font (size 1.27 1.27)) hide)
     )
+    (property "発注先" "Digi-Key" (at 87.63 25.4 0)
+      (effects (font (size 1.27 1.27)) hide)
+    )
     (pin "1")
     (pin "2")
@@
       (effects (font (size 1.27 1.27)) (justify left))
     )
-    (property "Footprint" "" (at 201.422 95.25 90)
+    (property "Footprint" "Resistor_SMD:R_0603_1608Metric" (at 201.422 95.25 90)
       (effects (font (size 1.27 1.27)) hide)
     )
     (property "Datasheet" "~" (at 203.2 95.25 0)
+      (effects (font (size 1.27 1.27)) hide)
+    )
+    (property "発注先" "Digi-Key" (at 203.2 95.25 0)
       (effects (font (size 1.27 1.27)) hide)
     )
@@
       (effects (font (size 1.27 1.27)) hide)
     )
+    (property "発注先" "Digi-Key" (at 152.4 69.85 0)
+      (effects (font (size 1.27 1.27)) hide)
+    )
     (pin "1")
     (pin "2")
@@
       (effects (font (size 1.27 1.27)) (justify right))
     )
-    (property "Footprint" "" (at 215.9 82.55 0)
+    (property "Footprint" "LED_SMD:LED_0603_1608Metric" (at 215.9 82.55 0)
       (effects (font (size 1.27 1.27)) hide)
     )
@@
       (effects (font (size 1.27 1.27)) hide)
     )
+    (property "発注先" "Digi-Key" (at 215.9 82.55 0)
+      (effects (font (size 1.27 1.27)) hide)
+    )
     (pin "1")
     (pin "2")
@@
       (effects (font (size 1.27 1.27)) (justify left))
     )
-    (property "Footprint" "" (at 239.522 95.25 90)
+    (property "Footprint" "Resistor_SMD:R_0603_1608Metric" (at 239.522 95.25 90)
       (effects (font (size 1.27 1.27)) hide)
     )
@@
       (effects (font (size 1.27 1.27)) hide)
     )
+    (property "発注先" "Digi-Key" (at 241.3 95.25 0)
+      (effects (font (size 1.27 1.27)) hide)
+    )
     (pin "1")
     (pin "2")
@@
     )
     (property "在庫" "" (at 68.58 25.4 0)
+      (effects (font (size 1.27 1.27)) hide)
+    )
+    (property "発注先" "Digi-Key" (at 68.58 25.4 0)
       (effects (font (size 1.27 1.27)) hide)
     )
@@
       (effects (font (size 1.27 1.27)) hide)
     )
+    (property "発注先" "Digi-Key" (at 38.1 116.84 0)
+      (effects (font (size 1.27 1.27)) hide)
+    )
     (pin "1")
     (pin "2")
@@
       (effects (font (size 1.27 1.27)) hide)
     )
+    (property "発注先" "Digi-Key" (at 88.9 158.75 0)
+      (effects (font (size 1.27 1.27)) hide)
+    )
     (pin "1")
     (pin "2")
@@
       (effects (font (size 1.27 1.27)) (justify left))
     )
-    (property "Footprint" "" (at 166.0652 35.56 0)
+    (property "Footprint" "Capacitor_SMD:C_0603_1608Metric" (at 166.0652 35.56 0)
       (effects (font (size 1.27 1.27)) hide)
     )
@@
       (effects (font (size 1.27 1.27)) hide)
     )
+    (property "発注先" "Digi-Key" (at 165.1 31.75 0)
+      (effects (font (size 1.27 1.27)) hide)
+    )
     (pin "1")
     (pin "2")
@@
       (effects (font (size 1.27 1.27)) (justify left))
     )
-    (property "Footprint" "" (at 214.122 38.1 90)
+    (property "Footprint" "Resistor_SMD:R_0603_1608Metric" (at 214.122 38.1 90)
       (effects (font (size 1.27 1.27)) hide)
     )
@@
       (effects (font (size 1.27 1.27)) hide)
     )
+    (property "発注先" "Digi-Key" (at 215.9 38.1 0)
+      (effects (font (size 1.27 1.27)) hide)
+    )
     (pin "1")
     (pin "2")
@@
       (effects (font (size 1.27 1.27)) (justify left))
     )
-    (property "Footprint" "" (at 82.2452 48.26 0)
+    (property "Footprint" "Capacitor_SMD:C_0603_1608Metric" (at 82.2452 48.26 0)
       (effects (font (size 1.27 1.27)) hide)
     )
@@
       (effects (font (size 1.27 1.27)) hide)
     )
+    (property "発注先" "Digi-Key" (at 81.28 44.45 0)
+      (effects (font (size 1.27 1.27)) hide)
+    )
     (pin "1")
     (pin "2")
@@
       (effects (font (size 1.27 1.27)) (justify left))
     )
-    (property "Footprint" "" (at 140.6652 35.56 0)
+    (property "Footprint" "Capacitor_SMD:C_0603_1608Metric" (at 140.6652 35.56 0)
       (effects (font (size 1.27 1.27)) hide)
     )
@@
       (effects (font (size 1.27 1.27)) hide)
     )
+    (property "発注先" "Digi-Key" (at 139.7 31.75 0)
+      (effects (font (size 1.27 1.27)) hide)
+    )
     (pin "1")
     (pin "2")
@@
       (effects (font (size 1.27 1.27)) (justify left))
     )
-    (property "Footprint" "" (at 130.302 184.15 90)
+    (property "Footprint" "Resistor_SMD:R_0603_1608Metric" (at 130.302 184.15 90)
       (effects (font (size 1.27 1.27)) hide)
     )
@@
       (effects (font (size 1.27 1.27)) hide)
     )
+    (property "発注先" "Digi-Key" (at 132.08 184.15 0)
+      (effects (font (size 1.27 1.27)) hide)
+    )
     (pin "1")
     (pin "2")
@@
       (effects (font (size 1.27 1.27)) hide)
     )
+    (property "発注先" "Digi-Key" (at 38.1 129.54 0)
+      (effects (font (size 1.27 1.27)) hide)
+    )
     (pin "1")
     (pin "2")
@@
       (effects (font (size 1.27 1.27)) (justify left))
     )
-    (property "Footprint" "" (at 94.9452 48.26 0)
+    (property "Footprint" "Capacitor_SMD:C_0603_1608Metric" (at 94.9452 48.26 0)
       (effects (font (size 1.27 1.27)) hide)
     )
@@
     )
     (property "在庫" "" (at 93.98 44.45 0)
+      (effects (font (size 1.27 1.27)) hide)
+    )
+    (property "発注先" "Digi-Key" (at 93.98 44.45 0)
       (effects (font (size 1.27 1.27)) hide)
     )
@@
       (effects (font (size 1.27 1.27)) hide)
     )
+    (property "発注先" "Digi-Key" (at 63.5 123.19 0)
+      (effects (font (size 1.27 1.27)) hide)
+    )
     (pin "1")
     (pin "2")
@@
       (effects (font (size 1.27 1.27)) hide)
     )
+    (property "発注先" "Digi-Key" (at 152.4 57.15 0)
+      (effects (font (size 1.27 1.27)) hide)
+    )
     (pin "1")
     (pin "2")
@@
       (effects (font (size 1.27 1.27)) hide)
     )
+    (property "発注先" "Digi-Key" (at 68.58 38.1 0)
+      (effects (font (size 1.27 1.27)) hide)
+    )
     (pin "1")
     (pin "2")
@@
       (effects (font (size 1.27 1.27)) (justify right))
     )
-    (property "Footprint" "" (at 203.2 82.55 0)
+    (property "Footprint" "LED_SMD:LED_0603_1608Metric" (at 203.2 82.55 0)
       (effects (font (size 1.27 1.27)) hide)
     )
@@
       (effects (font (size 1.27 1.27)) hide)
     )
+    (property "発注先" "Digi-Key" (at 203.2 82.55 0)
+      (effects (font (size 1.27 1.27)) hide)
+    )
     (pin "1")
     (pin "2")
@@
       (effects (font (size 1.27 1.27)) (justify right))
     )
-    (property "Footprint" "" (at 241.3 82.55 0)
+    (property "Footprint" "LED_SMD:LED_0603_1608Metric" (at 241.3 82.55 0)
       (effects (font (size 1.27 1.27)) hide)
     )
@@
       (effects (font (size 1.27 1.27)) hide)
     )
+    (property "発注先" "Digi-Key" (at 241.3 82.55 0)
+      (effects (font (size 1.27 1.27)) hide)
+    )
     (pin "1")
     (pin "2")
@@
       (effects (font (size 1.27 1.27)) hide)
     )
+    (property "発注先" "Digi-Key" (at 101.6 190.5 0)
+      (effects (font (size 1.27 1.27)) hide)
+    )
     (pin "1")
     (pin "2")
@@
       (effects (font (size 1.27 1.27)) (justify left))
     )
-    (property "Footprint" "" (at 258.572 38.1 90)
+    (property "Footprint" "Resistor_SMD:R_0603_1608Metric" (at 258.572 38.1 90)
       (effects (font (size 1.27 1.27)) hide)
     )
@@
       (effects (font (size 1.27 1.27)) hide)
     )
+    (property "発注先" "Digi-Key" (at 260.35 38.1 0)
+      (effects (font (size 1.27 1.27)) hide)
+    )
     (pin "1")
     (pin "2")
@@
       (effects (font (size 1.27 1.27)))
     )
-    (property "Footprint" "" (at 92.71 103.1748 0)
+    (property "Footprint" "Capacitor_SMD:C_0603_1608Metric" (at 92.71 103.1748 0)
       (effects (font (size 1.27 1.27)) hide)
     )
@@
       (effects (font (size 1.27 1.27)) hide)
     )
+    (property "発注先" "Digi-Key" (at 88.9 104.14 0)
+      (effects (font (size 1.27 1.27)) hide)
+    )
     (pin "1")
     (pin "2")
@@
       (effects (font (size 1.27 1.27)) hide)
     )
+    (property "発注先" "Digi-Key" (at 69.85 106.68 0)
+      (effects (font (size 1.27 1.27)) hide)
+    )

Commit message: add footprint
Parts:
- R12, R13, R14, R15, R17, R18: footprint (none) -> Resistor_SMD:R_0603_1608Metric
Changed lines of the file:
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@@
       (effects (font (size 1.27 1.27)) (justify right))
     )
-    (property "Footprint" "" (at 90.678 146.05 90)
+    (property "Footprint" "Resistor_SMD:R_0603_1608Metric" (at 90.678 146.05 90)
       (effects (font (size 1.27 1.27)) hide)
     )
@@
       (effects (font (size 1.27 1.27)) (justify right))
     )
-    (property "Footprint" "" (at 90.678 171.45 90)
+    (property "Footprint" "Resistor_SMD:R_0603_1608Metric" (at 90.678 171.45 90)
       (effects (font (size 1.27 1.27)) hide)
     )
@@
       (effects (font (size 1.27 1.27)) (justify right))
     )
-    (property "Footprint" "" (at 154.178 69.85 90)
+    (property "Footprint" "Resistor_SMD:R_0603_1608Metric" (at 154.178 69.85 90)
       (effects (font (size 1.27 1.27)) hide)
     )
@@
       (effects (font (size 1.27 1.27)))
     )
-    (property "Footprint" "" (at 68.58 27.178 90)
+    (property "Footprint" "Resistor_SMD:R_0603_1608Metric" (at 68.58 27.178 90)
       (effects (font (size 1.27 1.27)) hide)
     )
@@
       (effects (font (size 1.27 1.27)) (justify right))
     )
-    (property "Footprint" "" (at 90.678 158.75 90)
+    (property "Footprint" "Resistor_SMD:R_0603_1608Metric" (at 90.678 158.75 90)
       (effects (font (size 1.27 1.27)) hide)
     )
@@
       (effects (font (size 1.27 1.27)) (justify right))
     )
-    (property "Footprint" "" (at 154.178 57.15 90)
-      (effects (font (size 1.27 1.27)) hide)
-    )
+    (property "Footprint" "Resistor_SMD:R_0603_1608Metric" (at 154.178 57.15 90)
+      (effects (font (size 1.27 1.27)) hide)
+    )

Commit message: add footprints to C
Parts:
- C13, C14: footprint (none) -> Capacitor_SMD:C_0402_1005Metric
- C15, C19: footprint (none) -> Capacitor_SMD:C_0805_2012Metric
Changed lines of the file:
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@@
       (effects (font (size 1.27 1.27)))
     )
-    (property "Footprint" "" (at 41.91 115.8748 0)
+    (property "Footprint" "Capacitor_SMD:C_0402_1005Metric" (at 41.91 115.8748 0)
       (effects (font (size 1.27 1.27)) hide)
     )
@@
       (effects (font (size 1.27 1.27)))
     )
-    (property "Footprint" "" (at 41.91 128.5748 0)
+    (property "Footprint" "Capacitor_SMD:C_0402_1005Metric" (at 41.91 128.5748 0)
       (effects (font (size 1.27 1.27)) hide)
     )
@@
       (effects (font (size 1.27 1.27)))
     )
-    (property "Footprint" "" (at 105.41 189.5348 0)
+    (property "Footprint" "Capacitor_SMD:C_0805_2012Metric" (at 105.41 189.5348 0)
       (effects (font (size 1.27 1.27)) hide)
     )
@@
       (effects (font (size 1.27 1.27)))
     )
-    (property "Footprint" "" (at 73.66 105.7148 0)
-      (effects (font (size 1.27 1.27)) hide)
-    )
+    (property "Footprint" "Capacitor_SMD:C_0805_2012Metric" (at 73.66 105.7148 0)
+      (effects (font (size 1.27 1.27)) hide)
+    )

Commit message: add tolerance
Other:
- note added: "0.1%"
Changed lines of the file:
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@@
+    (effects (font (size 1.27 1.27)) (justify left bottom))
+  )
+  (text "0.1%" (at 154.94 62.23 0)
     (effects (font (size 1.27 1.27)) (justify left bottom))
   )
@@
     (effects (font (size 5.08 5.08)) (justify left bottom))
   )
+  (text "0.1%" (at 154.94 74.93 0)
+    (effects (font (size 1.27 1.27)) (justify left bottom))
+  )
   (text "RESET PUSHBUTTON" (at 191.77 30.48 0)
