File: connectors.kicad_sch (KiCad schematic)
At the start: 30 parts, among them J1 Power, J10 Conn_01x03_Pin, J11 Conn_01x03_Pin, J15 Conn_01x04_Pin, J16 Conn_02x05_Odd_Even, J17 Conn_01x02_Pin, J18 Conn_01x06_Pin, J2 Analog, J3 Digital/PWM, J4 Digital/PWM, J5 USB_C_Receptacle, J6 Conn_01x02_Pin, J6 Conn_01x03_Pin, J8 Conn_02x03_Odd_Even, J9 Conn_01x03_Pin

Commit message: add sheet name, explain
Other:
- note added: "CONNECTORS"
Changed lines of the file:
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@@
     (effects (font (size 2.54 2.54)) (justify left bottom))
+  )
+  (text "CONNECTORS" (at 190.5 177.8 0)
+    (effects (font (size 5.08 5.08)) (justify left bottom))
   )
   (text "I2C" (at 231.14 72.39 0)

Commit message: add connector, modify
add SPI connector, modification, add pullup, modify shield connection with GND
Parts:
- removed C1: C, symbol Device:C
- removed J17, J6: Conn_01x02_Pin, symbol Connector:Conn_01x02_Pin
- removed R1: R, symbol Device:R
- added J13: Conn_01x02_Pin, symbol Connector:Conn_01x02_Pin
- added J17: Conn_01x04_Pin, symbol Connector:Conn_01x04_Pin
- added J19: Conn_01x06_Pin, symbol Connector:Conn_01x06_Pin
- added R1 (x4): R, symbol Device:R
Connections:
- net SHIELD is gone; now on net GND: D1.1 (GND), J5.S1 (SHIELD)
- net CANH: now also J13.1 (Pin_1)
- net CANL: now also J13.2 (Pin_2)
- net CS/10: now also J19.5 (Pin_5)
- net GND: now also J17.4 (Pin_4), J19.6 (Pin_6)
- net MISO/12: now also J19.4 (Pin_4), R1.2
- net MOSI/11: now also J19.3 (Pin_3), R1.2
- net SCK/13: now also J19.2 (Pin_2)
- net SCL: now also J17.2 (Pin_2), R1.2
- net SDA: now also J17.3 (Pin_3), R1.2
- net VCC: now also J17.1 (Pin_1), J19.1 (Pin_1), R1.1, R1.1, R1.1, R1.1
Other:
- note added: "SPI"
- moved on the sheet: C1, D1, J1, J10, J11, J15, J16, J18, J2, J3, J4, J5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

Commit message: modify symbol number, constant
Parts:
- C1: value C -> 0.1u
- renumbered J13 to J10, J15 to J11, J17 to J12, J19 to J13, J16 to J14, J8 to J17, J9 to J3, J10 to J4, J11 to J5, J18 to J9
