File: connectors.kicad_sch (KiCad schematic)
At the start: 33 parts, among them J1 Power, J10 Conn_01x02_Pin, J11 Conn_01x04_Pin, J12 Conn_01x04_Pin, J13 Conn_01x06_Pin, J14 Conn_02x05_Odd_Even, J17 Conn_02x03_Odd_Even, J2 Analog, J3 Conn_01x03_Pin, J3 Digital/PWM, J4 Conn_01x03_Pin, J4 Digital/PWM, J5 Conn_01x03_Pin, J5 USB_C_Receptacle, J6 Conn_01x02_Pin, J6 Conn_01x03_Pin, J9 Conn_01x06_Pin

Commit message: decide constant
Parts:
- R1, R2, R3: value R -> 15k
- R1: value R -> 3k
- R1: value R -> 100k
Changed lines of the file:
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@@
       (effects (font (size 1.27 1.27)) (justify left))
     )
-    (property "Value" "R" (at 34.29 160.02 0)
+    (property "Value" "15k" (at 34.29 160.02 0)
       (effects (font (size 1.27 1.27)) (justify left))
     )
@@
       (effects (font (size 1.27 1.27)) (justify left))
     )
-    (property "Value" "R" (at 104.14 64.77 0)
+    (property "Value" "15k" (at 104.14 64.77 0)
       (effects (font (size 1.27 1.27)) (justify left))
     )
@@
       (effects (font (size 1.27 1.27)) (justify left))
     )
-    (property "Value" "R" (at 46.99 160.02 0)
+    (property "Value" "15k" (at 46.99 160.02 0)
       (effects (font (size 1.27 1.27)) (justify left))
     )
@@
       (effects (font (size 1.27 1.27)) (justify left))
     )
-    (property "Value" "R" (at 161.29 68.58 0)
+    (property "Value" "3k" (at 161.29 68.58 0)
       (effects (font (size 1.27 1.27)) (justify left))
     )
@@
       (effects (font (size 1.27 1.27)) (justify left))
     )
-    (property "Value" "R" (at 102.87 158.75 0)
+    (property "Value" "100k" (at 102.87 158.75 0)
       (effects (font (size 1.27 1.27)) (justify left))
     )
@@
       (effects (font (size 1.27 1.27)) (justify left))
     )
-    (property "Value" "R" (at 173.99 97.79 0)
+    (property "Value" "3k" (at 173.99 97.79 0)
       (effects (font (size 1.27 1.27)) (justify left))
     )
@@
       (effects (font (size 1.27 1.27)) (justify left))
     )
-    (property "Value" "R" (at 161.29 97.79 0)
+    (property "Value" "3k" (at 161.29 97.79 0)
       (effects (font (size 1.27 1.27)) (justify left))
     )
@@
       (effects (font (size 1.27 1.27)) (justify left))
     )
-    (property "Value" "R" (at 173.99 68.58 0)
+    (property "Value" "3k" (at 173.99 68.58 0)
       (effects (font (size 1.27 1.27)) (justify left))
     )
@@
       (effects (font (size 1.27 1.27)) (justify left))
     )
-    (property "Value" "R" (at 104.14 96.52 0)
+    (property "Value" "15k" (at 104.14 96.52 0)
       (effects (font (size 1.27 1.27)) (justify left))
     )
@@
       (effects (font (size 1.27 1.27)) (justify left))
     )
-    (property "Value" "R" (at 102.87 133.35 0)
+    (property "Value" "100k" (at 102.87 133.35 0)
       (effects (font (size 1.27 1.27)) (justify left))
     )
@@
       (effects (font (size 1.27 1.27)) (justify left))
     )
-    (property "Value" "R" (at 102.87 184.15 0)
-      (effects (font (size 1.27 1.27)) (justify left))
-    )
+    (property "Value" "100k" (at 102.87 184.15 0)
+      (effects (font (size 1.27 1.27)) (justify left))
+    )

Commit message: add and modify 発注先 and footprint
Parts:
- C1: footprint (none) -> Capacitor_SMD:C_0603_1608Metric; 発注先 (none) -> Digi-Key
- R1, R2, R3: footprint (none) -> Resistor_SMD:R_0603_1608Metric; 発注先 (none) -> Digi-Key
- R1: 発注先 (none) -> Digi-Key
Changed lines of the file:
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@@
       (effects (font (size 1.27 1.27)) (justify left))
     )
-    (property "Footprint" "" (at 29.972 158.75 90)
+    (property "Footprint" "Resistor_SMD:R_0603_1608Metric" (at 29.972 158.75 90)
       (effects (font (size 1.27 1.27)) hide)
     )
@@
       (effects (font (size 1.27 1.27)) hide)
     )
+    (property "発注先" "Digi-Key" (at 31.75 158.75 0)
+      (effects (font (size 1.27 1.27)) hide)
+    )
     (pin "1")
     (pin "2")
@@
       (effects (font (size 1.27 1.27)) (justify left))
     )
-    (property "Footprint" "" (at 99.822 63.5 90)
+    (property "Footprint" "Resistor_SMD:R_0603_1608Metric" (at 99.822 63.5 90)
       (effects (font (size 1.27 1.27)) hide)
     )
@@
       (effects (font (size 1.27 1.27)) hide)
     )
+    (property "発注先" "Digi-Key" (at 101.6 63.5 0)
+      (effects (font (size 1.27 1.27)) hide)
+    )
     (pin "1")
     (pin "2")
@@
       (effects (font (size 1.27 1.27)) (justify left))
     )
-    (property "Footprint" "" (at 42.672 158.75 90)
+    (property "Footprint" "Resistor_SMD:R_0603_1608Metric" (at 42.672 158.75 90)
       (effects (font (size 1.27 1.27)) hide)
     )
@@
     )
     (property "在庫" "" (at 44.45 158.75 0)
+      (effects (font (size 1.27 1.27)) hide)
+    )
+    (property "発注先" "Digi-Key" (at 44.45 158.75 0)
       (effects (font (size 1.27 1.27)) hide)
     )
@@
       (effects (font (size 1.27 1.27)) hide)
     )
+    (property "発注先" "Digi-Key" (at 158.75 67.31 0)
+      (effects (font (size 1.27 1.27)) hide)
+    )
     (pin "1")
     (pin "2")
@@
       (effects (font (size 1.27 1.27)) hide)
     )
+    (property "発注先" "Digi-Key" (at 100.33 157.48 0)
+      (effects (font (size 1.27 1.27)) hide)
+    )
     (pin "1")
     (pin "2")
@@
       (effects (font (size 1.27 1.27)) (justify left))
     )
-    (property "Footprint" "" (at 113.9952 135.89 0)
+    (property "Footprint" "Capacitor_SMD:C_0603_1608Metric" (at 113.9952 135.89 0)
       (effects (font (size 1.27 1.27)) hide)
     )
@@
     )
     (property "在庫" "" (at 113.03 132.08 0)
+      (effects (font (size 1.27 1.27)) hide)
+    )
+    (property "発注先" "Digi-Key" (at 113.03 132.08 0)
       (effects (font (size 1.27 1.27)) hide)
     )
@@
     )
     (property "在庫" "" (at 171.45 96.52 0)
+      (effects (font (size 1.27 1.27)) hide)
+    )
+    (property "発注先" "Digi-Key" (at 171.45 96.52 0)
       (effects (font (size 1.27 1.27)) hide)
     )
@@
       (effects (font (size 1.27 1.27)) hide)
     )
+    (property "発注先" "Digi-Key" (at 158.75 96.52 0)
+      (effects (font (size 1.27 1.27)) hide)
+    )
     (pin "1")
     (pin "2")
@@
     )
     (property "在庫" "" (at 171.45 67.31 0)
+      (effects (font (size 1.27 1.27)) hide)
+    )
+    (property "発注先" "Digi-Key" (at 171.45 67.31 0)
       (effects (font (size 1.27 1.27)) hide)
     )
@@
       (effects (font (size 1.27 1.27)) (justify left))
     )
-    (property "Footprint" "" (at 99.822 95.25 90)
+    (property "Footprint" "Resistor_SMD:R_0603_1608Metric" (at 99.822 95.25 90)
       (effects (font (size 1.27 1.27)) hide)
     )
@@
     )
     (property "在庫" "" (at 101.6 95.25 0)
+      (effects (font (size 1.27 1.27)) hide)
+    )
+    (property "発注先" "Digi-Key" (at 101.6 95.25 0)
       (effects (font (size 1.27 1.27)) hide)
     )
@@
       (effects (font (size 1.27 1.27)) (justify left))
     )
-    (property "Footprint" "" (at 113.9952 186.69 0)
+    (property "Footprint" "Capacitor_SMD:C_0603_1608Metric" (at 113.9952 186.69 0)
       (effects (font (size 1.27 1.27)) hide)
     )
@@
     )
     (property "在庫" "" (at 113.03 182.88 0)
+      (effects (font (size 1.27 1.27)) hide)
+    )
+    (property "発注先" "Digi-Key" (at 113.03 182.88 0)
       (effects (font (size 1.27 1.27)) hide)
     )
@@
       (effects (font (size 1.27 1.27)) hide)
     )
+    (property "発注先" "Digi-Key" (at 100.33 132.08 0)
+      (effects (font (size 1.27 1.27)) hide)
+    )
     (pin "1")
     (pin "2")
@@
     )
     (property "在庫" "" (at 100.33 182.88 0)
+      (effects (font (size 1.27 1.27)) hide)
+    )
+    (property "発注先" "Digi-Key" (at 100.33 182.88 0)
       (effects (font (size 1.27 1.27)) hide)
     )
@@
       (effects (font (size 1.27 1.27)) (justify left))
     )
-    (property "Footprint" "" (at 113.9952 161.29 0)
+    (property "Footprint" "Capacitor_SMD:C_0603_1608Metric" (at 113.9952 161.29 0)
       (effects (font (size 1.27 1.27)) hide)
     )
@@
       (effects (font (size 1.27 1.27)) hide)
     )
+    (property "発注先" "Digi-Key" (at 113.03 157.48 0)
+      (effects (font (size 1.27 1.27)) hide)
+    )

Commit message: add footprint
Parts:
- R1: footprint (none) -> Resistor_SMD:R_0603_1608Metric
Changed lines of the file:
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@@
       (effects (font (size 1.27 1.27)) (justify left))
     )
-    (property "Footprint" "" (at 156.972 67.31 90)
+    (property "Footprint" "Resistor_SMD:R_0603_1608Metric" (at 156.972 67.31 90)
       (effects (font (size 1.27 1.27)) hide)
     )
@@
       (effects (font (size 1.27 1.27)) (justify left))
     )
-    (property "Footprint" "" (at 98.552 157.48 90)
+    (property "Footprint" "Resistor_SMD:R_0603_1608Metric" (at 98.552 157.48 90)
       (effects (font (size 1.27 1.27)) hide)
     )
@@
       (effects (font (size 1.27 1.27)) (justify left))
     )
-    (property "Footprint" "" (at 169.672 96.52 90)
+    (property "Footprint" "Resistor_SMD:R_0603_1608Metric" (at 169.672 96.52 90)
       (effects (font (size 1.27 1.27)) hide)
     )
@@
       (effects (font (size 1.27 1.27)) (justify left))
     )
-    (property "Footprint" "" (at 156.972 96.52 90)
+    (property "Footprint" "Resistor_SMD:R_0603_1608Metric" (at 156.972 96.52 90)
       (effects (font (size 1.27 1.27)) hide)
     )
@@
       (effects (font (size 1.27 1.27)) (justify left))
     )
-    (property "Footprint" "" (at 169.672 67.31 90)
+    (property "Footprint" "Resistor_SMD:R_0603_1608Metric" (at 169.672 67.31 90)
       (effects (font (size 1.27 1.27)) hide)
     )
@@
       (effects (font (size 1.27 1.27)) (justify left))
     )
-    (property "Footprint" "" (at 98.552 132.08 90)
+    (property "Footprint" "Resistor_SMD:R_0603_1608Metric" (at 98.552 132.08 90)
       (effects (font (size 1.27 1.27)) hide)
     )
@@
       (effects (font (size 1.27 1.27)) (justify left))
     )
-    (property "Footprint" "" (at 98.552 182.88 90)
-      (effects (font (size 1.27 1.27)) hide)
-    )
+    (property "Footprint" "Resistor_SMD:R_0603_1608Metric" (at 98.552 182.88 90)
+      (effects (font (size 1.27 1.27)) hide)
+    )

Commit message: コネクタフットプリント割当
Parts:
- J10, J6: footprint (none) -> Connector_JST:JST_XH_B2B-XH-A_1x02_P2.50mm_Vertical
- J11, J12: footprint (none) -> Connector_JST:JST_XH_B4B-XH-A_1x04_P2.50mm_Vertical
- J13, J9: footprint (none) -> Connector_JST:JST_XH_B6B-XH-A_1x06_P2.50mm_Vertical
- J14: footprint (none) -> Connector_PinHeader_2.54mm:PinHeader_2x05_P2.54mm_Vertical
- J3, J4, J5, J6: footprint (none) -> Connector_JST:JST_XH_B3B-XH-A_1x03_P2.50mm_Vertical
Changed lines of the file:
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@@
       (effects (font (size 1.27 1.27)))
     )
-    (property "Footprint" "" (at 86.36 34.29 0)
+    (property "Footprint" "Connector_JST:JST_XH_B3B-XH-A_1x03_P2.50mm_Vertical" (at 86.36 34.29 0)
       (effects (font (size 1.27 1.27)) hide)
     )
@@
       (effects (font (size 1.27 1.27)))
     )
-    (property "Footprint" "" (at 85.09 127 0)
+    (property "Footprint" "Connector_JST:JST_XH_B3B-XH-A_1x03_P2.50mm_Vertical" (at 85.09 127 0)
       (effects (font (size 1.27 1.27)) hide)
     )
@@
       (effects (font (size 1.27 1.27)))
     )
-    (property "Footprint" "" (at 156.21 142.24 0)
+    (property "Footprint" "Connector_JST:JST_XH_B6B-XH-A_1x06_P2.50mm_Vertical" (at 156.21 142.24 0)
       (effects (font (size 1.27 1.27)) hide)
     )
@@
       (effects (font (size 1.27 1.27)) (justify right))
     )
-    (property "Footprint" "" (at 177.8 106.68 0)
+    (property "Footprint" "Connector_JST:JST_XH_B6B-XH-A_1x06_P2.50mm_Vertical" (at 177.8 106.68 0)
       (effects (font (size 1.27 1.27)) hide)
     )
@@
       (effects (font (size 1.27 1.27)) (justify right))
     )
-    (property "Footprint" "" (at 177.8 74.93 0)
+    (property "Footprint" "Connector_JST:JST_XH_B4B-XH-A_1x04_P2.50mm_Vertical" (at 177.8 74.93 0)
       (effects (font (size 1.27 1.27)) hide)
     )
@@
       (effects (font (size 1.27 1.27)))
     )
-    (property "Footprint" "" (at 95.25 87.63 0)
+    (property "Footprint" "Connector_JST:JST_XH_B2B-XH-A_1x02_P2.50mm_Vertical" (at 95.25 87.63 0)
       (effects (font (size 1.27 1.27)) hide)
     )
@@
       (effects (font (size 1.27 1.27)))
     )
-    (property "Footprint" "" (at 85.09 177.8 0)
+    (property "Footprint" "Connector_JST:JST_XH_B3B-XH-A_1x03_P2.50mm_Vertical" (at 85.09 177.8 0)
       (effects (font (size 1.27 1.27)) hide)
     )
@@
       (effects (font (size 1.27 1.27)))
     )
-    (property "Footprint" "" (at 95.25 55.88 0)
+    (property "Footprint" "Connector_JST:JST_XH_B2B-XH-A_1x02_P2.50mm_Vertical" (at 95.25 55.88 0)
       (effects (font (size 1.27 1.27)) hide)
     )
@@
       (effects (font (size 1.27 1.27)) (justify right))
     )
-    (property "Footprint" "" (at 176.53 31.75 0)
+    (property "Footprint" "Connector_JST:JST_XH_B4B-XH-A_1x04_P2.50mm_Vertical" (at 176.53 31.75 0)
       (effects (font (size 1.27 1.27)) hide)
     )
@@
       (effects (font (size 1.27 1.27)))
     )
-    (property "Footprint" "" (at 219.71 106.68 0)
+    (property "Footprint" "Connector_PinHeader_2.54mm:PinHeader_2x05_P2.54mm_Vertical" (at 219.71 106.68 0)
       (effects (font (size 1.27 1.27)) hide)
     )
@@
       (effects (font (size 1.27 1.27)))
     )
-    (property "Footprint" "" (at 85.09 152.4 0)
+    (property "Footprint" "Connector_JST:JST_XH_B3B-XH-A_1x03_P2.50mm_Vertical" (at 85.09 152.4 0)
       (effects (font (size 1.27 1.27)) hide)
     )
@@
       (effects (font (size 1.27 1.27)) (justify right))
     )
-    (property "Footprint" "" (at 161.29 48.26 0)
-      (effects (font (size 1.27 1.27)) hide)
-    )
+    (property "Footprint" "Connector_JST:JST_XH_B2B-XH-A_1x02_P2.50mm_Vertical" (at 161.29 48.26 0)
+      (effects (font (size 1.27 1.27)) hide)
+    )

Commit message: modify SPI connector pin assign
Connections:
- net MISO/12: now also J13.3 (Pin_3), R1.2; no longer J13.4 (Pin_4), R1.2
- net MOSI/11: now also J13.4 (Pin_4), R1.2; no longer J13.3 (Pin_3), R1.2
Changed lines of the file:
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@@
   (junction (at 38.1 101.6) (diameter 0) (color 0 0 0 0)
   )
+  (junction (at 158.75 106.68) (diameter 0) (color 0 0 0 0)
+  )
   (junction (at 113.03 127) (diameter 0) (color 0 0 0 0)
   )
@@
   (junction (at 158.75 74.93) (diameter 0) (color 0 0 0 0)
   )
-  (junction (at 158.75 106.68) (diameter 0) (color 0 0 0 0)
-  )
   (junction (at 100.33 177.8) (diameter 0) (color 0 0 0 0)
   )
@@
   (junction (at 113.03 177.8) (diameter 0) (color 0 0 0 0)
   )
+  (junction (at 171.45 109.22) (diameter 0) (color 0 0 0 0)
+  )
   (junction (at 171.45 77.47) (diameter 0) (color 0 0 0 0)
-  )
-  (junction (at 171.45 109.22) (diameter 0) (color 0 0 0 0)
   )
   (junction (at 92.71 36.83) (diameter 0) (color 0 0 0 0)
@@
     (stroke (width 0) (type default))
   )
+  (wire (pts (xy 157.48 109.22) (xy 171.45 109.22))
+    (stroke (width 0) (type default))
+  )
   (wire (pts (xy 30.48 100.33) (xy 30.48 101.6))
     (stroke (width 0) (type default))
@@
   )
   (wire (pts (xy 170.18 29.21) (xy 171.45 29.21))
+    (stroke (width 0) (type default))
+  )
+  (wire (pts (xy 157.48 106.68) (xy 158.75 106.68))
     (stroke (width 0) (type default))
   )
@@
     (stroke (width 0) (type default))
   )
-  (wire (pts (xy 157.48 106.68) (xy 158.75 106.68))
-    (stroke (width 0) (type default))
-  )
   (wire (pts (xy 171.45 62.23) (xy 171.45 63.5))
     (stroke (width 0) (type default))
@@
   )
   (wire (pts (xy 54.61 52.07) (xy 54.61 54.61))
-    (stroke (width 0) (type default))
-  )
-  (wire (pts (xy 157.48 109.22) (xy 171.45 109.22))
     (stroke (width 0) (type default))
   )
@@
     (effects (font (size 1.27 1.27)) (justify left))
   )
-  (hierarchical_label "MISO{slash}12" (shape bidirectional) (at 157.48 109.22 180) (fields_autoplaced)
+  (hierarchical_label "MISO{slash}12" (shape bidirectional) (at 157.48 106.68 180) (fields_autoplaced)
     (effects (font (size 1.27 1.27)) (justify right))
   )
@@
     (effects (font (size 1.27 1.27)) (justify right))
   )
-  (hierarchical_label "MOSI{slash}11" (shape bidirectional) (at 157.48 106.68 180) (fields_autoplaced)
-    (effects (font (size 1.27 1.27)) (justify right))
-  )
+  (hierarchical_label "MOSI{slash}11" (shape bidirectional) (at 157.48 109.22 180) (fields_autoplaced)
+    (effects (font (size 1.27 1.27)) (justify right))
+  )

Commit message: modify footprint path and 3dmodel path
Parts:
- J5: footprint SamacSys_Parts:5077CR-16-SMC2-BK-TR -> ProjectEV-kicad-library:5077CR-16-SMC2-BK-TR
Changed lines of the file:
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@@
       (effects (font (size 1.27 1.27)))
     )
-    (property "Footprint" "SamacSys_Parts:5077CR-16-SMC2-BK-TR" (at 41.91 59.69 0)
+    (property "Footprint" "ProjectEV-kicad-library:5077CR-16-SMC2-BK-TR" (at 41.91 59.69 0)
       (effects (font (size 1.27 1.27)) hide)
     )

Commit message: Arduino header削除、ピンアサイン修正
ハイサイドスイッチ信号、UARTなど
Arduino互換ピンはXHで出す
回路図一部修正
パターン削除、部品配置
Parts:
- removed J1: Power, Connector_PinSocket_2.54mm:PinSocket_1x08_P2.54mm_Vertical, symbol Connector_Generic:Conn_01x08
- removed J17: Conn_02x03_Odd_Even, Connector_PinHeader_2.54mm:PinHeader_2x03_P2.54mm_Vertical, symbol Connector_Generic:Conn_02x03_Odd_Even
- removed J2: Analog, Connector_PinSocket_2.54mm:PinSocket_1x06_P2.54mm_Vertical, symbol Connector_Generic:Conn_01x06
- removed J3: Digital/PWM, Connector_PinSocket_2.54mm:PinSocket_1x10_P2.54mm_Vertical, symbol Connector_Generic:Conn_01x10
- removed J4: Digital/PWM, Connector_PinSocket_2.54mm:PinSocket_1x08_P2.54mm_Vertical, symbol Connector_Generic:Conn_01x08
- added C1: 0.1u, Capacitor_SMD:C_0603_1608Metric, symbol Device:C
- added J10: Conn_01x04_Pin, Connector_JST:JST_XH_B4B-XH-A_1x04_P2.50mm_Vertical, symbol Connector:Conn_01x04_Pin
- added J14: Conn_01x03_Pin, Connector_JST:JST_XH_B3B-XH-A_1x03_P2.50mm_Vertical, symbol Connector:Conn_01x03_Pin
- added R1: 100k, Resistor_SMD:R_0603_1608Metric, symbol Device:R
- renumbered J14 to J15, J9 to J16, J10 to J9
Connections:
- net GND: now also J16.1 (Pin_1), C1.2, J10.4 (Pin_4), J14.3 (Pin_3), R1.2; no longer J16.6 (Pin_6)
- net OPT_I/O_1: now also J16.5 (Pin_5); no longer J16.2 (Pin_2)
- net OPT_I/O_2: now also J16.4 (Pin_4); no longer J16.3 (Pin_3)
- net OPT_I/O_3: now also J16.3 (Pin_3); no longer J16.4 (Pin_4)
- net OPT_I/O_4: now also J16.2 (Pin_2); no longer J16.5 (Pin_5)
- net VCC: now also J16.6 (Pin_6), J10.1 (Pin_1), J14.1 (Pin_1); no longer J16.1 (Pin_1)
- new net ANALOG_I/O_1: C1.1, J14.2 (Pin_2), R1.1
- new net RX: J10.3 (Pin_3)
- new net TX: J10.2 (Pin_2)
Other:
- note added: "ANALOG I/O"
- note added: "OPT"
- note added: "SERIAL1 (UART)"
- note removed: "ARDUINO HEADER"
- moved on the sheet: J16

Commit message: デバッグインターフェースのフットプリント変更
2.54mm pitch -> 1.00 mm pitch
Parts:
- J15: footprint Connector_PinHeader_2.54mm:PinHeader_2x05_P2.54mm_Vertical -> Connector_PinHeader_1.00mm:PinHeader_2x05_P1.00mm_Vertical
Changed lines of the file:
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@@
       (effects (font (size 1.27 1.27)))
     )
-    (property "Footprint" "Connector_PinHeader_2.54mm:PinHeader_2x05_P2.54mm_Vertical" (at 219.71 106.68 0)
+    (property "Footprint" "Connector_PinHeader_1.00mm:PinHeader_2x05_P1.00mm_Vertical" (at 219.71 106.68 0)
       (effects (font (size 1.27 1.27)) hide)
     )
