File: connectors.kicad_sch (KiCad schematic)
At the start: 32 parts, among them J10 Conn_01x04_Pin, J11 Conn_01x04_Pin, J12 Conn_01x04_Pin, J13 Conn_01x06_Pin, J14 Conn_01x03_Pin, J15 Conn_02x05_Odd_Even, J16 Conn_01x06_Pin, J3 Conn_01x03_Pin, J4 Conn_01x03_Pin, J5 Conn_01x03_Pin, J5 USB_C_Receptacle, J6 Conn_01x02_Pin, J6 Conn_01x03_Pin, J9 Conn_01x02_Pin

Commit message: ピンアサイン修正
OPTIONAL I/O の電源ピン
Connections:
- net GND: now also J16.6 (Pin_6); no longer J16.1 (Pin_1)
- net OPT_I/O_1: now also J16.2 (Pin_2); no longer J16.5 (Pin_5)
- net OPT_I/O_2: now also J16.3 (Pin_3); no longer J16.4 (Pin_4)
- net OPT_I/O_3: now also J16.4 (Pin_4); no longer J16.3 (Pin_3)
- net OPT_I/O_4: now also J16.5 (Pin_5); no longer J16.2 (Pin_2)
- net VCC: now also J16.1 (Pin_1); no longer J16.6 (Pin_6)
Other:
- moved on the sheet: J16
Changed lines of the file:
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@@
     )
   )
-  (symbol (lib_id "Connector:Conn_01x06_Pin") (at 222.25 71.12 180) (unit 1)
-    (in_bom yes) (on_board yes) (dnp no) (fields_autoplaced)
-    (property "Reference" "J16" (at 223.52 68.58 0)
+  (symbol (lib_id "Connector:Conn_01x06_Pin") (at 222.25 68.58 0) (mirror y) (unit 1)
+    (in_bom yes) (on_board yes) (dnp no)
+    (property "Reference" "J16" (at 223.52 71.12 0)
       (effects (font (size 1.27 1.27)) (justify right))
     )
-    (property "Value" "Conn_01x06_Pin" (at 223.52 71.12 0)
+    (property "Value" "Conn_01x06_Pin" (at 223.52 68.58 0)
       (effects (font (size 1.27 1.27)) (justify right))
     )
-    (property "Footprint" "Connector_JST:JST_XH_B6B-XH-A_1x06_P2.50mm_Vertical" (at 222.25 71.12 0)
+    (property "Footprint" "Connector_JST:JST_XH_B6B-XH-A_1x06_P2.50mm_Vertical" (at 222.25 68.58 0)
       (effects (font (size 1.27 1.27)) hide)
     )
-    (property "Datasheet" "~" (at 222.25 71.12 0)
+    (property "Datasheet" "~" (at 222.25 68.58 0)
       (effects (font (size 1.27 1.27)) hide)
     )
