File: level-shift.kicad_sch (KiCad schematic)
At the start: 3 parts, among them Q2 2N7002K

Commit message: add sheet name, explain
Other:
- note added: "LEVEL SHIFT"
Changed lines of the file:
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@@
     (stroke (width 0) (type default))
+  )
+  (text "LEVEL SHIFT" (at 190.5 177.8 0)
+    (effects (font (size 5.08 5.08)) (justify left bottom))
   )
   (hierarchical_label "VCC_SIG" (shape output) (at 139.7 76.2 0) (fields_autoplaced)

Commit message: modify symbol number, constant
Parts:
- renumbered R40 to R47, R41 to R48
Changed lines of the file:
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@@
   (symbol (lib_id "Device:R") (at 127 69.85 0) (unit 1)
     (in_bom yes) (on_board yes) (dnp no) (fields_autoplaced)
-    (property "Reference" "R41" (at 129.54 68.58 0)
+    (property "Reference" "R48" (at 129.54 68.58 0)
       (effects (font (size 1.27 1.27)) (justify left))
     )
@@
       (project "main-ECU-board"
         (path "/10edd9b6-c7a8-40f4-bfe3-c9724324d30f/aaf3b5fe-1b86-4630-ab8c-ff326b8bda0a"
-          (reference "R41") (unit 1)
+          (reference "R48") (unit 1)
         )
       )
@@
   (symbol (lib_id "Device:R") (at 114.3 95.25 0) (unit 1)
     (in_bom yes) (on_board yes) (dnp no) (fields_autoplaced)
-    (property "Reference" "R40" (at 116.84 93.98 0)
+    (property "Reference" "R47" (at 116.84 93.98 0)
       (effects (font (size 1.27 1.27)) (justify left))
     )
@@
       (project "main-ECU-board"
         (path "/10edd9b6-c7a8-40f4-bfe3-c9724324d30f/aaf3b5fe-1b86-4630-ab8c-ff326b8bda0a"
-          (reference "R40") (unit 1)
+          (reference "R47") (unit 1)
         )
       )
@@
   (symbol (lib_id "power:GND") (at 127 104.14 0) (unit 1)
     (in_bom yes) (on_board yes) (dnp no) (fields_autoplaced)
-    (property "Reference" "#PWR086" (at 127 110.49 0)
+    (property "Reference" "#PWR091" (at 127 110.49 0)
       (effects (font (size 1.27 1.27)) hide)
     )
@@
       (project "main-ECU-board"
         (path "/10edd9b6-c7a8-40f4-bfe3-c9724324d30f/aaf3b5fe-1b86-4630-ab8c-ff326b8bda0a"
-          (reference "#PWR086") (unit 1)
+          (reference "#PWR091") (unit 1)
         )
       )
