File: load-switch.kicad_sch (KiCad schematic)
At the start: 14 parts, among them IC3 TPS2H160AQPWPRQ1, IC4 TPS2H160AQPWPRQ1

Commit message: modify signal name
Connections:
- net AIR_M_OUT_12V renamed AIR_M_OUT
- net AIR_M_SIG_5V renamed AIR_M_SIG
- net AIR_P_OUT_12V renamed AIR_P_OUT
- net AIR_P_SIG_5V renamed AIR_P_SIG
- net PRECHARGE_OUT_12V renamed PRECHARGE_OUT
- net PRECHARGE_SIG_5V renamed PRECHARGE_SIG
- net READY_TO_DRIVE_OUT_12V renamed READY_TO_DRIVE_OUT
- net READY_TO_DRIVE_SIG_5V renamed READY_TO_DRIVE_SIG
Changed lines of the file:
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@@
     (effects (font (size 1.27 1.27)) (justify left bottom))
   )
-  (hierarchical_label "PRECHARGE_OUT_12V" (shape output) (at 124.46 81.28 0) (fields_autoplaced)
+  (hierarchical_label "PRECHARGE_OUT" (shape output) (at 124.46 81.28 0) (fields_autoplaced)
     (effects (font (size 1.27 1.27)) (justify left))
   )
@@
     (effects (font (size 1.27 1.27)) (justify left))
   )
-  (hierarchical_label "READY_TO_DRIVE_SIG_5V" (shape input) (at 63.5 50.8 180) (fields_autoplaced)
+  (hierarchical_label "READY_TO_DRIVE_SIG" (shape input) (at 63.5 50.8 180) (fields_autoplaced)
     (effects (font (size 1.27 1.27)) (justify right))
   )
-  (hierarchical_label "AIR_P_OUT_12V" (shape output) (at 238.76 71.12 0) (fields_autoplaced)
+  (hierarchical_label "AIR_P_OUT" (shape output) (at 238.76 71.12 0) (fields_autoplaced)
     (effects (font (size 1.27 1.27)) (justify left))
   )
-  (hierarchical_label "AIR_P_SIG_5V" (shape input) (at 177.8 50.8 180) (fields_autoplaced)
+  (hierarchical_label "AIR_P_SIG" (shape input) (at 177.8 50.8 180) (fields_autoplaced)
     (effects (font (size 1.27 1.27)) (justify right))
   )
@@
     (effects (font (size 1.27 1.27)) (justify right))
   )
-  (hierarchical_label "AIR_M_OUT_12V" (shape output) (at 238.76 81.28 0) (fields_autoplaced)
+  (hierarchical_label "AIR_M_OUT" (shape output) (at 238.76 81.28 0) (fields_autoplaced)
     (effects (font (size 1.27 1.27)) (justify left))
   )
@@
     (effects (font (size 1.27 1.27)) (justify right))
   )
-  (hierarchical_label "PRECHARGE_SIG_5V" (shape input) (at 63.5 63.5 180) (fields_autoplaced)
+  (hierarchical_label "PRECHARGE_SIG" (shape input) (at 63.5 63.5 180) (fields_autoplaced)
     (effects (font (size 1.27 1.27)) (justify right))
   )
@@
     (effects (font (size 1.27 1.27)) (justify right))
   )
-  (hierarchical_label "READY_TO_DRIVE_OUT_12V" (shape output) (at 124.46 71.12 0) (fields_autoplaced)
+  (hierarchical_label "READY_TO_DRIVE_OUT" (shape output) (at 124.46 71.12 0) (fields_autoplaced)
     (effects (font (size 1.27 1.27)) (justify left))
   )
@@
     (effects (font (size 1.27 1.27)) (justify right))
   )
-  (hierarchical_label "AIR_M_SIG_5V" (shape input) (at 177.8 63.5 180) (fields_autoplaced)
+  (hierarchical_label "AIR_M_SIG" (shape input) (at 177.8 63.5 180) (fields_autoplaced)
     (effects (font (size 1.27 1.27)) (justify right))
   )

Commit message: add sheet name, explain
Other:
- note added: "LOAD SWITCH"
Changed lines of the file:
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@@
     (stroke (width 0) (type default))
   )
+  (text "LOAD SWITCH" (at 190.5 177.8 0)
+    (effects (font (size 5.08 5.08)) (justify left bottom))
+  )
   (text "WHEN DIAG_EN IS LOW, ~{STx} IS HIGH IMPEDANCE.\nWHEN YOU WANT TO USE THE DIAGNOSTIC FUNCTIONS,\nSET DIAG_EN PIN OF THE DEVICE YOU CHOOSE TO HIGH."
-    (at 203.2 38.1 0)
-    (effects (font (size 1.27 1.27)) (justify left bottom))
+    (at 38.1 177.8 0)
+    (effects (font (size 2.54 2.54)) (justify left bottom))
   )
   (hierarchical_label "PRECHARGE_OUT" (shape output) (at 124.46 81.28 0) (fields_autoplaced)

Commit message: modify symbol number, constant
Parts:
- renumbered R34 to R37, R37 to R38, R31 to R39, R32 to R40, R33 to R41, R38 to R42
Changed lines of the file:
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@@
   (symbol (lib_id "power:GND") (at 81.28 91.44 0) (unit 1)
     (in_bom yes) (on_board yes) (dnp no) (fields_autoplaced)
-    (property "Reference" "#PWR059" (at 81.28 97.79 0)
+    (property "Reference" "#PWR084" (at 81.28 97.79 0)
       (effects (font (size 1.27 1.27)) hide)
     )
@@
       (project "main-ECU-board"
         (path "/10edd9b6-c7a8-40f4-bfe3-c9724324d30f/2f8be702-5d98-41c6-b186-35624bc097b2"
-          (reference "#PWR059") (unit 1)
+          (reference "#PWR084") (unit 1)
         )
       )
@@
   (symbol (lib_id "power:GND") (at 69.85 101.6 0) (unit 1)
     (in_bom yes) (on_board yes) (dnp no) (fields_autoplaced)
-    (property "Reference" "#PWR071" (at 69.85 107.95 0)
+    (property "Reference" "#PWR083" (at 69.85 107.95 0)
       (effects (font (size 1.27 1.27)) hide)
     )
@@
       (project "main-ECU-board"
         (path "/10edd9b6-c7a8-40f4-bfe3-c9724324d30f/2f8be702-5d98-41c6-b186-35624bc097b2"
-          (reference "#PWR071") (unit 1)
+          (reference "#PWR083") (unit 1)
         )
       )
@@
   (symbol (lib_id "power:GND") (at 236.22 91.44 0) (unit 1)
     (in_bom yes) (on_board yes) (dnp no) (fields_autoplaced)
-    (property "Reference" "#PWR073" (at 236.22 97.79 0)
+    (property "Reference" "#PWR090" (at 236.22 97.79 0)
       (effects (font (size 1.27 1.27)) hide)
     )
@@
       (project "main-ECU-board"
         (path "/10edd9b6-c7a8-40f4-bfe3-c9724324d30f/2f8be702-5d98-41c6-b186-35624bc097b2"
-          (reference "#PWR073") (unit 1)
+          (reference "#PWR090") (unit 1)
         )
       )
@@
   (symbol (lib_id "power:GND") (at 215.9 104.14 0) (unit 1)
     (in_bom yes) (on_board yes) (dnp no) (fields_autoplaced)
-    (property "Reference" "#PWR072" (at 215.9 110.49 0)
+    (property "Reference" "#PWR089" (at 215.9 110.49 0)
       (effects (font (size 1.27 1.27)) hide)
     )
@@
       (project "main-ECU-board"
         (path "/10edd9b6-c7a8-40f4-bfe3-c9724324d30f/2f8be702-5d98-41c6-b186-35624bc097b2"
-          (reference "#PWR072") (unit 1)
+          (reference "#PWR089") (unit 1)
         )
       )
@@
   (symbol (lib_id "Device:R") (at 50.8 107.95 0) (unit 1)
     (in_bom yes) (on_board yes) (dnp no) (fields_autoplaced)
-    (property "Reference" "R34" (at 53.34 106.68 0)
+    (property "Reference" "R37" (at 53.34 106.68 0)
       (effects (font (size 1.27 1.27)) (justify left))
     )
@@
       (project "main-ECU-board"
         (path "/10edd9b6-c7a8-40f4-bfe3-c9724324d30f/2f8be702-5d98-41c6-b186-35624bc097b2"
-          (reference "R34") (unit 1)
+          (reference "R37") (unit 1)
         )
       )
@@
   (symbol (lib_id "Device:R") (at 69.85 50.8 90) (unit 1)
     (in_bom yes) (on_board yes) (dnp no) (fields_autoplaced)
-    (property "Reference" "R31" (at 69.85 44.45 90)
+    (property "Reference" "R39" (at 69.85 44.45 90)
       (effects (font (size 1.27 1.27)))
     )
@@
       (project "main-ECU-board"
         (path "/10edd9b6-c7a8-40f4-bfe3-c9724324d30f/2f8be702-5d98-41c6-b186-35624bc097b2"
-          (reference "R31") (unit 1)
+          (reference "R39") (unit 1)
         )
       )
@@
   (symbol (lib_id "Device:R") (at 69.85 95.25 0) (unit 1)
     (in_bom yes) (on_board yes) (dnp no) (fields_autoplaced)
-    (property "Reference" "R38" (at 72.39 93.98 0)
+    (property "Reference" "R42" (at 72.39 93.98 0)
       (effects (font (size 1.27 1.27)) (justify left))
     )
@@
       (project "main-ECU-board"
         (path "/10edd9b6-c7a8-40f4-bfe3-c9724324d30f/2f8be702-5d98-41c6-b186-35624bc097b2"
-          (reference "R38") (unit 1)
+          (reference "R42") (unit 1)
         )
       )
@@
   (symbol (lib_id "Device:R") (at 69.85 76.2 90) (unit 1)
     (in_bom yes) (on_board yes) (dnp no) (fields_autoplaced)
-    (property "Reference" "R33" (at 69.85 69.85 90)
+    (property "Reference" "R41" (at 69.85 69.85 90)
       (effects (font (size 1.27 1.27)))
     )
@@
       (project "main-ECU-board"
         (path "/10edd9b6-c7a8-40f4-bfe3-c9724324d30f/2f8be702-5d98-41c6-b186-35624bc097b2"
-          (reference "R33") (unit 1)
+          (reference "R41") (unit 1)
         )
       )
@@
   (symbol (lib_id "power:GND") (at 121.92 91.44 0) (unit 1)
     (in_bom yes) (on_board yes) (dnp no) (fields_autoplaced)
-    (property "Reference" "#PWR067" (at 121.92 97.79 0)
+    (property "Reference" "#PWR086" (at 121.92 97.79 0)
       (effects (font (size 1.27 1.27)) hide)
     )
@@
       (project "main-ECU-board"
         (path "/10edd9b6-c7a8-40f4-bfe3-c9724324d30f/2f8be702-5d98-41c6-b186-35624bc097b2"
-          (reference "#PWR067") (unit 1)
+          (reference "#PWR086") (unit 1)
         )
       )
@@
   (symbol (lib_id "power:GND") (at 195.58 91.44 0) (unit 1)
     (in_bom yes) (on_board yes) (dnp no) (fields_autoplaced)
-    (property "Reference" "#PWR074" (at 195.58 97.79 0)
+    (property "Reference" "#PWR088" (at 195.58 97.79 0)
       (effects (font (size 1.27 1.27)) hide)
     )
@@
       (project "main-ECU-board"
         (path "/10edd9b6-c7a8-40f4-bfe3-c9724324d30f/2f8be702-5d98-41c6-b186-35624bc097b2"
-          (reference "#PWR074") (unit 1)
+          (reference "#PWR088") (unit 1)
         )
       )
@@
   (symbol (lib_id "power:GND") (at 184.15 101.6 0) (unit 1)
     (in_bom yes) (on_board yes) (dnp no) (fields_autoplaced)
-    (property "Reference" "#PWR075" (at 184.15 107.95 0)
+    (property "Reference" "#PWR087" (at 184.15 107.95 0)
       (effects (font (size 1.27 1.27)) hide)
     )
@@
       (project "main-ECU-board"
         (path "/10edd9b6-c7a8-40f4-bfe3-c9724324d30f/2f8be702-5d98-41c6-b186-35624bc097b2"
-          (reference "#PWR075") (unit 1)
+          (reference "#PWR087") (unit 1)
         )
       )
@@
   (symbol (lib_id "Device:R") (at 50.8 133.35 0) (unit 1)
     (in_bom yes) (on_board yes) (dnp no) (fields_autoplaced)
-    (property "Reference" "R37" (at 53.34 132.08 0)
+    (property "Reference" "R38" (at 53.34 132.08 0)
       (effects (font (size 1.27 1.27)) (justify left))
     )
@@
       (project "main-ECU-board"
         (path "/10edd9b6-c7a8-40f4-bfe3-c9724324d30f/2f8be702-5d98-41c6-b186-35624bc097b2"
-          (reference "R37") (unit 1)
+          (reference "R38") (unit 1)
         )
       )
@@
   (symbol (lib_id "power:GND") (at 101.6 104.14 0) (unit 1)
     (in_bom yes) (on_board yes) (dnp no) (fields_autoplaced)
-    (property "Reference" "#PWR068" (at 101.6 110.49 0)
+    (property "Reference" "#PWR085" (at 101.6 110.49 0)
       (effects (font (size 1.27 1.27)) hide)
     )
@@
       (project "main-ECU-board"
         (path "/10edd9b6-c7a8-40f4-bfe3-c9724324d30f/2f8be702-5d98-41c6-b186-35624bc097b2"
-          (reference "#PWR068") (unit 1)
+          (reference "#PWR085") (unit 1)
         )
       )
@@
   (symbol (lib_id "Device:R") (at 69.85 63.5 90) (unit 1)
     (in_bom yes) (on_board yes) (dnp no) (fields_autoplaced)
-    (property "Reference" "R32" (at 69.85 57.15 90)
+    (property "Reference" "R40" (at 69.85 57.15 90)
       (effects (font (size 1.27 1.27)))
     )
@@
       (project "main-ECU-board"
         (path "/10edd9b6-c7a8-40f4-bfe3-c9724324d30f/2f8be702-5d98-41c6-b186-35624bc097b2"
-          (reference "R32") (unit 1)
-        )
-      )
+          (reference "R40") (unit 1)
+        )
+      )
