File: load-switch.kicad_sch (KiCad schematic)
At the start: 14 parts, among them IC3 TPS2H160AQPWPRQ1, IC4 TPS2H160AQPWPRQ1

Commit message: decide constant, modify
Parts:
- added D10, D9: RB160M-30TR, Diode_SMD:D_SOD-123F, symbol Device:D
- added R49, R50: 1k, symbol Device:R
- R35, R36, R37, R38, R39, R40, R41, R43, R44, R45: value R -> 10k
- R42, R46: value R -> 1k
Connections:
- net GND: now also D10.1 (K), D9.1 (K), R49.2, R50.2; no longer IC3.8 (GND), IC4.8 (GND)
- new net: D9.2 (A), IC3.8 (GND), R49.1
- new net: D10.2 (A), IC4.8 (GND), R50.1
Other:
- moved on the sheet: IC3, IC4, R35, R36, R37, R38, R39, R40, R41, R42, R43, R44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

Commit message: re-annotate
Parts:
- renumbered R42 to R39, R39 to R40, R40 to R41, R41 to R42, R49 to R43, R46 to R44, R43 to R45, R44 to R46, R45 to R47, R50 to R48
Changed lines of the file:
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@@
   (symbol (lib_id "Device:R") (at 196.85 76.2 90) (unit 1)
     (in_bom yes) (on_board yes) (dnp no) (fields_autoplaced)
-    (property "Reference" "R45" (at 196.85 69.85 90)
+    (property "Reference" "R47" (at 196.85 69.85 90)
       (effects (font (size 1.27 1.27)))
     )
@@
       (project "main-ECU-board"
         (path "/10edd9b6-c7a8-40f4-bfe3-c9724324d30f/2f8be702-5d98-41c6-b186-35624bc097b2"
-          (reference "R45") (unit 1)
+          (reference "R47") (unit 1)
         )
       )
@@
   (symbol (lib_id "Device:R") (at 88.9 107.95 0) (unit 1)
     (in_bom yes) (on_board yes) (dnp no) (fields_autoplaced)
-    (property "Reference" "R49" (at 91.44 106.68 0)
+    (property "Reference" "R43" (at 91.44 106.68 0)
       (effects (font (size 1.27 1.27)) (justify left))
     )
@@
       (project "main-ECU-board"
         (path "/10edd9b6-c7a8-40f4-bfe3-c9724324d30f/2f8be702-5d98-41c6-b186-35624bc097b2"
-          (reference "R49") (unit 1)
+          (reference "R43") (unit 1)
         )
       )
@@
   (symbol (lib_id "Device:R") (at 190.5 95.25 0) (unit 1)
     (in_bom yes) (on_board yes) (dnp no) (fields_autoplaced)
-    (property "Reference" "R46" (at 193.04 93.98 0)
+    (property "Reference" "R44" (at 193.04 93.98 0)
       (effects (font (size 1.27 1.27)) (justify left))
     )
@@
       (project "main-ECU-board"
         (path "/10edd9b6-c7a8-40f4-bfe3-c9724324d30f/2f8be702-5d98-41c6-b186-35624bc097b2"
-          (reference "R46") (unit 1)
+          (reference "R44") (unit 1)
         )
       )
@@
   (symbol (lib_id "power:GND") (at 101.6 114.3 0) (unit 1)
     (in_bom yes) (on_board yes) (dnp no) (fields_autoplaced)
-    (property "Reference" "#PWR092" (at 101.6 120.65 0)
+    (property "Reference" "#PWR084" (at 101.6 120.65 0)
       (effects (font (size 1.27 1.27)) hide)
     )
@@
       (project "main-ECU-board"
         (path "/10edd9b6-c7a8-40f4-bfe3-c9724324d30f/2f8be702-5d98-41c6-b186-35624bc097b2"
-          (reference "#PWR092") (unit 1)
+          (reference "#PWR084") (unit 1)
         )
       )
@@
   (symbol (lib_id "Device:R") (at 82.55 50.8 90) (unit 1)
     (in_bom yes) (on_board yes) (dnp no) (fields_autoplaced)
-    (property "Reference" "R39" (at 82.55 44.45 90)
+    (property "Reference" "R40" (at 82.55 44.45 90)
       (effects (font (size 1.27 1.27)))
     )
@@
       (project "main-ECU-board"
         (path "/10edd9b6-c7a8-40f4-bfe3-c9724324d30f/2f8be702-5d98-41c6-b186-35624bc097b2"
-          (reference "R39") (unit 1)
+          (reference "R40") (unit 1)
         )
       )
@@
   (symbol (lib_id "Device:R") (at 203.2 107.95 0) (unit 1)
     (in_bom yes) (on_board yes) (dnp no) (fields_autoplaced)
-    (property "Reference" "R50" (at 205.74 106.68 0)
+    (property "Reference" "R48" (at 205.74 106.68 0)
       (effects (font (size 1.27 1.27)) (justify left))
     )
@@
       (project "main-ECU-board"
         (path "/10edd9b6-c7a8-40f4-bfe3-c9724324d30f/2f8be702-5d98-41c6-b186-35624bc097b2"
-          (reference "R50") (unit 1)
+          (reference "R48") (unit 1)
         )
       )
@@
   (symbol (lib_id "Device:R") (at 76.2 95.25 0) (unit 1)
     (in_bom yes) (on_board yes) (dnp no) (fields_autoplaced)
-    (property "Reference" "R42" (at 78.74 93.98 0)
+    (property "Reference" "R39" (at 78.74 93.98 0)
       (effects (font (size 1.27 1.27)) (justify left))
     )
@@
       (project "main-ECU-board"
         (path "/10edd9b6-c7a8-40f4-bfe3-c9724324d30f/2f8be702-5d98-41c6-b186-35624bc097b2"
+          (reference "R39") (unit 1)
+        )
+      )
+    )
+  )
+  (symbol (lib_id "Device:R") (at 82.55 76.2 90) (unit 1)
+    (in_bom yes) (on_board yes) (dnp no) (fields_autoplaced)
+    (property "Reference" "R42" (at 82.55 69.85 90)
+      (effects (font (size 1.27 1.27)))
+    )
+    (property "Value" "10k" (at 82.55 72.39 90)
+      (effects (font (size 1.27 1.27)))
+    )
+    (property "Footprint" "" (at 82.55 77.978 90)
+      (effects (font (size 1.27 1.27)) hide)
+    )
+    (property "Datasheet" "~" (at 82.55 76.2 0)
+      (effects (font (size 1.27 1.27)) hide)
+    )
+    (pin "1")
+    (pin "2")
+    (instances
+      (project "main-ECU-board"
+        (path "/10edd9b6-c7a8-40f4-bfe3-c9724324d30f/2f8be702-5d98-41c6-b186-35624bc097b2"
           (reference "R42") (unit 1)
         )
@@
     )
   )
-  (symbol (lib_id "Device:R") (at 82.55 76.2 90) (unit 1)
-    (in_bom yes) (on_board yes) (dnp no) (fields_autoplaced)
-    (property "Reference" "R41" (at 82.55 69.85 90)
-      (effects (font (size 1.27 1.27)))
-    )
-    (property "Value" "10k" (at 82.55 72.39 90)
-      (effects (font (size 1.27 1.27)))
-    )
-    (property "Footprint" "" (at 82.55 77.978 90)
-      (effects (font (size 1.27 1.27)) hide)
-    )
-    (property "Datasheet" "~" (at 82.55 76.2 0)
-      (effects (font (size 1.27 1.27)) hide)
-    )
-    (pin "1")
-    (pin "2")
-    (instances
-      (project "main-ECU-board"
-        (path "/10edd9b6-c7a8-40f4-bfe3-c9724324d30f/2f8be702-5d98-41c6-b186-35624bc097b2"
-          (reference "R41") (unit 1)
-        )
-      )
-    )
-  )
   (symbol (lib_id "power:GND") (at 134.62 106.68 0) (unit 1)
     (in_bom yes) (on_board yes) (dnp no) (fields_autoplaced)
@@
   (symbol (lib_id "Device:R") (at 196.85 63.5 90) (unit 1)
     (in_bom yes) (on_board yes) (dnp no) (fields_autoplaced)
-    (property "Reference" "R44" (at 196.85 57.15 90)
+    (property "Reference" "R46" (at 196.85 57.15 90)
       (effects (font (size 1.27 1.27)))
     )
@@
       (project "main-ECU-board"
         (path "/10edd9b6-c7a8-40f4-bfe3-c9724324d30f/2f8be702-5d98-41c6-b186-35624bc097b2"
-          (reference "R44") (unit 1)
+          (reference "R46") (unit 1)
         )
       )
@@
   (symbol (lib_id "Device:R") (at 196.85 50.8 90) (unit 1)
     (in_bom yes) (on_board yes) (dnp no) (fields_autoplaced)
-    (property "Reference" "R43" (at 196.85 44.45 90)
+    (property "Reference" "R45" (at 196.85 44.45 90)
       (effects (font (size 1.27 1.27)))
     )
@@
       (project "main-ECU-board"
         (path "/10edd9b6-c7a8-40f4-bfe3-c9724324d30f/2f8be702-5d98-41c6-b186-35624bc097b2"
-          (reference "R43") (unit 1)
+          (reference "R45") (unit 1)
         )
       )
@@
   (symbol (lib_id "Device:R") (at 82.55 63.5 90) (unit 1)
     (in_bom yes) (on_board yes) (dnp no) (fields_autoplaced)
-    (property "Reference" "R40" (at 82.55 57.15 90)
+    (property "Reference" "R41" (at 82.55 57.15 90)
       (effects (font (size 1.27 1.27)))
     )
@@
       (project "main-ECU-board"
         (path "/10edd9b6-c7a8-40f4-bfe3-c9724324d30f/2f8be702-5d98-41c6-b186-35624bc097b2"
-          (reference "R40") (unit 1)
+          (reference "R41") (unit 1)
         )
       )
@@
   (symbol (lib_id "power:GND") (at 215.9 114.3 0) (unit 1)
     (in_bom yes) (on_board yes) (dnp no) (fields_autoplaced)
-    (property "Reference" "#PWR091" (at 215.9 120.65 0)
+    (property "Reference" "#PWR088" (at 215.9 120.65 0)
       (effects (font (size 1.27 1.27)) hide)
     )
@@
       (project "main-ECU-board"
         (path "/10edd9b6-c7a8-40f4-bfe3-c9724324d30f/2f8be702-5d98-41c6-b186-35624bc097b2"
-          (reference "#PWR091") (unit 1)
-        )
-      )
+          (reference "#PWR088") (unit 1)
+        )
+      )

Commit message: modify constant, add 発注先 and footprint
Parts:
- D10, D9: 発注先 (none) -> 秋月電子
- IC3, IC4: 発注先 (none) -> Digi-Key
- R35, R36, R37, R38, R40, R41, R42, R45, R46, R47: value 10k -> 15k; footprint (none) -> Resistor_SMD:R_0603_1608Metric; 発注先 (none) -> Digi-Key
- R39, R43, R44, R48: footprint (none) -> Resistor_SMD:R_0603_1608Metric; 発注先 (none) -> Digi-Key
Changed lines of the file:
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@@
       (effects (font (size 1.27 1.27)))
     )
-    (property "Value" "10k" (at 196.85 72.39 90)
-      (effects (font (size 1.27 1.27)))
-    )
-    (property "Footprint" "" (at 196.85 77.978 90)
+    (property "Value" "15k" (at 196.85 72.39 90)
+      (effects (font (size 1.27 1.27)))
+    )
+    (property "Footprint" "Resistor_SMD:R_0603_1608Metric" (at 196.85 77.978 90)
       (effects (font (size 1.27 1.27)) hide)
     )
@@
       (effects (font (size 1.27 1.27)) hide)
     )
+    (property "発注先" "Digi-Key" (at 196.85 76.2 0)
+      (effects (font (size 1.27 1.27)) hide)
+    )
     (pin "1")
     (pin "2")
@@
       (effects (font (size 1.27 1.27)) (justify left))
     )
-    (property "Footprint" "" (at 87.122 107.95 90)
+    (property "Footprint" "Resistor_SMD:R_0603_1608Metric" (at 87.122 107.95 90)
       (effects (font (size 1.27 1.27)) hide)
     )
@@
       (effects (font (size 1.27 1.27)) hide)
     )
+    (property "発注先" "Digi-Key" (at 88.9 107.95 0)
+      (effects (font (size 1.27 1.27)) hide)
+    )
     (pin "1")
     (pin "2")
@@
       (effects (font (size 1.27 1.27)) (justify left))
     )
-    (property "Footprint" "" (at 188.722 95.25 90)
+    (property "Footprint" "Resistor_SMD:R_0603_1608Metric" (at 188.722 95.25 90)
       (effects (font (size 1.27 1.27)) hide)
     )
@@
       (effects (font (size 1.27 1.27)) hide)
     )
+    (property "発注先" "Digi-Key" (at 190.5 95.25 0)
+      (effects (font (size 1.27 1.27)) hide)
+    )
     (pin "1")
     (pin "2")
@@
       (effects (font (size 1.27 1.27)) (justify left))
     )
-    (property "Value" "10k" (at 53.34 121.92 0)
-      (effects (font (size 1.27 1.27)) (justify left))
-    )
-    (property "Footprint" "" (at 49.022 120.65 90)
+    (property "Value" "15k" (at 53.34 121.92 0)
+      (effects (font (size 1.27 1.27)) (justify left))
+    )
+    (property "Footprint" "Resistor_SMD:R_0603_1608Metric" (at 49.022 120.65 90)
       (effects (font (size 1.27 1.27)) hide)
     )
@@
       (effects (font (size 1.27 1.27)) hide)
     )
+    (property "発注先" "Digi-Key" (at 50.8 120.65 0)
+      (effects (font (size 1.27 1.27)) hide)
+    )
     (pin "1")
     (pin "2")
@@
       (effects (font (size 1.27 1.27)))
     )
-    (property "Value" "10k" (at 82.55 46.99 90)
-      (effects (font (size 1.27 1.27)))
-    )
-    (property "Footprint" "" (at 82.55 52.578 90)
+    (property "Value" "15k" (at 82.55 46.99 90)
+      (effects (font (size 1.27 1.27)))
+    )
+    (property "Footprint" "Resistor_SMD:R_0603_1608Metric" (at 82.55 52.578 90)
       (effects (font (size 1.27 1.27)) hide)
     )
@@
       (effects (font (size 1.27 1.27)) hide)
     )
+    (property "発注先" "Digi-Key" (at 82.55 50.8 0)
+      (effects (font (size 1.27 1.27)) hide)
+    )
     (pin "1")
     (pin "2")
@@
       (effects (font (size 1.27 1.27)) (justify left))
     )
-    (property "Footprint" "" (at 201.422 107.95 90)
+    (property "Footprint" "Resistor_SMD:R_0603_1608Metric" (at 201.422 107.95 90)
       (effects (font (size 1.27 1.27)) hide)
     )
     (property "Datasheet" "~" (at 203.2 107.95 0)
+      (effects (font (size 1.27 1.27)) hide)
+    )
+    (property "発注先" "Digi-Key" (at 203.2 107.95 0)
       (effects (font (size 1.27 1.27)) hide)
     )
@@
       (effects (font (size 1.27 1.27)) hide)
     )
+    (property "発注先" "秋月電子" (at 101.6 107.95 0)
+      (effects (font (size 1.27 1.27)) hide)
+    )
     (pin "1")
     (pin "2")
@@
       (effects (font (size 1.27 1.27)) (justify left))
     )
-    (property "Footprint" "" (at 74.422 95.25 90)
+    (property "Footprint" "Resistor_SMD:R_0603_1608Metric" (at 74.422 95.25 90)
       (effects (font (size 1.27 1.27)) hide)
     )
@@
       (effects (font (size 1.27 1.27)) hide)
     )
+    (property "発注先" "Digi-Key" (at 76.2 95.25 0)
+      (effects (font (size 1.27 1.27)) hide)
+    )
     (pin "1")
     (pin "2")
@@
       (effects (font (size 1.27 1.27)))
     )
-    (property "Value" "10k" (at 82.55 72.39 90)
-      (effects (font (size 1.27 1.27)))
-    )
-    (property "Footprint" "" (at 82.55 77.978 90)
+    (property "Value" "15k" (at 82.55 72.39 90)
+      (effects (font (size 1.27 1.27)))
+    )
+    (property "Footprint" "Resistor_SMD:R_0603_1608Metric" (at 82.55 77.978 90)
       (effects (font (size 1.27 1.27)) hide)
     )
@@
       (effects (font (size 1.27 1.27)) hide)
     )
+    (property "発注先" "Digi-Key" (at 82.55 76.2 0)
+      (effects (font (size 1.27 1.27)) hide)
+    )
     (pin "1")
     (pin "2")
@@
       (effects (font (size 1.27 1.27)))
     )
-    (property "Value" "10k" (at 196.85 59.69 90)
-      (effects (font (size 1.27 1.27)))
-    )
-    (property "Footprint" "" (at 196.85 65.278 90)
+    (property "Value" "15k" (at 196.85 59.69 90)
+      (effects (font (size 1.27 1.27)))
+    )
+    (property "Footprint" "Resistor_SMD:R_0603_1608Metric" (at 196.85 65.278 90)
       (effects (font (size 1.27 1.27)) hide)
     )
@@
       (effects (font (size 1.27 1.27)) hide)
     )
+    (property "発注先" "Digi-Key" (at 196.85 63.5 0)
+      (effects (font (size 1.27 1.27)) hide)
+    )
     (pin "1")
     (pin "2")
@@
     (property "Arrow Price/Stock" "https://www.arrow.com/en/products/tps2h160aqpwprq1/texas-instruments" (at 128.27 91.44 0)
       (effects (font (size 1.27 1.27)) (justify left) hide)
+    )
+    (property "発注先" "Digi-Key" (at 96.52 71.12 0)
+      (effects (font (size 1.27 1.27)) hide)
     )
     (pin "1")
@@
       (effects (font (size 1.27 1.27)) (justify left))
     )
-    (property "Value" "10k" (at 53.34 147.32 0)
-      (effects (font (size 1.27 1.27)) (justify left))
-    )
-    (property "Footprint" "" (at 49.022 146.05 90)
+    (property "Value" "15k" (at 53.34 147.32 0)
+      (effects (font (size 1.27 1.27)) (justify left))
+    )
+    (property "Footprint" "Resistor_SMD:R_0603_1608Metric" (at 49.022 146.05 90)
       (effects (font (size 1.27 1.27)) hide)
     )
@@
       (effects (font (size 1.27 1.27)) hide)
     )
+    (property "発注先" "Digi-Key" (at 50.8 146.05 0)
+      (effects (font (size 1.27 1.27)) hide)
+    )
     (pin "1")
     (pin "2")
@@
       (effects (font (size 1.27 1.27)))
     )
-    (property "Value" "10k" (at 196.85 46.99 90)
-      (effects (font (size 1.27 1.27)))
-    )
-    (property "Footprint" "" (at 196.85 52.578 90)
+    (property "Value" "15k" (at 196.85 46.99 90)
+      (effects (font (size 1.27 1.27)))
+    )
+    (property "Footprint" "Resistor_SMD:R_0603_1608Metric" (at 196.85 52.578 90)
       (effects (font (size 1.27 1.27)) hide)
     )
@@
       (effects (font (size 1.27 1.27)) hide)
     )
+    (property "発注先" "Digi-Key" (at 196.85 50.8 0)
+      (effects (font (size 1.27 1.27)) hide)
+    )
     (pin "1")
     (pin "2")
@@
       (effects (font (size 1.27 1.27)))
     )
-    (property "Value" "10k" (at 44.45 123.19 90)
-      (effects (font (size 1.27 1.27)))
-    )
-    (property "Footprint" "" (at 44.45 125.222 90)
+    (property "Value" "15k" (at 44.45 123.19 90)
+      (effects (font (size 1.27 1.27)))
+    )
+    (property "Footprint" "Resistor_SMD:R_0603_1608Metric" (at 44.45 125.222 90)
       (effects (font (size 1.27 1.27)) hide)
     )
     (property "Datasheet" "~" (at 44.45 127 0)
+      (effects (font (size 1.27 1.27)) hide)
+    )
+    (property "発注先" "Digi-Key" (at 44.45 127 0)
       (effects (font (size 1.27 1.27)) hide)
     )
@@
       (effects (font (size 1.27 1.27)) hide)
     )
+    (property "発注先" "秋月電子" (at 215.9 107.95 0)
+      (effects (font (size 1.27 1.27)) hide)
+    )
     (pin "1")
     (pin "2")
@@
       (effects (font (size 1.27 1.27)))
     )
-    (property "Value" "10k" (at 82.55 59.69 90)
-      (effects (font (size 1.27 1.27)))
-    )
-    (property "Footprint" "" (at 82.55 65.278 90)
+    (property "Value" "15k" (at 82.55 59.69 90)
+      (effects (font (size 1.27 1.27)))
+    )
+    (property "Footprint" "Resistor_SMD:R_0603_1608Metric" (at 82.55 65.278 90)
       (effects (font (size 1.27 1.27)) hide)
     )
@@
       (effects (font (size 1.27 1.27)) hide)
     )
+    (property "発注先" "Digi-Key" (at 82.55 63.5 0)
+      (effects (font (size 1.27 1.27)) hide)
+    )
     (pin "1")
     (pin "2")
@@
       (effects (font (size 1.27 1.27)))
     )
-    (property "Value" "10k" (at 44.45 148.59 90)
-      (effects (font (size 1.27 1.27)))
-    )
-    (property "Footprint" "" (at 44.45 154.178 90)
+    (property "Value" "15k" (at 44.45 148.59 90)
+      (effects (font (size 1.27 1.27)))
+    )
+    (property "Footprint" "Resistor_SMD:R_0603_1608Metric" (at 44.45 154.178 90)
       (effects (font (size 1.27 1.27)) hide)
     )
@@
       (effects (font (size 1.27 1.27)) hide)
     )
+    (property "発注先" "Digi-Key" (at 44.45 152.4 0)
+      (effects (font (size 1.27 1.27)) hide)
+    )
     (pin "1")
     (pin "2")
@@
       (effects (font (size 1.27 1.27)) (justify left) hide)
     )
-    (pin "1")
+    (property "発注先" "Digi-Key" (at 210.82 71.12 0)
+      (effects (font (size 1.27 1.27)) hide)
+    )
+    (pin "1")

Commit message: サーマルパッドの接続先変更
Connections:
- net GND: no longer IC3.17 (EP), IC4.17 (EP)
- net at D9.2 (A), IC3.8 (GND), R43.1: now also IC3.17 (EP)
- net at D10.2 (A), IC4.8 (GND), R48.1: now also IC4.17 (EP)
Other:
- moved on the sheet: D10, D9, R43, R48

Commit message: Arduino header削除、ピンアサイン修正
ハイサイドスイッチ信号、UARTなど
Arduino互換ピンはXHで出す
回路図一部修正
パターン削除、部品配置
Parts:
- renumbered R35 to R36, R36 to R37, R37 to R38, R38 to R39, R39 to R40, R40 to R41, R41 to R42, R42 to R43, R43 to R44, R44 to R45, R45 to R46, R46 to R47, R47 to R48, R48 to R49

Commit message: シャットダウン検知をMOSFETから分圧回路に変更、リファレンス指定子"IC?"を"U?"に変更
Parts:
- renumbered IC3 to U4, IC4 to U5
Changed lines of the file:
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@@
   (symbol (lib_id "SamacSys_Parts:TPS2H160AQPWPRQ1") (at 96.52 71.12 0) (unit 1)
     (in_bom yes) (on_board yes) (dnp no) (fields_autoplaced)
-    (property "Reference" "IC3" (at 114.3 63.5 0)
+    (property "Reference" "U4" (at 114.3 63.5 0)
       (effects (font (size 1.27 1.27)))
     )
@@
       (project "main-ECU-board"
         (path "/10edd9b6-c7a8-40f4-bfe3-c9724324d30f/2f8be702-5d98-41c6-b186-35624bc097b2"
-          (reference "IC3") (unit 1)
+          (reference "U4") (unit 1)
         )
       )
@@
   (symbol (lib_id "SamacSys_Parts:TPS2H160AQPWPRQ1") (at 210.82 71.12 0) (unit 1)
     (in_bom yes) (on_board yes) (dnp no) (fields_autoplaced)
-    (property "Reference" "IC4" (at 228.6 63.5 0)
+    (property "Reference" "U5" (at 228.6 63.5 0)
       (effects (font (size 1.27 1.27)))
     )
@@
       (project "main-ECU-board"
         (path "/10edd9b6-c7a8-40f4-bfe3-c9724324d30f/2f8be702-5d98-41c6-b186-35624bc097b2"
-          (reference "IC4") (unit 1)
-        )
-      )
+          (reference "U5") (unit 1)
+        )
+      )
