File: main-ECU-board.kicad_pcb (KiCad board)
At the start: 2 copper layers, 4 parts, among them J1 Power, J2 Analog, J3 Digital/PWM, J4 Digital/PWM

Commit message: add, modify
Parts:
- added ?: , , F.Cu at (238.8, 101.6)
Other:
- board text added: "ICSP"
Changed lines of the file:
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@@
     )
   )
+  (footprint "" (layer "F.Cu")
+    (at 238.76 101.6)
+    (fp_text reference "" (at 0 0) (layer "F.SilkS")
+        (effects (font (size 1.27 1.27) (thickness 0.15)))
+    )
+    (fp_text value "" (at 0 0) (layer "F.SilkS")
+        (effects (font (size 1.27 1.27) (thickness 0.15)))
+    )
+    (pad "8" thru_hole oval (at 0 0 90) (size 1.7 1.7) (drill 1) (layers "*.Cu" "*.Mask")
+      (pinfunction "Pin_8") (pintype "passive+no_connect"))
+  )
+  (gr_rect (start 237.617 120.65) (end 242.697 128.27)
+    (stroke (width 0.15) (type solid)) (fill none) (layer "Dwgs.User"))
+  (gr_text "ICSP" (at 240.157 124.46 90) (layer "Dwgs.User")
+    (effects (font (size 1 1) (thickness 0.15)))
+  )
 )

Commit message: 回路図からフットプリント追加、Arduinoピン修正
Parts:
- removed ?: , 
- added C1: 10u, Capacitor_SMD:C_0805_2012Metric, F.Cu at (134.3, 144.8)
- added C10: 0.1u, Capacitor_SMD:C_0603_1608Metric, F.Cu at (147.8, 136.4)
- added C11: 0.1u, Capacitor_SMD:C_0603_1608Metric, F.Cu at (157.7, 102.2)
- added C12: 0.1u, Capacitor_SMD:C_0603_1608Metric, F.Cu at (157.7, 104.7)
- added C13: 8p, Capacitor_SMD:C_0402_1005Metric, F.Cu at (122.1, 154.2)
- added C14: 8p, Capacitor_SMD:C_0402_1005Metric, F.Cu at (122.1, 156.2)
- added C15: 4.7u, Capacitor_SMD:C_0805_2012Metric, F.Cu at (110.3, 149.2)
- added C16: 0.1u, Capacitor_SMD:C_0603_1608Metric, F.Cu at (105.4, 131.4)
- added C17: 0.1u, Capacitor_SMD:C_0603_1608Metric, F.Cu at (105.4, 133.9)
- added C18: 1u, Capacitor_SMD:C_0603_1608Metric, F.Cu at (105.4, 136.4)
- added C19: 4.7u, Capacitor_SMD:C_0805_2012Metric, F.Cu at (110.3, 152.3)
- added C2: 10u, Capacitor_SMD:C_0805_2012Metric, F.Cu at (134.3, 147.8)
- added C20: 0.1u, Capacitor_SMD:C_0603_1608Metric, F.Cu at (105.4, 139.0)
- added C21: 0.1u, Capacitor_SMD:C_0603_1608Metric, F.Cu at (105.4, 141.5)
- added C22: 0.1u, Capacitor_SMD:C_0603_1608Metric, F.Cu at (105.4, 144.0)
- added C23: 0.1u, Capacitor_SMD:C_0603_1608Metric, F.Cu at (140.6, 112.1)
- added C24: 0.1u, Capacitor_SMD:C_0603_1608Metric, F.Cu at (140.6, 114.6)
- added C25: 0.1u, Capacitor_SMD:C_0603_1608Metric, F.Cu at (140.6, 117.2)
- added C3: 0.1u, Capacitor_SMD:C_0603_1608Metric, F.Cu at (147.8, 131.4)
- added C4: 33n, Capacitor_SMD:C_0402_1005Metric, F.Cu at (155.1, 144.3)
- added C5: 47u, Capacitor_SMD:CP_Elec_6.3x5.4_Nichicon, F.Cu at (141.7, 147.3)
- added C6: 0.1u, Capacitor_SMD:C_0603_1608Metric, F.Cu at (147.8, 133.9)
- added C7: 47p, Capacitor_SMD:C_0402_1005Metric, F.Cu at (155.1, 146.2)
- added C8: 22u, Capacitor_SMD:C_0805_2012Metric, F.Cu at (134.3, 150.8)
- added C9: 22u, Capacitor_SMD:C_0805_2012Metric, F.Cu at (134.3, 153.8)
- added D1: UDZVTE-175.1B, Diode_SMD:D_SOD-323_HandSoldering, F.Cu at (149.5, 153.5)
- added D10: RB160M-30TR, Diode_SMD:D_SOD-123F, F.Cu at (167.4, 97.2)
- added D2: CUHS20S30, SamacSys_Parts:CUHS20S40H3F, F.Cu at (150.8, 145.5)
- added D3: LED_R, LED_SMD:LED_0603_1608Metric, F.Cu at (154.6, 153.5)
- added D4: NUP2105L, Package_TO_SOT_SMD:SOT-23, F.Cu at (162.2, 109.7)
- added D5: LED_G, LED_SMD:LED_0603_1608Metric, F.Cu at (128.0, 146.0)
- added D6: LED_G, LED_SMD:LED_0603_1608Metric, F.Cu at (128.0, 148.6)
- added D7: LED_G, LED_SMD:LED_0603_1608Metric, F.Cu at (128.0, 151.2)
- added D8: PRTR5V0U2X_215, digikey-footprints:TO-253-4, F.Cu at (110.1, 122.8)
- added D9: RB160M-30TR, Diode_SMD:D_SOD-123F, F.Cu at (167.4, 93.9)
- added F1: MF-USHT020KX-2, Fuse:Fuse_1210_3225Metric, F.Cu at (149.8, 149.9)
- added FB1: BLM18PG471SN1D, digikey-footprints:0603, F.Cu at (127.8, 153.7)
- added FB2: BLM18PG471SN1D, digikey-footprints:0603, F.Cu at (127.8, 156.2)
- added IC1: TCAN1042DQ1, ProjectEV-kicad-library:SOIC127P600X175-8N, F.Cu at (164.0, 104.2)
- added IC2: R7FA4M1AB3CFM#AA0, ProjectEV-kicad-library:QFP50P1200X1200X170-64N, F.Cu at (122.7, 137.4)
- added IC3: TPS2H160AQPWPRQ1, ProjectEV-kicad-library:SOP65P640X120-17N, F.Cu at (160.2, 83.1)
- added IC4: TPS2H160AQPWPRQ1, ProjectEV-kicad-library:SOP65P640X120-17N, F.Cu at (160.2, 89.9)
- added J10: Conn_01x02_Pin, Connector_JST:JST_XH_B2B-XH-A_1x02_P2.50mm_Vertical, F.Cu at (118.8, 114.2)
- added J11: Conn_01x04_Pin, Connector_JST:JST_XH_B4B-XH-A_1x04_P2.50mm_Vertical, F.Cu at (142.1, 98.7)
- added J12: Conn_01x04_Pin, Connector_JST:JST_XH_B4B-XH-A_1x04_P2.50mm_Vertical, F.Cu at (142.1, 106.5)
- added J13: Conn_01x06_Pin, Connector_JST:JST_XH_B6B-XH-A_1x06_P2.50mm_Vertical, F.Cu at (118.8, 90.8)
- added J14: Conn_02x05_Odd_Even, Connector_PinHeader_2.54mm:PinHeader_2x05_P2.54mm_Vertical, F.Cu at (137.1, 82.0)
- added J15: Power, Connector_PinSocket_2.54mm:PinSocket_1x08_P2.54mm_Vertical, F.Cu at (220.0, 150.0)
- added J16: Analog, Connector_PinSocket_2.54mm:PinSocket_1x06_P2.54mm_Vertical, F.Cu at (242.9, 150.0)
- added J17: Conn_02x03_Odd_Even, Connector_PinHeader_2.54mm:PinHeader_2x03_P2.54mm_Vertical, F.Cu at (110.3, 113.2)
- added J18: Digital/PWM, Connector_PinSocket_2.54mm:PinSocket_1x10_P2.54mm_Vertical, F.Cu at (210.9, 101.7)
- added J19: Digital/PWM, Connector_PinSocket_2.54mm:PinSocket_1x08_P2.54mm_Vertical, F.Cu at (237.8, 101.7)
- added J5: Conn_01x03_Pin, Connector_JST:JST_XH_B3B-XH-A_1x03_P2.50mm_Vertical, F.Cu at (106.9, 98.7)
- added J6: Conn_01x03_Pin, Connector_JST:JST_XH_B3B-XH-A_1x03_P2.50mm_Vertical, F.Cu at (106.9, 106.5)
- added J7: Conn_01x02_Pin, Connector_JST:JST_XH_B2B-XH-A_1x02_P2.50mm_Vertical, F.Cu at (118.8, 98.7)
- added J8: Conn_01x02_Pin, Connector_JST:JST_XH_B2B-XH-A_1x02_P2.50mm_Vertical, F.Cu at (118.8, 106.5)
- added J9: Conn_01x06_Pin, Connector_JST:JST_XH_B6B-XH-A_1x06_P2.50mm_Vertical, F.Cu at (118.8, 83.0)
- added L1: 6.8u, ProjectEV-kicad-library:NR10050T150M, F.Cu at (138.9, 136.7)
- added Q1: AO3401A, Package_TO_SOT_SMD:SOT-23, F.Cu at (155.0, 150.0)
- added Q2: 2N7002K, Package_TO_SOT_SMD:SOT-23, F.Cu at (162.2, 120.2)
- added R1: 430k, Resistor_SMD:R_0603_1608Metric, F.Cu at (147.8, 139.0)
- added R10: 60.4, Resistor_SMD:R_0603_1608Metric, F.Cu at (157.7, 112.2)
- added R11: 60.4, Resistor_SMD:R_0603_1608Metric, F.Cu at (157.7, 114.7)
- added R12: 5.1k, Resistor_SMD:R_0603_1608Metric, F.Cu at (105.4, 146.5)
- added R13: 5.1k, Resistor_SMD:R_0603_1608Metric, F.Cu at (109.4, 131.4)
- added R14: 5.1k, Resistor_SMD:R_0603_1608Metric, F.Cu at (109.4, 133.9)
- added R15: 5.1k, Resistor_SMD:R_0603_1608Metric, F.Cu at (109.4, 136.4)
- added R16: 15k, Resistor_SMD:R_0603_1608Metric, F.Cu at (109.4, 139.0)
- added R17: 100k, Resistor_SMD:R_0603_1608Metric, F.Cu at (109.4, 141.5)
- added R18: 13.7k, Resistor_SMD:R_0603_1608Metric, F.Cu at (109.4, 144.0)
- added R19: 300, Resistor_SMD:R_0603_1608Metric, F.Cu at (109.4, 146.5)
- added R2: 51.1k, Resistor_SMD:R_0603_1608Metric, F.Cu at (147.8, 141.5)
- added R20: 15k, Resistor_SMD:R_0603_1608Metric, F.Cu at (113.4, 131.4)
- added R21: 300, Resistor_SMD:R_0603_1608Metric, F.Cu at (113.4, 133.9)
- added R22: 300, Resistor_SMD:R_0603_1608Metric, F.Cu at (113.4, 136.4)
- added R23: 15k, Resistor_SMD:R_0603_1608Metric, F.Cu at (113.4, 139.0)
- added R24: 15k, Resistor_SMD:R_0603_1608Metric, F.Cu at (140.6, 119.7)
- added R25: 15k, Resistor_SMD:R_0603_1608Metric, F.Cu at (140.6, 122.2)
- added R26: 100k, Resistor_SMD:R_0603_1608Metric, F.Cu at (144.6, 112.1)
- added R27: 100k, Resistor_SMD:R_0603_1608Metric, F.Cu at (144.6, 114.6)
- added R28: 100k, Resistor_SMD:R_0603_1608Metric, F.Cu at (144.6, 117.2)
- added R29: 15k, Resistor_SMD:R_0603_1608Metric, F.Cu at (144.6, 119.7)
- added R3: 15k, Resistor_SMD:R_0603_1608Metric, F.Cu at (151.8, 131.4)
- added R30: 15k, Resistor_SMD:R_0603_1608Metric, F.Cu at (144.6, 122.2)
- added R31: 3k, Resistor_SMD:R_0603_1608Metric, F.Cu at (148.6, 112.1)
- added R32: 3k, Resistor_SMD:R_0603_1608Metric, F.Cu at (148.6, 114.6)
- added R33: 3k, Resistor_SMD:R_0603_1608Metric, F.Cu at (148.6, 117.2)
- added R34: 3k, Resistor_SMD:R_0603_1608Metric, F.Cu at (148.6, 119.7)
- added R35: 15k, Resistor_SMD:R_0603_1608Metric, F.Cu at (166.6, 80.9)
- added R36: 15k, Resistor_SMD:R_0603_1608Metric, F.Cu at (166.6, 83.4)
- added R37: 15k, Resistor_SMD:R_0603_1608Metric, F.Cu at (166.6, 86.0)
- added R38: 15k, Resistor_SMD:R_0603_1608Metric, F.Cu at (166.6, 88.5)
- added R39: 1k, Resistor_SMD:R_0603_1608Metric, F.Cu at (166.6, 91.0)
- added R4: 0, Resistor_SMD:R_0603_1608Metric, F.Cu at (151.8, 133.9)
- added R40: 15k, Resistor_SMD:R_0603_1608Metric, F.Cu at (170.6, 80.9)
- added R41: 15k, Resistor_SMD:R_0603_1608Metric, F.Cu at (170.6, 83.4)
- added R42: 15k, Resistor_SMD:R_0603_1608Metric, F.Cu at (170.6, 86.0)
- added R43: 1k, Resistor_SMD:R_0603_1608Metric, F.Cu at (170.6, 88.5)
- added R44: 1k, Resistor_SMD:R_0603_1608Metric, F.Cu at (170.6, 91.0)
- added R45: 15k, Resistor_SMD:R_0603_1608Metric, F.Cu at (174.6, 80.9)
- added R46: 15k, Resistor_SMD:R_0603_1608Metric, F.Cu at (174.6, 83.4)
- added R47: 15k, Resistor_SMD:R_0603_1608Metric, F.Cu at (174.6, 86.0)
- added R48: 1k, Resistor_SMD:R_0603_1608Metric, F.Cu at (174.6, 88.5)
- added R49: 1M, Resistor_SMD:R_0603_1608Metric, F.Cu at (157.7, 119.2)
- added R5: 52.3k, Resistor_SMD:R_0603_1608Metric, F.Cu at (151.8, 136.4)
- added R50: 15k, Resistor_SMD:R_0603_1608Metric, F.Cu at (157.7, 121.8)
- added R6: 10k, Resistor_SMD:R_0603_1608Metric, F.Cu at (151.8, 139.0)
- added R7: 300, Resistor_SMD:R_0603_1608Metric, F.Cu at (151.8, 141.5)
- added R8: 15k, Resistor_SMD:R_0603_1608Metric, F.Cu at (157.7, 107.2)
- added R9: 1k, Resistor_SMD:R_0603_1608Metric, F.Cu at (157.7, 109.7)
- added SW1: SW_MEC_5E, Button_Switch_THT:SW_PUSH_6mm_H7.3mm, F.Cu at (117.5, 146.7)
- added U1: TPS62933, Package_TO_SOT_SMD:SOT-583-8, F.Cu at (138.3, 153.2)
- added Y1: ABM8W-12.0000MHZ-8-K1Z-T3, Crystal:Crystal_SMD_3225-4Pin_3.2x2.5mm, F.Cu at (118.1, 155.4)
- J1: value Power -> Conn_01x02_Pin; footprint Connector_PinSocket_2.54mm:PinSocket_1x08_P2.54mm_Vertical -> Connector_PinHeader_2.54mm:PinHeader_1x02_P2.54mm_Vertical
- J2: value Analog -> USB_C_Receptacle; footprint Connector_PinSocket_2.54mm:PinSocket_1x06_P2.54mm_Vertical -> SamacSys_Parts:5077CR-16-SMC2-BK-TR
- J3: value Digital/PWM -> Conn_01x03_Pin; footprint Connector_PinSocket_2.54mm:PinSocket_1x10_P2.54mm_Vertical -> Connector_JST:JST_XH_B3B-XH-A_1x03_P2.50mm_Vertical
- J4: value Digital/PWM -> Conn_01x03_Pin; footprint Connector_PinSocket_2.54mm:PinSocket_1x08_P2.54mm_Vertical -> Connector_JST:JST_XH_B3B-XH-A_1x03_P2.50mm_Vertical
- moved J4 114.6 mm to (106.9, 90.8), turned to 0 degrees
- moved J2 101.6 mm to (147.9, 85.0), turned to 0 degrees
- moved J1 97.5 mm to (105.7, 150.1), turned to 0 degrees
- moved J3 89.1 mm to (106.9, 83.0), turned to 0 degrees
Connections:
- J1 pad 1: unconnected-(J1-Pin_1-Pad1) -> NC
- J1 pad 2: /IOREF -> GND
- J3 pad 1: /SCL/A5 -> +5V
- J3 pad 2: /SDA/A4 -> A0
- J3 pad 3: /AREF -> GND
- J4 pad 1: /7 -> +5V
- J4 pad 2: /*6 -> A1
- J4 pad 3: /*5 -> GND

Commit message: 機能ごとにざっくり部品配置
Parts:
- SW1: value SW_MEC_5E -> SW_Push
- moved J5 91.1 mm to (182.5, 149.5), turned to 90 degrees
- moved J4 88.0 mm to (172.5, 149.5), turned to 90 degrees
- moved J3 86.0 mm to (161.5, 149.5), turned to 90 degrees
- moved J8 81.5 mm to (195.0, 77.5), turned to 90 degrees
- moved R12 79.1 mm to (172.2, 104.3), turned to 180 degrees
- moved J16 78.3 mm to (165.9, 135.4)
- moved J15 78.3 mm to (143.0, 135.4)
- moved J18 78.3 mm to (133.9, 87.1)
- moved J19 78.3 mm to (160.8, 87.1)
- moved C15 71.5 mm to (163.2, 101.3), turned to -90 degrees
- moved C18 70.6 mm to (169.2, 106.3)
- moved Y1 69.7 mm to (159.0, 99.0)
- moved J7 69.5 mm to (185.0, 77.5), turned to 90 degrees
- moved R19 68.9 mm to (169.2, 112.3), turned to 180 degrees
- moved J17 68.6 mm to (178.7, 107.5)
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Connections:
- J13 pad 3: MOSI/11 -> MISO/12
- J13 pad 4: MISO/12 -> MOSI/11
- R32 pad 2: MOSI/11 -> MISO/12
- R34 pad 2: MISO/12 -> MOSI/11
- SW1 pad 2: GND -> ~{RESET}

Commit message: 部品配置更新
コネクタ、CANあたりはおおよそできた
Parts:
- moved R3 44.4 mm to (110.7, 127.0), turned to 180 degrees
- moved J8 38.5 mm to (157.5, 69.0)
- moved R30 38.5 mm to (152.5, 67.3)
- moved R26 36.5 mm to (158.3, 143.5)
- moved Q1 36.2 mm to (108.0, 123.5), turned to 180 degrees
- moved F1 35.6 mm to (104.0, 124.9), turned to -90 degrees
- moved C23 32.6 mm to (158.3, 145.5)
- moved D1 26.6 mm to (111.5, 123.5), turned to -90 degrees
- moved R27 25.7 mm to (169.3, 143.5)
- moved D9 23.1 mm to (130.5, 113.5), turned to 180 degrees
- moved C24 21.6 mm to (169.3, 145.5)
- moved C5 21.5 mm to (109.0, 117.0)
- moved J14 19.8 mm to (178.2, 68.8)
- moved J7 18.6 mm to (168.5, 69.0)
- moved R29 18.6 mm to (163.5, 67.3)
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
Commit message: 逆接保護まわり修正
Parts:
- moved J6 10.8 mm to (112.0, 148.0)
- moved F1 8.96 mm to (106.5, 133.5)
- moved Q1 2.97 mm to (105.1, 124.0)
- moved D1 2.97 mm to (108.6, 124.2)
- moved R3 2.28 mm to (108.6, 128.0), turned to -90 degrees
- moved J11 1.06 mm to (123.0, 150.5)
- moved C5 0.58 mm to (108.7, 117.5)
Changed lines of the file:
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@@
   )
   (footprint "Connector_JST:JST_XH_B4B-XH-A_1x04_P2.50mm_Vertical" (layer "F.Cu")
-    (at 121.975 150.75 90)
+    (at 123 150.5 90)
     (descr "JST XH series connector, B4B-XH-A (http://www.jst-mfg.com/product/pdf/eng/eXH.pdf), generated with kicad-footprint-generator")
     (tags "connector JST XH vertical")
@@
   )
   (footprint "Fuse:Fuse_1210_3225Metric" (layer "F.Cu")
-    (at 104 124.9 -90)
+    (at 106.5 133.5 -90)
     (descr "Fuse SMD 1210 (3225 Metric), square (rectangular) end terminal, IPC_7351 nominal, (Body size source: http://www.tortai-tech.com/upload/download/2011102023233369053.pdf), generated with kicad-footprint-generator")
     (tags "fuse")
@@
   )
   (footprint "Package_TO_SOT_SMD:SOT-23" (layer "F.Cu")
-    (at 108 123.5 180)
+    (at 105.0625 123.95 180)
     (descr "SOT, 3 Pin (https://www.jedec.org/system/files/docs/to-236h.pdf variant AB), generated with kicad-footprint-generator ipc_gullwing_generator.py")
     (tags "SOT TO_SOT_SMD")
@@
   )
   (footprint "Connector_JST:JST_XH_B3B-XH-A_1x03_P2.50mm_Vertical" (layer "F.Cu")
-    (at 108 138 90)
+    (at 112 148 90)
     (descr "JST XH series connector, B3B-XH-A (http://www.jst-mfg.com/product/pdf/eng/eXH.pdf), generated with kicad-footprint-generator")
     (tags "connector JST XH vertical")
@@
   )
   (footprint "Diode_SMD:D_SOD-323_HandSoldering" (layer "F.Cu")
-    (at 111.5 123.5 -90)
+    (at 108.625 124.25 -90)
     (descr "SOD-323")
     (tags "SOD-323")
@@
   )
   (footprint "Resistor_SMD:R_0603_1608Metric" (layer "F.Cu")
-    (at 110.675 127 180)
+    (at 108.625 128 -90)
     (descr "Resistor SMD 0603 (1608 Metric), square (rectangular) end terminal, IPC_7351 nominal, (Body size source: IPC-SM-782 page 72, https://www.pcb-3d.com/wordpress/wp-content/uploads/ipc-sm-782a_amendment_1_and_2.pdf), generated with kicad-footprint-generator")
     (tags "resistor")
@@
     (property "発注先" "Digi-Key")
     (attr smd)
-    (fp_text reference "R3" (at 0 -1.43) (layer "F.SilkS")
+    (fp_text reference "R3" (at 0 -1.43 -270) (layer "F.SilkS")
         (effects (font (size 1 1) (thickness 0.15)))
     )
-    (fp_text value "15k" (at 0 1.43) (layer "F.Fab")
+    (fp_text value "15k" (at 0 1.43 -270) (layer "F.Fab")
         (effects (font (size 1 1) (thickness 0.15)))
     )
-    (fp_text user "${REFERENCE}" (at 0 0) (layer "F.Fab")
+    (fp_text user "${REFERENCE}" (at 0 0 -270) (layer "F.Fab")
         (effects (font (size 0.4 0.4) (thickness 0.06)))
     )
@@
     (fp_line (start 0.8 0.4125) (end -0.8 0.4125)
       (stroke (width 0.1) (type solid)) (layer "F.Fab"))
-    (pad "1" smd roundrect (at -0.825 0 180) (size 0.8 0.95) (layers "F.Cu" "F.Paste" "F.Mask") (roundrect_rratio 0.25)
+    (pad "1" smd roundrect (at -0.825 0 270) (size 0.8 0.95) (layers "F.Cu" "F.Paste" "F.Mask") (roundrect_rratio 0.25)
       (net 18 "Net-(D1-A)") (pintype "passive"))
-    (pad "2" smd roundrect (at 0.825 0 180) (size 0.8 0.95) (layers "F.Cu" "F.Paste" "F.Mask") (roundrect_rratio 0.25)
+    (pad "2" smd roundrect (at 0.825 0 270) (size 0.8 0.95) (layers "F.Cu" "F.Paste" "F.Mask") (roundrect_rratio 0.25)
       (net 3 "GND") (pintype "passive"))
     (model "${KICAD6_3DMODEL_DIR}/Resistor_SMD.3dshapes/R_0603_1608Metric.wrl"
@@
   )
   (footprint "Capacitor_SMD:CP_Elec_6.3x5.4_Nichicon" (layer "F.Cu")
-    (at 109 117)
+    (at 108.7 117.5)
     (descr "SMD capacitor, aluminum electrolytic, Nichicon, 6.3x5.4mm")
     (tags "capacitor electrolytic")

Commit message: modify footprint path and 3dmodel path
Parts:
- D2: footprint SamacSys_Parts:CUHS20S40H3F -> ProjectEV-kicad-library:CUHS20S40H3F
- J2: footprint SamacSys_Parts:5077CR-16-SMC2-BK-TR -> ProjectEV-kicad-library:5077CR-16-SMC2-BK-TR
- moved IC4 0.98 mm to (125.0, 135.0)
- moved D10 0.98 mm to (131.0, 128.0)
- moved R44 0.98 mm to (131.0, 132.5)
- moved R45 0.98 mm to (131.0, 138.5)
- moved R46 0.98 mm to (131.0, 136.5)
- moved R47 0.98 mm to (131.0, 134.5)
- moved R48 0.98 mm to (131.0, 130.5)
- moved D9 0.71 mm to (131.0, 113.0)
- moved IC3 0.71 mm to (125.0, 120.0)
- moved R35 0.71 mm to (136.0, 120.5)
- moved R36 0.71 mm to (136.0, 118.5)
- moved R37 0.71 mm to (136.0, 122.5)
- moved R38 0.71 mm to (136.0, 116.5)
- moved R39 0.71 mm to (131.0, 117.5)
- moved R40 0.71 mm to (131.0, 123.5)
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
Commit message: 修正、電源回路のおおよその配置
Parts:
- moved D2 30.9 mm to (116.0, 85.0), turned to 180 degrees
- moved C7 24.6 mm to (119.0, 99.5)
- moved C4 21.3 mm to (121.5, 100.5), turned to 90 degrees
- moved R6 19.9 mm to (119.0, 101.0), turned to 180 degrees
- moved R5 19.9 mm to (119.0, 98.0), turned to 180 degrees
- moved R1 18.1 mm to (118.5, 108.0), turned to 180 degrees
- moved C3 17.3 mm to (123.8, 106.0)
- moved R2 16.8 mm to (118.5, 106.5), turned to 180 degrees
- moved C9 16.0 mm to (142.5, 102.5), turned to -90 degrees
- moved R4 15.8 mm to (123.5, 99.0), turned to 90 degrees
- moved R31 15.5 mm to (134.5, 76.5), turned to 180 degrees
- moved R7 15.0 mm to (151.7, 95.0)
- moved C8 14.8 mm to (140.0, 102.5), turned to -90 degrees
- moved D3 13.2 mm to (151.2, 92.0)
- moved R32 11.5 mm to (144.5, 74.0), turned to 180 degrees
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
Commit message: 電源回路の配置、フットプリント修正
Parts:
- L1: value 6.8u -> 22u; footprint ProjectEV-kicad-library:NR10050T150M -> ProjectEV-kicad-library:L_MGAH0603
- moved R7 13.3 mm to (143.5, 105.5), turned to -90 degrees
- moved D3 12.6 mm to (143.5, 102.0), turned to 90 degrees
- moved C10 3.04 mm to (141.5, 102.0)
- moved C9 3.04 mm to (139.5, 102.0)
- moved C8 2.55 mm to (137.5, 102.0)
- moved L1 2.06 mm to (131.0, 99.5)
- moved C6 1.28 mm to (124.8, 95.5), turned to 0 degrees
- moved R1 1.12 mm to (119.0, 107.0)
- moved R2 1.12 mm to (119.0, 105.5)
- moved R4 0.71 mm to (124.0, 98.5)
- moved C7 0.50 mm to (119.0, 100.0)
- moved R5 0.50 mm to (119.0, 98.5)
- moved R6 0.50 mm to (119.0, 101.5)
