File: main-ECU-board.kicad_pcb (KiCad board)
At the start: 2 copper layers, 117 parts, among them IC1 TCAN1042DQ1, IC2 R7FA4M1AB3CFM#AA0, IC3 TPS2H160AQPWPRQ1, IC4 TPS2H160AQPWPRQ1, J1 Conn_01x02_Pin, J10 Conn_01x02_Pin, J11 Conn_01x04_Pin, J12 Conn_01x04_Pin, J13 Conn_01x06_Pin, J14 Conn_02x05_Odd_Even, J15 Power, J16 Analog, J17 Conn_02x03_Odd_Even, J18 Digital/PWM, J19 Digital/PWM, J2 USB_C_Receptacle, J3 Conn_01x03_Pin, J4 Conn_01x03_Pin, J5 Conn_01x03_Pin, J6 Conn_01x03_Pin, J7 Conn_01x02_Pin, J8 Conn_01x02_Pin, J9 Conn_01x06_Pin, Q1 AO3401A, Q2 2N7002K, SW1 SW_Push, U1 TPS62933, Y1 ABM8W-12.0000MHZ-8-K1Z-T3

Commit message: 電源回路配置修正、AIRなどの駆動回路修正
Parts:
- moved J6 46.2 mm to (108.0, 102.0)
- moved J1 27.8 mm to (108.3, 76.8)
- moved R20 27.8 mm to (113.5, 72.6)
- moved R23 27.8 mm to (113.5, 75.9)
- moved SW1 27.8 mm to (103.8, 67.2)
- moved J11 26.2 mm to (108.0, 129.0)
- moved F1 25.5 mm to (111.5, 108.5), turned to 180 degrees
- moved D9 22.8 mm to (125.2, 135.0)
- moved R42 22.4 mm to (126.7, 141.5)
- moved R43 22.4 mm to (124.7, 137.0)
- moved R39 21.9 mm to (126.7, 139.0)
- moved R41 21.9 mm to (126.7, 143.0)
- moved IC3 21.4 mm to (120.7, 141.0)
- moved R40 21.4 mm to (126.7, 144.5)
- moved Q1 19.2 mm to (116.5, 108.5)
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
Commit message: 部品配置おおよそ終了
Parts:
- moved J4 60.2 mm to (189.0, 93.0)
- moved J9 60.0 mm to (179.0, 79.0)
- moved C24 57.8 mm to (185.0, 89.7), turned to 90 degrees
- moved R27 55.4 mm to (183.0, 89.7), turned to 90 degrees
- moved J3 43.8 mm to (189.0, 121.0)
- moved J5 43.5 mm to (189.0, 107.0)
- moved C25 42.1 mm to (185.0, 103.7), turned to 90 degrees
- moved C23 41.0 mm to (194.0, 122.5)
- moved R26 41.0 mm to (194.1, 120.5)
- moved R28 39.9 mm to (183.0, 103.7), turned to 90 degrees
- moved Q2 24.4 mm to (127.5, 111.0)
- moved R49 22.8 mm to (124.5, 110.9), turned to -90 degrees
- moved R50 21.4 mm to (130.5, 110.2), turned to -90 degrees
- moved IC3 13.7 mm to (130.0, 131.0)
- moved R39 13.7 mm to (136.0, 129.0)
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Connections:
- IC3 pad 17: GND -> Net-(D9-A)
- IC4 pad 17: GND -> Net-(D10-A)
Other:
- board outline added: 100 x 78 mm

Commit message: 電源、ハイサイドスイッチまわり配置修正
Parts:
- moved Q2 10.2 mm to (117.5, 113.0)
- moved R49 10.2 mm to (114.5, 112.9)
- moved R50 10.2 mm to (120.5, 112.2)
- moved D1 8.13 mm to (119.4, 101.8)
- moved Q1 8.13 mm to (115.9, 101.5)
- moved R3 8.13 mm to (119.4, 105.5)
- moved J6 6.52 mm to (107.5, 108.5)
- moved F1 6.46 mm to (115.5, 107.1), turned to -90 degrees
- moved C1 4.03 mm to (137.0, 106.0)
- moved C2 4.03 mm to (137.0, 104.0)
- moved C3 4.03 mm to (136.8, 102.0)
- moved C4 4.03 mm to (134.5, 96.5)
- moved C6 4.03 mm to (136.0, 92.5)
- moved C7 4.03 mm to (132.3, 96.0)
- moved L1 4.03 mm to (142.5, 96.5)
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
Commit message: 電源付近修正
Parts:
- moved F1 12.6 mm to (109.5, 96.0), turned to 180 degrees
- moved R3 6.75 mm to (114.5, 101.0), turned to 180 degrees
- moved Q1 4.75 mm to (118.5, 97.5), turned to 90 degrees
- moved Q2 2.00 mm to (117.5, 111.0)
- moved R49 2.00 mm to (114.5, 110.9)
- moved R50 2.00 mm to (120.5, 110.2)
- moved D1 1.47 mm to (118.2, 101.0), turned to 180 degrees
Changed lines of the file:
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@@
   )
   (footprint "Fuse:Fuse_1210_3225Metric" (layer "F.Cu")
-    (at 115.5 107.1 -90)
+    (at 109.5 96 180)
     (descr "Fuse SMD 1210 (3225 Metric), square (rectangular) end terminal, IPC_7351 nominal, (Body size source: http://www.tortai-tech.com/upload/download/2011102023233369053.pdf), generated with kicad-footprint-generator")
     (tags "fuse")
@@
     (property "発注先" "Digi-Key")
     (attr smd)
-    (fp_text reference "F1" (at 0 -2.28 -270) (layer "F.SilkS")
+    (fp_text reference "F1" (at 0 -2.28) (layer "F.SilkS")
         (effects (font (size 1 1) (thickness 0.15)))
     )
-    (fp_text value "MF-USHT020KX-2" (at 0 2.28 -270) (layer "F.Fab")
+    (fp_text value "MF-USHT020KX-2" (at 0 2.28) (layer "F.Fab")
         (effects (font (size 1 1) (thickness 0.15)))
     )
-    (fp_text user "${REFERENCE}" (at 0 0 -270) (layer "F.Fab")
+    (fp_text user "${REFERENCE}" (at 0 0) (layer "F.Fab")
         (effects (font (size 0.8 0.8) (thickness 0.12)))
     )
@@
     (fp_line (start 1.6 1.25) (end -1.6 1.25)
       (stroke (width 0.1) (type solid)) (layer "F.Fab"))
-    (pad "1" smd roundrect (at -1.4 0 270) (size 1.25 2.65) (layers "F.Cu" "F.Paste" "F.Mask") (roundrect_rratio 0.2)
+    (pad "1" smd roundrect (at -1.4 0 180) (size 1.25 2.65) (layers "F.Cu" "F.Paste" "F.Mask") (roundrect_rratio 0.2)
       (net 31 "Net-(Q1-D)") (pintype "passive"))
-    (pad "2" smd roundrect (at 1.4 0 270) (size 1.25 2.65) (layers "F.Cu" "F.Paste" "F.Mask") (roundrect_rratio 0.2)
+    (pad "2" smd roundrect (at 1.4 0 180) (size 1.25 2.65) (layers "F.Cu" "F.Paste" "F.Mask") (roundrect_rratio 0.2)
       (net 32 "+BATT") (pintype "passive"))
     (model "${KICAD6_3DMODEL_DIR}/Fuse.3dshapes/Fuse_1210_3225Metric.wrl"
@@
   )
   (footprint "Package_TO_SOT_SMD:SOT-23" (layer "F.Cu")
-    (at 115.9375 101.5 180)
+    (at 118.5 97.5 90)
     (descr "SOT, 3 Pin (https://www.jedec.org/system/files/docs/to-236h.pdf variant AB), generated with kicad-footprint-generator ipc_gullwing_generator.py")
     (tags "SOT TO_SOT_SMD")
@@
     (property "発注先" "秋月電子")
     (attr smd)
-    (fp_text reference "Q1" (at 0 -2.4) (layer "F.SilkS")
+    (fp_text reference "Q1" (at 0 -2.4 90) (layer "F.SilkS")
         (effects (font (size 1 1) (thickness 0.15)))
     )
-    (fp_text value "AO3401A" (at 0 2.4) (layer "F.Fab")
+    (fp_text value "AO3401A" (at 0 2.4 90) (layer "F.Fab")
         (effects (font (size 1 1) (thickness 0.15)))
     )
-    (fp_text user "${REFERENCE}" (at 0 0) (layer "F.Fab")
+    (fp_text user "${REFERENCE}" (at 0 0 90) (layer "F.Fab")
         (effects (font (size 0.32 0.32) (thickness 0.05)))
     )
@@
     (fp_line (start 0.65 1.45) (end -0.65 1.45)
       (stroke (width 0.1) (type solid)) (layer "F.Fab"))
-    (pad "1" smd roundrect (at -0.9375 -0.95 180) (size 1.475 0.6) (layers "F.Cu" "F.Paste" "F.Mask") (roundrect_rratio 0.25)
+    (pad "1" smd roundrect (at -0.9375 -0.95 90) (size 1.475 0.6) (layers "F.Cu" "F.Paste" "F.Mask") (roundrect_rratio 0.25)
       (net 18 "Net-(D1-A)") (pinfunction "G") (pintype "input"))
-    (pad "2" smd roundrect (at -0.9375 0.95 180) (size 1.475 0.6) (layers "F.Cu" "F.Paste" "F.Mask") (roundrect_rratio 0.25)
+    (pad "2" smd roundrect (at -0.9375 0.95 90) (size 1.475 0.6) (layers "F.Cu" "F.Paste" "F.Mask") (roundrect_rratio 0.25)
       (net 4 "+12V") (pinfunction "S") (pintype "passive"))
-    (pad "3" smd roundrect (at 0.9375 0 180) (size 1.475 0.6) (layers "F.Cu" "F.Paste" "F.Mask") (roundrect_rratio 0.25)
+    (pad "3" smd roundrect (at 0.9375 0 90) (size 1.475 0.6) (layers "F.Cu" "F.Paste" "F.Mask") (roundrect_rratio 0.25)
       (net 31 "Net-(Q1-D)") (pinfunction "D") (pintype "passive"))
     (model "${KICAD6_3DMODEL_DIR}/Package_TO_SOT_SMD.3dshapes/SOT-23.wrl"
@@
   )
   (footprint "Resistor_SMD:R_0603_1608Metric" (layer "F.Cu")
-    (at 114.5 112.875 -90)
+    (at 114.5 110.875 -90)
     (descr "Resistor SMD 0603 (1608 Metric), square (rectangular) end terminal, IPC_7351 nominal, (Body size source: IPC-SM-782 page 72, https://www.pcb-3d.com/wordpress/wp-content/uploads/ipc-sm-782a_amendment_1_and_2.pdf), generated with kicad-footprint-generator")
     (tags "resistor")
@@
   )
   (footprint "Diode_SMD:D_SOD-323_HandSoldering" (layer "F.Cu")
-    (at 119.4375 101.8 -90)
+    (at 118.2 101 180)
     (descr "SOD-323")
     (tags "SOD-323")
@@
     (property "発注先" "秋月電子")
     (attr smd)
-    (fp_text reference "D1" (at 0 -1.85 90) (layer "F.SilkS")
+    (fp_text reference "D1" (at 0 -1.85) (layer "F.SilkS")
         (effects (font (size 1 1) (thickness 0.15)))
     )
-    (fp_text value "UDZVTE-175.1B" (at 0.1 1.9 90) (layer "F.Fab")
+    (fp_text value "UDZVTE-175.1B" (at 0.1 1.9) (layer "F.Fab")
         (effects (font (size 1 1) (thickness 0.15)))
     )
-    (fp_text user "${REFERENCE}" (at 0 -1.85 90) (layer "F.Fab")
+    (fp_text user "${REFERENCE}" (at 0 -1.85) (layer "F.Fab")
         (effects (font (size 1 1) (thickness 0.15)))
     )
@@
     (fp_line (start 0.9 0.7) (end -0.9 0.7)
       (stroke (width 0.1) (type solid)) (layer "F.Fab"))
-    (pad "1" smd roundrect (at -1.25 0 270) (size 1 1) (layers "F.Cu" "F.Paste" "F.Mask") (roundrect_rratio 0.25)
+    (pad "1" smd roundrect (at -1.25 0 180) (size 1 1) (layers "F.Cu" "F.Paste" "F.Mask") (roundrect_rratio 0.25)
       (net 4 "+12V") (pinfunction "K") (pintype "passive"))
-    (pad "2" smd roundrect (at 1.25 0 270) (size 1 1) (layers "F.Cu" "F.Paste" "F.Mask") (roundrect_rratio 0.25)
+    (pad "2" smd roundrect (at 1.25 0 180) (size 1 1) (layers "F.Cu" "F.Paste" "F.Mask") (roundrect_rratio 0.25)
       (net 18 "Net-(D1-A)") (pinfunction "A") (pintype "passive"))
     (model "${KICAD6_3DMODEL_DIR}/Diode_SMD.3dshapes/D_SOD-323.wrl"
@@
   )
   (footprint "Resistor_SMD:R_0603_1608Metric" (layer "F.Cu")
-    (at 119.4375 105.55 -90)
+    (at 114.45 101 180)
     (descr "Resistor SMD 0603 (1608 Metric), square (rectangular) end terminal, IPC_7351 nominal, (Body size source: IPC-SM-782 page 72, https://www.pcb-3d.com/wordpress/wp-content/uploads/ipc-sm-782a_amendment_1_and_2.pdf), generated with kicad-footprint-generator")
     (tags "resistor")
@@
     (property "発注先" "Digi-Key")
     (attr smd)
-    (fp_text reference "R3" (at 0 -1.492 90) (layer "F.SilkS")
+    (fp_text reference "R3" (at 0 -1.492) (layer "F.SilkS")
         (effects (font (size 1 1) (thickness 0.15)))
     )
-    (fp_text value "15k" (at 0 1.43 90) (layer "F.Fab")
+    (fp_text value "15k" (at 0 1.43) (layer "F.Fab")
         (effects (font (size 1 1) (thickness 0.15)))
     )
-    (fp_text user "${REFERENCE}" (at 0 0 90) (layer "F.Fab")
+    (fp_text user "${REFERENCE}" (at 0 0) (layer "F.Fab")
         (effects (font (size 0.4 0.4) (thickness 0.06)))
     )
@@
     (fp_line (start 0.8 0.4125) (end -0.8 0.4125)
       (stroke (width 0.1) (type solid)) (layer "F.Fab"))
-    (pad "1" smd roundrect (at -0.825 0 270) (size 0.8 0.95) (layers "F.Cu" "F.Paste" "F.Mask") (roundrect_rratio 0.25)
+    (pad "1" smd roundrect (at -0.825 0 180) (size 0.8 0.95) (layers "F.Cu" "F.Paste" "F.Mask") (roundrect_rratio 0.25)
       (net 18 "Net-(D1-A)") (pintype "passive"))
-    (pad "2" smd roundrect (at 0.825 0 270) (size 0.8 0.95) (layers "F.Cu" "F.Paste" "F.Mask") (roundrect_rratio 0.25)
+    (pad "2" smd roundrect (at 0.825 0 180) (size 0.8 0.95) (layers "F.Cu" "F.Paste" "F.Mask") (roundrect_rratio 0.25)
       (net 3 "GND") (pintype "passive"))
     (model "${KICAD6_3DMODEL_DIR}/Resistor_SMD.3dshapes/R_0603_1608Metric.wrl"
@@
   )
   (footprint "Package_TO_SOT_SMD:SOT-23" (layer "F.Cu")
-    (at 117.5 113)
+    (at 117.5 111)
     (descr "SOT, 3 Pin (https://www.jedec.org/system/files/docs/to-236h.pdf variant AB), generated with kicad-footprint-generator ipc_gullwing_generator.py")
     (tags "SOT TO_SOT_SMD")
@@
   )
   (footprint "Resistor_SMD:R_0603_1608Metric" (layer "F.Cu")
-    (at 120.5 112.175 -90)
+    (at 120.5 110.175 -90)
     (descr "Resistor SMD 0603 (1608 Metric), square (rectangular) end terminal, IPC_7351 nominal, (Body size source: IPC-SM-782 page 72, https://www.pcb-3d.com/wordpress/wp-content/uploads/ipc-sm-782a_amendment_1_and_2.pdf), generated with kicad-footprint-generator")
     (tags "resistor")

Commit message: 電源と電源コネクタ、type-cコネクタまわりの配置修正
Parts:
- added REF**: MountingHole_3.2mm_M3_Pad_Via, MountingHole:MountingHole_3.2mm_M3_Pad_Via, F.Cu at (195.0, 133.0)
- added REF**: MountingHole_3.2mm_M3_Pad_Via, MountingHole:MountingHole_3.2mm_M3_Pad_Via, F.Cu at (105.0, 65.0)
- added REF**: MountingHole_3.2mm_M3_Pad_Via, MountingHole:MountingHole_3.2mm_M3_Pad_Via, F.Cu at (105.0, 133.0)
- added REF**: MountingHole_3.2mm_M3_Pad_Via, MountingHole:MountingHole_3.2mm_M3_Pad_Via, F.Cu at (195.0, 65.0)
- added REF**: MountingHole_3.2mm_M3_Pad_Via, MountingHole:MountingHole_3.2mm_M3_Pad_Via, F.Cu at (149.0, 65.0)
- moved SW1 12.9 mm to (114.5, 65.2)
- moved J6 12.5 mm to (107.5, 96.0)
- moved D8 10.5 mm to (114.5, 75.5), turned to 0 degrees
- moved R20 8.14 mm to (112.0, 70.6)
- moved F1 8.06 mm to (110.5, 104.0)
- moved R3 8.04 mm to (119.2, 107.5)
- moved R25 7.75 mm to (110.5, 79.8)
- moved D2 7.60 mm to (112.0, 82.5)
- moved J2 7.25 mm to (103.7, 78.5)
- moved R24 7.25 mm to (110.5, 77.2)
- moved Q1 6.80 mm to (116.5, 104.0), turned to 180 degrees
- moved D1 3.94 mm to (120.0, 104.5), turned to -90 degrees
- moved J11 2.00 mm to (107.5, 123.0)
- moved Q2 1.50 mm to (117.5, 112.5)
- moved R49 1.50 mm to (114.5, 112.4)
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Routing:
- net +5V: track 0.00 -> 12.1 mm
- net +12V: track 0.00 -> 12.0 mm
- net Net-(U1-SW): track 0.00 -> 4.76 mm

Commit message: 原点の設定、修正
パッド、D8の位置
Parts:
- moved D8 5.02 mm to (114.0, 80.5), turned to -90 degrees
- moved REF** 2.24 mm to (150.0, 67.0)
- moved C1 2.00 mm to (137.0, 108.0)
- moved C10 2.00 mm to (144.0, 108.0)
- moved C11 2.00 mm to (171.7, 78.3)
- moved C12 2.00 mm to (159.7, 79.8)
- moved C13 2.00 mm to (160.0, 104.5)
- moved C14 2.00 mm to (158.0, 104.5)
- moved C15 2.00 mm to (163.0, 103.5)
- moved C16 2.00 mm to (168.5, 112.5)
- moved C17 2.00 mm to (165.0, 103.5)
- moved C18 2.00 mm to (168.5, 109.5)
- moved C19 2.00 mm to (149.5, 110.0)
- moved C2 2.00 mm to (137.0, 106.0)
- moved C20 2.00 mm to (155.5, 103.5)
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
Commit message: 固定用穴追加
Parts:
- added REF**: MountingHole_3.2mm_M3_Pad_Via, MountingHole:MountingHole_3.2mm_M3_Pad_Via, F.Cu at (150.0, 130.0)
Changed lines of the file:
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@@
     )
+  )
+  (footprint "MountingHole:MountingHole_3.2mm_M3_Pad_Via" (layer "F.Cu")
+    (at 150 130)
+    (descr "Mounting Hole 3.2mm, M3")
+    (tags "mounting hole 3.2mm m3")
+    (attr exclude_from_pos_files exclude_from_bom)
+    (fp_text reference "REF**" (at 0 -4.2) (layer "F.SilkS")
+        (effects (font (size 1 1) (thickness 0.15)))
+    )
+    (fp_text value "MountingHole_3.2mm_M3_Pad_Via" (at 0 4.2) (layer "F.Fab")
+        (effects (font (size 1 1) (thickness 0.15)))
+    )
+    (fp_text user "${REFERENCE}" (at 0 0) (layer "F.Fab")
+        (effects (font (size 1 1) (thickness 0.15)))
+    )
+    (fp_circle (center 0 0) (end 3.2 0)
+      (stroke (width 0.15) (type solid)) (fill none) (layer "Cmts.User"))
+    (fp_circle (center 0 0) (end 3.45 0)
+      (stroke (width 0.05) (type solid)) (fill none) (layer "F.CrtYd"))
+    (pad "1" thru_hole circle (at -2.4 0) (size 0.8 0.8) (drill 0.5) (layers "*.Cu" "*.Mask"))
+    (pad "1" thru_hole circle (at -1.697056 -1.697056) (size 0.8 0.8) (drill 0.5) (layers "*.Cu" "*.Mask"))
+    (pad "1" thru_hole circle (at -1.697056 1.697056) (size 0.8 0.8) (drill 0.5) (layers "*.Cu" "*.Mask"))
+    (pad "1" thru_hole circle (at 0 -2.4) (size 0.8 0.8) (drill 0.5) (layers "*.Cu" "*.Mask"))
+    (pad "1" thru_hole circle (at 0 0) (size 6.4 6.4) (drill 3.2) (layers "*.Cu" "*.Mask"))
+    (pad "1" thru_hole circle (at 0 2.4) (size 0.8 0.8) (drill 0.5) (layers "*.Cu" "*.Mask"))
+    (pad "1" thru_hole circle (at 1.697056 -1.697056) (size 0.8 0.8) (drill 0.5) (layers "*.Cu" "*.Mask"))
+    (pad "1" thru_hole circle (at 1.697056 1.697056) (size 0.8 0.8) (drill 0.5) (layers "*.Cu" "*.Mask"))
+    (pad "1" thru_hole circle (at 2.4 0) (size 0.8 0.8) (drill 0.5) (layers "*.Cu" "*.Mask"))
   )
   (footprint "Capacitor_SMD:C_0603_1608Metric" (layer "F.Cu")

Commit message: 電源仮配線、デザインルール設定
Parts:
- moved C23 26.6 mm to (168.5, 117.0)
- moved C24 20.9 mm to (168.5, 104.5), turned to 0 degrees
- moved C25 16.5 mm to (168.5, 106.5), turned to 0 degrees
- moved R26 9.48 mm to (185.0, 119.7), turned to 90 degrees
- moved R15 4.61 mm to (149.5, 108.0), turned to 180 degrees
- moved R13 4.27 mm to (149.5, 105.0), turned to 180 degrees
- moved C14 4.03 mm to (157.8, 100.5), turned to 180 degrees
- moved C13 3.99 mm to (159.8, 100.5), turned to 0 degrees
- moved R14 3.91 mm to (149.5, 106.5), turned to 0 degrees
- moved Y1 2.02 mm to (158.8, 103.0)
- moved R27 2.00 mm to (185.0, 91.7)
- moved R28 2.00 mm to (185.0, 105.7)
- moved R17 1.50 mm to (171.5, 119.5)
- moved R18 1.50 mm to (168.5, 119.5)
- moved REF** 1.41 mm to (196.0, 136.0)
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Routing:
- net GND: track 0.00 -> 33.4 mm
- net +12V: track 12.0 -> 22.2 mm
- net +5V: track 12.1 -> 22.2 mm
- net +BATT: track 0.00 -> 8.66 mm
- net Net-(U1-FB): track 0.00 -> 4.95 mm
- net Net-(U1-EN): track 0.00 -> 4.94 mm
- net Net-(D1-A): track 0.00 -> 4.56 mm
- net Net-(Q1-D): track 0.00 -> 3.66 mm
- net Net-(U1-BST): track 0.00 -> 2.75 mm
- net Net-(U1-SS): track 0.00 -> 1.88 mm
- net Net-(C6-Pad1): track 0.00 -> 1.40 mm
- added copper zone on F.Cu, net +BATT
- added copper zone on F.Cu, net Net-(Q1-D)
Other:
- outline, holes or cut-outs redrawn
- copper layers 2 -> 4
