File: main-ECU-board.kicad_pcb (KiCad board)
At the start: 4 copper layers, 100 x 78 mm, 122 parts, among them IC1 TCAN1042DQ1, IC2 R7FA4M1AB3CFM#AA0, IC3 TPS2H160AQPWPRQ1, IC4 TPS2H160AQPWPRQ1, J1 Conn_01x02_Pin, J10 Conn_01x04_Pin, J11 Conn_01x04_Pin, J12 Conn_01x04_Pin, J13 Conn_01x06_Pin, J14 Conn_01x03_Pin, J15 Conn_02x05_Odd_Even, J16 Conn_01x06_Pin, J2 USB_C_Receptacle, J3 Conn_01x03_Pin, J4 Conn_01x03_Pin, J5 Conn_01x03_Pin, J6 Conn_01x03_Pin, J7 Conn_01x02_Pin, J8 Conn_01x02_Pin, J9 Conn_01x02_Pin, Q1 AO3401A, Q2 2N7002K, SW1 SW_Push, U1 TPS62933, Y1 ABM8W-12.0000MHZ-8-K1Z-T3

Commit message: デバッグインターフェースのフットプリント変更
2.54mm pitch -> 1.00 mm pitch
Parts:
- J15: footprint Connector_PinHeader_2.54mm:PinHeader_2x05_P2.54mm_Vertical -> Connector_PinHeader_1.00mm:PinHeader_2x05_P1.00mm_Vertical
- moved J10 72.5 mm to (160.0, 74.5)
- moved C11 5.00 mm to (167.5, 105.3)
- moved C12 5.00 mm to (167.5, 117.3)
- moved D4 5.00 mm to (167.5, 121.0)
- moved IC1 5.00 mm to (167.5, 110.0)
- moved R10 5.00 mm to (170.0, 116.5)
- moved R11 5.00 mm to (165.0, 116.5)
- moved R8 5.00 mm to (171.2, 113.5)
- moved R9 5.00 mm to (167.5, 114.8)
- moved J15 3.24 mm to (179.0, 107.0)

Commit message: ヒューズ変更、コネクタ配置変更、CANまわり配置修正
Parts:
- F1: value MF-USHT020KX-2 -> ERB-RD1R50X; footprint Fuse:Fuse_1210_3225Metric -> Fuse:Fuse_0402_1005Metric
- moved C11 10.3 mm to (171.0, 115.0), turned to -90 degrees
- moved R8 8.64 mm to (164.4, 118.8), turned to 0 degrees
- moved C12 7.63 mm to (161.0, 121.3)
- moved D4 7.63 mm to (161.0, 125.0)
- moved R10 7.63 mm to (163.5, 120.5)
- moved R11 7.63 mm to (158.5, 120.5)
- moved R9 7.63 mm to (161.0, 118.8)
- moved J13 7.50 mm to (125.0, 135.0)
- moved J7 7.50 mm to (150.0, 125.0)
- moved J8 7.50 mm to (137.5, 125.0)
- moved R29 7.50 mm to (146.0, 123.3)
- moved R30 7.50 mm to (133.5, 123.3)
- moved R32 7.50 mm to (121.0, 130.8)
- moved R34 7.50 mm to (121.0, 126.7)
- moved F1 5.83 mm to (110.0, 86.0), turned to -90 degrees
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Connections:
- F1 pad 1: Net-(Q1-D) -> +BATT
- F1 pad 2: +BATT -> Net-(Q1-D)
Routing:
- removed copper zone on F.Cu, net Net-(Q1-D)

Commit message: シルク修正
Parts:
- moved C11 10.7 mm to (167.2, 105.0), turned to 0 degrees
- moved C12 7.48 mm to (167.2, 117.0)
- moved D4 7.48 mm to (167.2, 120.8)
- moved R10 7.48 mm to (169.7, 116.2)
- moved R11 7.48 mm to (164.7, 116.2)
- moved R8 7.48 mm to (170.5, 114.5)
- moved R9 7.48 mm to (167.2, 114.5)
- moved IC1 5.33 mm to (167.2, 109.8), turned to -90 degrees
Changed lines of the file:
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@@
     (property "発注先" "Digi-Key")
     (attr smd)
-    (fp_text reference "R29" (at 0 1.25 90) (layer "F.SilkS")
+    (fp_text reference "R29" (at 0 1.5 90) (layer "F.SilkS")
         (effects (font (size 1 1) (thickness 0.15)))
     )
@@
     (property "発注先" "秋月電子")
     (attr smd)
-    (fp_text reference "D9" (at -3.162 0) (layer "F.SilkS")
+    (fp_text reference "D9" (at -3.35 0) (layer "F.SilkS")
         (effects (font (size 1 1) (thickness 0.15)))
     )
@@
     (property "発注先" "Digi-Key")
     (attr smd)
-    (fp_text reference "R44" (at 4.237 0) (layer "F.SilkS")
+    (fp_text reference "R44" (at 2.925 0) (layer "F.SilkS")
         (effects (font (size 1 1) (thickness 0.15)))
     )
@@
     (property "発注先" "Digi-Key")
     (attr smd)
-    (fp_text reference "R32" (at 0 -1.25 90) (layer "F.SilkS")
+    (fp_text reference "R32" (at 0 -1.5 90) (layer "F.SilkS")
         (effects (font (size 1 1) (thickness 0.15)))
     )
@@
     (property "発注先" "Digi-Key")
     (attr smd)
-    (fp_text reference "R30" (at 0 1.25 90) (layer "F.SilkS")
+    (fp_text reference "R30" (at 0 1.5 90) (layer "F.SilkS")
         (effects (font (size 1 1) (thickness 0.15)))
     )
@@
     (property "発注先" "秋月電子")
     (attr smd)
-    (fp_text reference "D10" (at -3.662 0) (layer "F.SilkS")
+    (fp_text reference "D10" (at -3.85 0) (layer "F.SilkS")
         (effects (font (size 1 1) (thickness 0.15)))
     )
@@
     (property "発注先" "Digi-Key")
     (attr smd)
-    (fp_text reference "R34" (at 0 1.25 -270) (layer "F.SilkS")
+    (fp_text reference "R34" (at 0 1.5 -270) (layer "F.SilkS")
         (effects (font (size 1 1) (thickness 0.15)))
     )
@@
   )
   (footprint "Resistor_SMD:R_0603_1608Metric" (layer "F.Cu")
-    (at 164.364 118.75)
+    (at 170.519 114.5)
     (descr "Resistor SMD 0603 (1608 Metric), square (rectangular) end terminal, IPC_7351 nominal, (Body size source: IPC-SM-782 page 72, https://www.pcb-3d.com/wordpress/wp-content/uploads/ipc-sm-782a_amendment_1_and_2.pdf), generated with kicad-footprint-generator")
     (tags "resistor")
@@
   )
   (footprint "Resistor_SMD:R_0603_1608Metric" (layer "F.Cu")
-    (at 163.5 120.5 180)
+    (at 169.655 116.25 180)
     (descr "Resistor SMD 0603 (1608 Metric), square (rectangular) end terminal, IPC_7351 nominal, (Body size source: IPC-SM-782 page 72, https://www.pcb-3d.com/wordpress/wp-content/uploads/ipc-sm-782a_amendment_1_and_2.pdf), generated with kicad-footprint-generator")
     (tags "resistor")
@@
   )
   (footprint "ProjectEV-kicad-library:SOIC127P600X175-8N" (layer "F.Cu")
-    (at 166.25 115 180)
+    (at 167.155 109.75 -90)
     (descr "D0008B")
     (tags "Integrated Circuit")
@@
     (property "発注先" "Digi-Key")
     (attr smd)
-    (fp_text reference "IC1" (at 0 0) (layer "F.SilkS")
+    (fp_text reference "IC1" (at 0 0 -270) (layer "F.SilkS")
         (effects (font (size 1.27 1.27) (thickness 0.254)))
     )
-    (fp_text value "TCAN1042DQ1" (at 0 0) (layer "F.SilkS") hide
+    (fp_text value "TCAN1042DQ1" (at 0 0 -270) (layer "F.SilkS") hide
         (effects (font (size 1.27 1.27) (thickness 0.254)))
     )
-    (fp_text user "${REFERENCE}" (at 0 0) (layer "F.Fab")
+    (fp_text user "${REFERENCE}" (at 0 0 -270) (layer "F.Fab")
         (effects (font (size 1.27 1.27) (thickness 0.254)))
     )
@@
     (fp_line (start 1.948 2.452) (end -1.948 2.452)
       (stroke (width 0.1) (type solid)) (layer "F.Fab"))
-    (pad "1" smd rect (at -2.711 -1.905 270) (size 0.65 1.528) (layers "F.Cu" "F.Paste" "F.Mask")
+    (pad "1" smd rect (at -2.711 -1.905) (size 0.65 1.528) (layers "F.Cu" "F.Paste" "F.Mask")
       (net 34 "4") (pinfunction "TXD") (pintype "input"))
-    (pad "2" smd rect (at -2.711 -0.635 270) (size 0.65 1.528) (layers "F.Cu" "F.Paste" "F.Mask")
+    (pad "2" smd rect (at -2.711 -0.635) (size 0.65 1.528) (layers "F.Cu" "F.Paste" "F.Mask")
       (net 3 "GND") (pinfunction "GND") (pintype "power_in"))
-    (pad "3" smd rect (at -2.711 0.635 270) (size 0.65 1.528) (layers "F.Cu" "F.Paste" "F.Mask")
+    (pad "3" smd rect (at -2.711 0.635) (size 0.65 1.528) (layers "F.Cu" "F.Paste" "F.Mask")
       (net 2 "+5V") (pinfunction "VCC") (pintype "power_in"))
-    (pad "4" smd rect (at -2.711 1.905 270) (size 0.65 1.528) (layers "F.Cu" "F.Paste" "F.Mask")
+    (pad "4" smd rect (at -2.711 1.905) (size 0.65 1.528) (layers "F.Cu" "F.Paste" "F.Mask")
       (net 35 "5") (pinfunction "RXD") (pintype "output"))
-    (pad "5" smd rect (at 2.711 1.905 270) (size 0.65 1.528) (layers "F.Cu" "F.Paste" "F.Mask")
+    (pad "5" smd rect (at 2.711 1.905) (size 0.65 1.528) (layers "F.Cu" "F.Paste" "F.Mask")
       (net 36 "unconnected-(IC1-NC-Pad5)") (pinfunction "NC") (pintype "no_connect"))
-    (pad "6" smd rect (at 2.711 0.635 270) (size 0.65 1.528) (layers "F.Cu" "F.Paste" "F.Mask")
+    (pad "6" smd rect (at 2.711 0.635) (size 0.65 1.528) (layers "F.Cu" "F.Paste" "F.Mask")
       (net 21 "CANL") (pinfunction "CANL") (pintype "bidirectional"))
-    (pad "7" smd rect (at 2.711 -0.635 270) (size 0.65 1.528) (layers "F.Cu" "F.Paste" "F.Mask")
+    (pad "7" smd rect (at 2.711 -0.635) (size 0.65 1.528) (layers "F.Cu" "F.Paste" "F.Mask")
       (net 22 "CANH") (pinfunction "CANH") (pintype "bidirectional"))
-    (pad "8" smd rect (at 2.711 -1.905 270) (size 0.65 1.528) (layers "F.Cu" "F.Paste" "F.Mask")
+    (pad "8" smd rect (at 2.711 -1.905) (size 0.65 1.528) (layers "F.Cu" "F.Paste" "F.Mask")
       (net 37 "Net-(IC1-STB)") (pinfunction "STB") (pintype "input"))
     (model "${KICAD_PROJECTEV_DIR}/SamacSys_Parts.3dshapes/TCAN1042DQ1.stp"
@@
   )
   (footprint "Package_TO_SOT_SMD:SOT-23" (layer "F.Cu")
-    (at 161 125 90)
+    (at 167.155 120.75 90)
     (descr "SOT, 3 Pin (https://www.jedec.org/system/files/docs/to-236h.pdf variant AB), generated with kicad-footprint-generator ipc_gullwing_generator.py")
     (tags "SOT TO_SOT_SMD")
@@
   )
   (footprint "Capacitor_SMD:C_0603_1608Metric" (layer "F.Cu")
-    (at 161 121.275 -90)
+    (at 167.155 117.025 -90)
     (descr "Capacitor SMD 0603 (1608 Metric), square (rectangular) end terminal, IPC_7351 nominal, (Body size source: IPC-SM-782 page 76, https://www.pcb-3d.com/wordpress/wp-content/uploads/ipc-sm-782a_amendment_1_and_2.pdf), generated with kicad-footprint-generator")
     (tags "capacitor")
@@
     (property "発注先" "秋月電子")
     (attr smd)
-    (fp_text reference "D2" (at 0 2.7) (layer "F.SilkS")
-        (effects (font (size 1.27 1.27) (thickness 0.254)))
+    (fp_text reference "D2" (at 0 2.5) (layer "F.SilkS")
+        (effects (font (size 1 1) (thickness 0.15)))
     )
     (fp_text value "CUHS20S30" (at -0.475 0) (layer "F.SilkS") hide
@@
     (property "発注先" "Digi-Key")
     (attr smd)
-    (fp_text reference "R49" (at 4.237 0) (layer "F.SilkS")
+    (fp_text reference "R49" (at 2.925 0) (layer "F.SilkS")
         (effects (font (size 1 1) (thickness 0.15)))
     )
@@
   )
   (footprint "Resistor_SMD:R_0603_1608Metric" (layer "F.Cu")
-    (at 158.5 120.5 180)
+    (at 164.655 116.25 180)
     (descr "Resistor SMD 0603 (1608 Metric), square (rectangular) end terminal, IPC_7351 nominal, (Body size source: IPC-SM-782 page 72, https://www.pcb-3d.com/wordpress/wp-content/uploads/ipc-sm-782a_amendment_1_and_2.pdf), generated with kicad-footprint-generator")
     (tags "resistor")
@@
   )
   (footprint "Capacitor_SMD:C_0603_1608Metric" (layer "F.Cu")
-    (at 170.961 115 -90)
+    (at 167.155 105.039)
     (descr "Capacitor SMD 0603 (1608 Metric), square (rectangular) end terminal, IPC_7351 nominal, (Body size source: IPC-SM-782 page 76, https://www.pcb-3d.com/wordpress/wp-content/uploads/ipc-sm-782a_amendment_1_and_2.pdf), generated with kicad-footprint-generator")
     (tags "capacitor")
@@
     (property "発注先" "Digi-Key")
     (attr smd)
-    (fp_text reference "C11" (at 0 -1.539 90) (layer "F.SilkS")
+    (fp_text reference "C11" (at 0 -1.539) (layer "F.SilkS")
         (effects (font (size 1 1) (thickness 0.15)))
     )
-    (fp_text value "0.1u" (at 0 1.43 90) (layer "F.Fab")
+    (fp_text value "0.1u" (at 0 1.43) (layer "F.Fab")
         (effects (font (size 1 1) (thickness 0.15)))
     )
-    (fp_text user "${REFERENCE}" (at 0 0 90) (layer "F.Fab")
+    (fp_text user "${REFERENCE}" (at 0 0) (layer "F.Fab")
         (effects (font (size 0.4 0.4) (thickness 0.06)))
     )
@@
     (fp_line (start 0.8 0.4) (end -0.8 0.4)
       (stroke (width 0.1) (type solid)) (layer "F.Fab"))
-    (pad "1" smd roundrect (at -0.775 0 270) (size 0.9 0.95) (layers "F.Cu" "F.Paste" "F.Mask") (roundrect_rratio 0.25)
+    (pad "1" smd roundrect (at -0.775 0) (size 0.9 0.95) (layers "F.Cu" "F.Paste" "F.Mask") (roundrect_rratio 0.25)
       (net 2 "+5V") (pintype "passive"))
-    (pad "2" smd roundrect (at 0.775 0 270) (size 0.9 0.95) (layers "F.Cu" "F.Paste" "F.Mask") (roundrect_rratio 0.25)
+    (pad "2" smd roundrect (at 0.775 0) (size 0.9 0.95) (layers "F.Cu" "F.Paste" "F.Mask") (roundrect_rratio 0.25)
       (net 3 "GND") (pintype "passive"))
     (model "${KICAD6_3DMODEL_DIR}/Capacitor_SMD.3dshapes/C_0603_1608Metric.wrl"
@@
     (property "発注先" "Digi-Key")
     (attr smd)
-    (fp_text reference "R33" (at 0 1.25 -270) (layer "F.SilkS")
+    (fp_text reference "R33" (at 0 1.5 -270) (layer "F.SilkS")
         (effects (font (size 1 1) (thickness 0.15)))
     )
@@
   )
   (footprint "Resistor_SMD:R_0603_1608Metric" (layer "F.Cu")
-    (at 161 118.75 180)
+    (at 167.155 114.5 180)
     (descr "Resistor SMD 0603 (1608 Metric), square (rectangular) end terminal, IPC_7351 nominal, (Body size source: IPC-SM-782 page 72, https://www.pcb-3d.com/wordpress/wp-content/uploads/ipc-sm-782a_amendment_1_and_2.pdf), generated with kicad-footprint-generator")
     (tags "resistor")
@@
     (property "発注先" "Digi-Key")
     (attr smd)
-    (fp_text reference "R31" (at 0 -1.25 90) (layer "F.SilkS")
+    (fp_text reference "R31" (at 0 -1.5 90) (layer "F.SilkS")
         (effects (font (size 1 1) (thickness 0.15)))
     )

Commit message: 電源パターン修正
合わせてその他部品配置の修正、コネクタ配置修正
Parts:
- moved J13 13.5 mm to (112.5, 130.0), turned to 0 degrees
- moved J16 12.0 mm to (175.0, 67.5), turned to 0 degrees
- moved J10 8.75 mm to (157.2, 67.5), turned to 0 degrees
- moved R31 7.98 mm to (174.2, 126.0), turned to 0 degrees
- moved R33 7.98 mm to (178.3, 126.0), turned to 180 degrees
- moved R32 6.48 mm to (116.7, 126.0), turned to 0 degrees
- moved R29 5.78 mm to (149.2, 118.5), turned to 180 degrees
- moved R30 5.78 mm to (136.7, 118.5), turned to 180 degrees
- moved J12 5.59 mm to (172.5, 130.0), turned to 0 degrees
- moved J9 5.59 mm to (160.0, 130.0), turned to 0 degrees
- moved Q2 5.59 mm to (122.5, 93.8)
- moved R50 5.59 mm to (119.5, 93.6)
- moved R51 5.59 mm to (125.5, 92.9)
- moved D9 5.15 mm to (132.2, 104.2)
- moved IC3 5.15 mm to (127.5, 110.0)
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Routing:
- net Net-(U1-SW): track 0.00 -> 1.58 mm
- net +5V: track 0.00 -> 1.54 mm
- net Net-(U1-FB): track 5.13 -> 3.93 mm
- net +12V: track 0.00 -> 1.01 mm
- net Net-(U1-BST): track 2.75 -> 2.14 mm
- removed copper zone on B.Cu, net GND
- removed copper zone on F.Cu, net GND
- removed copper zone on In1.Cu, net GND
- removed copper zone on In2.Cu, net GND

Commit message: 部品配置修正、基板外形サイズ変更
Parts:
- moved J15 33.5 mm to (145.5, 108.0), turned to 90 degrees
- moved J8 17.7 mm to (152.5, 120.0)
- moved R30 17.7 mm to (154.2, 116.0)
- moved Q2 15.2 mm to (137.5, 96.2)
- moved R50 15.2 mm to (134.5, 96.1)
- moved R51 15.2 mm to (140.5, 95.4)
- moved J3 12.2 mm to (180.0, 117.5)
- moved R26 12.2 mm to (176.0, 114.2)
- moved R7 11.4 mm to (146.8, 93.0), turned to -90 degrees
- moved J7 10.6 mm to (140.0, 130.0)
- moved R29 10.6 mm to (141.7, 126.0)
- moved J11 8.75 mm to (110.0, 117.5)
- moved C1 8.38 mm to (129.5, 96.5)
- moved C2 8.38 mm to (129.5, 94.5)
- moved C3 8.38 mm to (128.8, 92.5)
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Connections:
- J16 pad 1: GND -> +5V
- J16 pad 2: P205_OPT_I/O -> P003_OPT_I/O
- J16 pad 3: P113_OPT_I/O -> P004_OPT_I/O
- J16 pad 4: P004_OPT_I/O -> P113_OPT_I/O
- J16 pad 5: P003_OPT_I/O -> P205_OPT_I/O
- J16 pad 6: +5V -> GND
Routing:
- removed copper zone on F.Cu, net +5V

Commit message: シルク修正、部品配置修正、電源パターン修正
Parts:
- moved J8 12.7 mm to (140.0, 117.5)
- moved R30 12.7 mm to (141.7, 113.5)
- moved J15 1.25 mm to (145.5, 106.8)
- moved R36 1.25 mm to (138.8, 108.5)
- moved R37 1.25 mm to (138.8, 106.8)
- moved R38 1.25 mm to (138.8, 110.2)
- moved R39 1.25 mm to (138.8, 105.0)
Routing:
- net Net-(D1-A): track 2.81 -> 4.56 mm
- added copper zone on F.Cu, net +5V
- added copper zone on F.Cu, net +BATT
- added copper zone on F.Cu, net Net-(Q1-D)
Other:
- board size 100 x 78 mm -> 100 x 65 mm
Changed lines of the file:
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@@
     (property "発注先" "Digi-Key")
     (attr smd)
-    (fp_text reference "L1" (at 4.75 -3) (layer "F.SilkS")
+    (fp_text reference "L1" (at 5 -3.25) (layer "F.SilkS")
         (effects (font (size 1 1) (thickness 0.15)))
     )
@@
   )
   (footprint "Resistor_SMD:R_0603_1608Metric" (layer "F.Cu")
-    (at 154.175 116 180)
+    (at 141.675 113.5 180)
     (descr "Resistor SMD 0603 (1608 Metric), square (rectangular) end terminal, IPC_7351 nominal, (Body size source: IPC-SM-782 page 72, https://www.pcb-3d.com/wordpress/wp-content/uploads/ipc-sm-782a_amendment_1_and_2.pdf), generated with kicad-footprint-generator")
     (tags "resistor")
@@
   )
   (footprint "Resistor_SMD:R_0603_1608Metric" (layer "F.Cu")
-    (at 138.75 108 180)
+    (at 138.75 106.75 180)
     (descr "Resistor SMD 0603 (1608 Metric), square (rectangular) end terminal, IPC_7351 nominal, (Body size source: IPC-SM-782 page 72, https://www.pcb-3d.com/wordpress/wp-content/uploads/ipc-sm-782a_amendment_1_and_2.pdf), generated with kicad-footprint-generator")
     (tags "resistor")
@@
     (property "発注先" "Digi-Key")
     (attr smd)
-    (fp_text reference "IC3" (at 0 0 180) (layer "F.SilkS")
+    (fp_text reference "IC3" (at 0 -4 180) (layer "F.SilkS")
         (effects (font (size 1.27 1.27) (thickness 0.254)))
     )
@@
     (property "発注先" "Digi-Key")
     (attr smd)
-    (fp_text reference "IC2" (at 0 0 -90) (layer "F.SilkS")
+    (fp_text reference "IC2" (at -6.25 -6.75) (layer "F.SilkS")
         (effects (font (size 1.27 1.27) (thickness 0.254)))
     )
@@
   )
   (footprint "Connector_JST:JST_XH_B2B-XH-A_1x02_P2.50mm_Vertical" (layer "F.Cu")
-    (at 152.5 120)
+    (at 140 117.5)
     (descr "JST XH series connector, B2B-XH-A (http://www.jst-mfg.com/product/pdf/eng/eXH.pdf), generated with kicad-footprint-generator")
     (tags "connector JST XH vertical")
@@
     (property "発注先" "Digi-Key")
     (attr smd)
-    (fp_text reference "IC1" (at 0 0 90) (layer "F.SilkS")
+    (fp_text reference "IC1" (at 0 3.655 90) (layer "F.SilkS")
         (effects (font (size 1.27 1.27) (thickness 0.254)))
     )
@@
   )
   (footprint "Resistor_SMD:R_0603_1608Metric" (layer "F.Cu")
-    (at 138.75 111.5 180)
+    (at 138.75 110.25 180)
     (descr "Resistor SMD 0603 (1608 Metric), square (rectangular) end terminal, IPC_7351 nominal, (Body size source: IPC-SM-782 page 72, https://www.pcb-3d.com/wordpress/wp-content/uploads/ipc-sm-782a_amendment_1_and_2.pdf), generated with kicad-footprint-generator")
     (tags "resistor")
@@
     (property "発注先" "Digi-Key")
     (attr smd)
-    (fp_text reference "IC4" (at 0 0 180) (layer "F.SilkS")
+    (fp_text reference "IC4" (at 0 -4 180) (layer "F.SilkS")
         (effects (font (size 1.27 1.27) (thickness 0.254)))
     )
@@
   )
   (footprint "Resistor_SMD:R_0603_1608Metric" (layer "F.Cu")
-    (at 138.75 109.75)
+    (at 138.75 108.5)
     (descr "Resistor SMD 0603 (1608 Metric), square (rectangular) end terminal, IPC_7351 nominal, (Body size source: IPC-SM-782 page 72, https://www.pcb-3d.com/wordpress/wp-content/uploads/ipc-sm-782a_amendment_1_and_2.pdf), generated with kicad-footprint-generator")
     (tags "resistor")
@@
   )
   (footprint "Resistor_SMD:R_0603_1608Metric" (layer "F.Cu")
-    (at 138.75 106.25 180)
+    (at 138.75 105 180)
     (descr "Resistor SMD 0603 (1608 Metric), square (rectangular) end terminal, IPC_7351 nominal, (Body size source: IPC-SM-782 page 72, https://www.pcb-3d.com/wordpress/wp-content/uploads/ipc-sm-782a_amendment_1_and_2.pdf), generated with kicad-footprint-generator")
     (tags "resistor")
@@
   )
   (footprint "Connector_PinHeader_1.00mm:PinHeader_2x05_P1.00mm_Vertical" (layer "F.Cu")
-    (at 145.5 108 90)
+    (at 145.5 106.75 90)
     (descr "Through hole straight pin header, 2x05, 1.00mm pitch, double rows")
     (tags "Through hole pin header THT 2x05 1.00mm double row")
@@
   (gr_rect (start 100 35) (end 200 135)
     (stroke (width 0.15) (type default)) (fill none) (layer "Dwgs.User"))
-  (gr_arc (start 200 146) (mid 199.414214 147.414214) (end 198 148)
+  (gr_arc (start 200 133) (mid 199.414214 134.414214) (end 198 135)
     (stroke (width 0.1) (type default)) (layer "Edge.Cuts"))
-  (gr_line (start 102 148) (end 198 148)
+  (gr_line (start 102 135) (end 198 135)
     (stroke (width 0.1) (type default)) (layer "Edge.Cuts"))
   (gr_arc (start 100 72) (mid 100.585786 70.585786) (end 102 70)
     (stroke (width 0.1) (type default)) (layer "Edge.Cuts"))
-  (gr_line (start 200 146) (end 200 72)
+  (gr_line (start 200 133) (end 200 72)
     (stroke (width 0.1) (type default)) (layer "Edge.Cuts"))
   (gr_line (start 198 70) (end 102 70)
     (stroke (width 0.1) (type default)) (layer "Edge.Cuts"))
-  (gr_arc (start 102 148) (mid 100.585786 147.414214) (end 100 146)
+  (gr_arc (start 102 135) (mid 100.585786 134.414214) (end 100 133)
     (stroke (width 0.1) (type default)) (layer "Edge.Cuts"))
-  (gr_line (start 100 72) (end 100 146)
+  (gr_line (start 100 72) (end 100 133)
     (stroke (width 0.1) (type default)) (layer "Edge.Cuts"))
   (gr_arc (start 198 70) (mid 199.414214 70.585786) (end 200 72)
@@
   (segment (start 125.325 86.5) (end 125.325 89) (width 0.5) (layer "F.Cu") (net 8))
   (segment (start 125.325 89) (end 125.575 89.25) (width 0.5) (layer "F.Cu") (net 8))
+  (segment (start 109.2 97.75) (end 110.95 97.75) (width 0.5) (layer "F.Cu") (net 18))
   (segment (start 111.55 95.1875) (end 111.55 97.15) (width 0.5) (layer "F.Cu") (net 18))
   (segment (start 111.55 97.15) (end 110.95 97.75) (width 0.5) (layer "F.Cu") (net 18))
@@
       )
     )
+  )
+  (zone (net 2) (net_name "+5V") (layer "F.Cu") (hatch edge 0.5)
+    (priority 5)
+    (connect_pads yes (clearance 0))
+    (min_thickness 0.25) (filled_areas_thickness no)
+    (fill yes (thermal_gap 0.5) (thermal_bridge_width 0.5))
+    (polygon
+      (pts
+        (xy 137 85.25)
+        (xy 136.5 85.75)
+        (xy 136.5 89.25)
+        (xy 137 89.75)
+        (xy 147 89.75)
+        (xy 147.5 89.25)
+        (xy 147.5 85.75)
+        (xy 147 85.25)
+      )
+    )
+  )
+  (zone (net 32) (net_name "+BATT") (layer "F.Cu") (hatch edge 0.5)
+    (priority 1)
+    (connect_pads yes (clearance 0))
+    (min_thickness 0.25) (filled_areas_thickness no)
+    (fill yes (thermal_gap 0.5) (thermal_bridge_width 0.5))
+    (polygon
+      (pts
+        (xy 107 83.75)
+        (xy 106.5 84.25)
+        (xy 106.5 89.25)
+        (xy 109 91.75)
+        (xy 109.5 91.75)
+        (xy 109.75 91.5)
+        (xy 109.75 89.75)
+        (xy 108.5 88.5)
+        (xy 108.5 84.25)
+        (xy 108 83.75)
+      )
+    )
+  )
+  (zone (net 31) (net_name "Net-(Q1-D)") (layer "F.Cu") (hatch edge 0.5)
+    (priority 4)
+    (connect_pads yes (clearance 0))
+    (min_thickness 0.25) (filled_areas_thickness no)
+    (fill yes (thermal_gap 0.5) (thermal_bridge_width 0.5))
+    (polygon
+      (pts
+        (xy 110.5 90.75)
+        (xy 110.25 91)
+        (xy 110.25 92)
+        (xy 112.25 94)
+        (xy 112.75 94)
+        (xy 113 93.75)
+        (xy 113 92.75)
+        (xy 111 90.75)
+      )
+    )
