File: main-ECU-board.kicad_pcb (KiCad board)
At the start: 4 copper layers, 100 x 65 mm, 122 parts, among them IC1 TCAN1042DQ1, IC2 R7FA4M1AB3CFM#AA0, IC3 TPS2H160AQPWPRQ1, IC4 TPS2H160AQPWPRQ1, J1 Conn_01x02_Pin, J10 Conn_01x04_Pin, J11 Conn_01x04_Pin, J12 Conn_01x04_Pin, J13 Conn_01x06_Pin, J14 Conn_01x03_Pin, J15 Conn_02x05_Odd_Even, J16 Conn_01x06_Pin, J2 USB_C_Receptacle, J3 Conn_01x03_Pin, J4 Conn_01x03_Pin, J5 Conn_01x03_Pin, J6 Conn_01x03_Pin, J7 Conn_01x02_Pin, J8 Conn_01x02_Pin, J9 Conn_01x02_Pin, Q1 AO3401A, Q2 2N7002K, SW1 SW_Push, U1 TPS62933, Y1 ABM8W-12.0000MHZ-8-K1Z-T3

Commit message: 電源パターン追加修正、電源部品配置修正
Parts:
- moved D8 0.74 mm to (119.3, 81.2), turned to 90 degrees
- moved C8 0.25 mm to (141.2, 90.2)
- moved C9 0.25 mm to (143.2, 90.2)
- moved L1 0.25 mm to (135.2, 87.8)
Routing:
- net Net-(U1-SW): track 1.58 -> 2.33 mm
Changed lines of the file:
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@@
   )
   (footprint "ProjectEV-kicad-library:L_MGAH0603" (layer "F.Cu")
-    (at 135.25 87.5)
+    (at 135.25 87.75)
     (descr "https://www.laird.com/sites/default/files/2022-01/MGAH0603%20Series.pdf")
     (tags "Inductor bmrx mchi")
@@
   )
   (footprint "Capacitor_SMD:C_0805_2012Metric" (layer "F.Cu")
-    (at 143.25 90 -90)
+    (at 143.25 90.25 -90)
     (descr "Capacitor SMD 0805 (2012 Metric), square (rectangular) end terminal, IPC_7351 nominal, (Body size source: IPC-SM-782 page 76, https://www.pcb-3d.com/wordpress/wp-content/uploads/ipc-sm-782a_amendment_1_and_2.pdf, https://docs.google.com/spreadsheets/d/1BsfQQcO9C6DZCsRaXUlFlo91Tg2WpOkGARC1WS5S8t0/edit?usp=sharing), generated with kicad-footprint-generator")
     (tags "capacitor")
@@
   )
   (footprint "digikey-footprints:TO-253-4" (layer "F.Cu")
-    (at 120 81.5 180)
+    (at 119.3 81.25 90)
     (descr "https://www.digikey.com/products/en?keywords=1727-3884-1")
     (property "Category" "Circuit Protection")
@@
     (property "発注先" "Digi-Key")
     (attr smd)
-    (fp_text reference "D8" (at 0 -2.75 180) (layer "F.SilkS")
+    (fp_text reference "D8" (at 0 -2.75 90) (layer "F.SilkS")
         (effects (font (size 1 1) (thickness 0.15)))
     )
-    (fp_text value "PRTR5V0U2X_215" (at 0 3.25) (layer "F.Fab")
+    (fp_text value "PRTR5V0U2X_215" (at 0 3.25 90) (layer "F.Fab")
         (effects (font (size 1 1) (thickness 0.15)))
     )
-    (fp_text user "${REFERENCE}" (at 0.1 -0.1 90) (layer "F.Fab")
+    (fp_text user "${REFERENCE}" (at 0.1 -0.1) (layer "F.Fab")
         (effects (font (size 0.5 0.5) (thickness 0.05)))
     )
@@
     (fp_line (start 0.7 -1.5) (end 0.7 1.5)
       (stroke (width 0.1) (type solid)) (layer "F.Fab"))
-    (pad "1" smd rect (at -1 -0.75 180) (size 0.7 1) (layers "F.Cu" "F.Paste" "F.Mask")
+    (pad "1" smd rect (at -1 -0.75 90) (size 0.7 1) (layers "F.Cu" "F.Paste" "F.Mask")
       (net 3 "GND") (pinfunction "GND") (pintype "passive"))
-    (pad "2" smd rect (at -1 0.95 180) (size 0.7 0.6) (layers "F.Cu" "F.Paste" "F.Mask")
+    (pad "2" smd rect (at -1 0.95 90) (size 0.7 0.6) (layers "F.Cu" "F.Paste" "F.Mask")
       (net 27 "USB_D_M") (pinfunction "I/O1") (pintype "output"))
-    (pad "3" smd rect (at 1 0.95 180) (size 0.7 0.6) (layers "F.Cu" "F.Paste" "F.Mask")
+    (pad "3" smd rect (at 1 0.95 90) (size 0.7 0.6) (layers "F.Cu" "F.Paste" "F.Mask")
       (net 28 "USB_D_P") (pinfunction "I/O2") (pintype "output"))
-    (pad "4" smd rect (at 1 -0.95 180) (size 0.7 0.6) (layers "F.Cu" "F.Paste" "F.Mask")
+    (pad "4" smd rect (at 1 -0.95 90) (size 0.7 0.6) (layers "F.Cu" "F.Paste" "F.Mask")
       (net 19 "VBUS") (pinfunction "VCC") (pintype "passive"))
   )
@@
   )
   (footprint "Capacitor_SMD:C_0805_2012Metric" (layer "F.Cu")
-    (at 141.25 90 -90)
+    (at 141.25 90.25 -90)
     (descr "Capacitor SMD 0805 (2012 Metric), square (rectangular) end terminal, IPC_7351 nominal, (Body size source: IPC-SM-782 page 76, https://www.pcb-3d.com/wordpress/wp-content/uploads/ipc-sm-782a_amendment_1_and_2.pdf, https://docs.google.com/spreadsheets/d/1BsfQQcO9C6DZCsRaXUlFlo91Tg2WpOkGARC1WS5S8t0/edit?usp=sharing), generated with kicad-footprint-generator")
     (tags "capacitor")
@@
   (segment (start 127.25 88.23) (end 127.25 89.26) (width 0.3) (layer "F.Cu") (net 5))
   (segment (start 128.25 84.25) (end 128.25 85.675) (width 0.5) (layer "F.Cu") (net 6))
-  (segment (start 129.8 85.55) (end 130 85.75) (width 0.5) (layer "F.Cu") (net 7))
-  (segment (start 129.8 84.25) (end 129.8 85.55) (width 0.5) (layer "F.Cu") (net 7))
+  (segment (start 129.8 86.3) (end 130 86.5) (width 0.5) (layer "F.Cu") (net 7))
+  (segment (start 129.8 84.25) (end 129.8 86.3) (width 0.5) (layer "F.Cu") (net 7))
   (segment (start 125.575 89.25) (end 126.64 89.25) (width 0.5) (layer "F.Cu") (net 8))
   (segment (start 126.64 89.25) (end 126.65 89.26) (width 0.5) (layer "F.Cu") (net 8))
@@
         (xy 128.25 89)
         (xy 129.25 88)
-        (xy 129.25 85.75)
-        (xy 129.75 85.25)
-        (xy 133.5 85.25)
-        (xy 134 85.75)
+        (xy 129.25 86.25)
+        (xy 129.75 85.75)
+        (xy 133.5 85.75)
+        (xy 134 86.25)
         (xy 134 89.25)
         (xy 133.5 89.75)
@@
     (polygon
       (pts
-        (xy 137 85.25)
-        (xy 136.5 85.75)
+        (xy 137 85.75)
+        (xy 136.5 86.25)
         (xy 136.5 89.25)
         (xy 137 89.75)
         (xy 147 89.75)
         (xy 147.5 89.25)
-        (xy 147.5 85.75)
-        (xy 147 85.25)
+        (xy 147.5 86.25)
+        (xy 147 85.75)
       )
     )
@@
   )
   (zone (net 4) (net_name "+12V") (layer "F.Cu") (hatch edge 0.5)
-    (connect_pads yes (clearance 0))
-    (min_thickness 0.25) (filled_areas_thickness no)
-    (fill yes (thermal_gap 0.5) (thermal_bridge_width 0.5))
-    (polygon
-      (pts
-        (xy 126 93)
-        (xy 125 93)
-        (xy 124.75 93.25)
-        (xy 124.75 94)
-        (xy 124.5 94.25)
-        (xy 125.5 94.25)
-        (xy 126 93.75)
-      )
-    )
-  )
-  (zone (net 4) (net_name "+12V") (layer "F.Cu") (hatch edge 0.5)
     (priority 2)
     (connect_pads yes (clearance 0))
@@
     (polygon
       (pts
-        (xy 113.25 94.25)
-        (xy 112.75 94.75)
+        (xy 113.25 94.5)
+        (xy 112.75 95)
         (xy 112.75 98)
         (xy 113.25 98.5)
-        (xy 127.75 98.5)
-        (xy 129.25 97)
+        (xy 127.5 98.5)
+        (xy 129.25 96.75)
         (xy 129.25 93.75)
         (xy 128.5 93)
@@
         (xy 127.6 91.4)
         (xy 126 93)
-        (xy 126 93.75)
-        (xy 125.5 94.25)
+        (xy 126 94)
+        (xy 125.5 94.5)
+      )
+    )
+  )
+  (zone (net 2) (net_name "+5V") (layer "F.Cu") (hatch edge 0.5)
+    (connect_pads yes (clearance 0))
+    (min_thickness 0.25) (filled_areas_thickness no)
+    (fill yes (thermal_gap 0.5) (thermal_bridge_width 0.5))
+    (polygon
+      (pts
+        (xy 125.25 81.25)
+        (xy 126.25 82.25)
+        (xy 132 82.25)
+        (xy 136.5 86.75)
+        (xy 138 86.75)
+        (xy 138.5 86.25)
+        (xy 138.5 85.75)
+        (xy 133 80.25)
+        (xy 125.75 80.25)
+        (xy 125.25 80.75)
       )
     )

Commit message: 電源、クロック、一部部品配置修正
Parts:
- moved SW1 6.52 mm to (137.2, 75.0), turned to 0 degrees
- moved D8 2.83 mm to (121.7, 82.8), turned to -90 degrees
- moved R17 2.55 mm to (171.2, 105.0)
- moved C14 2.53 mm to (161.6, 83.0)
- moved R18 2.51 mm to (171.2, 103.2)
- moved R36 2.50 mm to (138.8, 106.0)
- moved R37 2.50 mm to (138.8, 104.2)
- moved R38 2.50 mm to (138.8, 107.8)
- moved R39 2.50 mm to (138.8, 102.5)
- moved Y1 2.02 mm to (162.0, 86.0), turned to -90 degrees
- moved D2 1.82 mm to (127.0, 80.2)
- moved C13 1.68 mm to (164.5, 86.6), turned to -90 degrees
- moved C22 1.25 mm to (161.0, 107.2), turned to 0 degrees
- moved D7 1.15 mm to (154.8, 109.0), turned to 180 degrees
- moved R42 1.12 mm to (161.0, 109.0)
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Connections:
- Y1 pad 4: unconnected-(Y1-Pad4) -> GND
Routing:
- net VBUS: track 0.00 -> 8.94 mm, vias 0 -> 2
- net USB_D_P: track 0.00 -> 8.66 mm
- net USB_D_M: track 0.00 -> 7.89 mm
- net +12V: track 1.01 -> 1.94 mm
- net +5V: vias 0 -> 24
- added copper zone on In2.Cu, net +5V
- added copper zone on F.Cu, net VBUS
